Commit message: Correcting reference frames for geometries

File: model/complete_soft_hand.urdf.xacro (robot description, xacro)
@@ -17,8 +17,8 @@
 		<!-- abductor joint between palm_link and finger_abd_link - fake between palm and proximal -->
 		<joint name="${name}_abd_joint" type="revolute">
-				<origin xyz="${position}" rpy="${orientation}" />
+			<origin xyz="${position}" rpy="${orientation}" />
 			<parent link="${parent}"/>
 			<child link="${name}_knuckle_link"/>
-				<axis xyz="0 0 1" />
+			<axis xyz="0 0 1" />
 			<limit lower="${inner_lb *pi/180}" upper="${inner_ub *pi/180}" effort="${effort}" velocity="${velocity}"/>
 		</joint>
@@ -35,20 +35,20 @@
 		<!-- immaginary link-->
 		<!-- joint and link FAKE 1-->
-			<joint name="${name}_fake_joint1" type="revolute">
-					<origin xyz="0 0 0" rpy="0 0 0" />
-				<parent link="${name}_knuckle_link"/>
-				<child link="${name}_fake_link1"/>
-					<axis xyz="0 1 0" />
-				<limit lower="${inner_lb *pi/180}" upper="${inner_ub *pi/180}" effort="${effort}" velocity="${velocity}"/>
-			</joint>
-			<link name="${name}_fake_link1">
-			</link>
+		<joint name="${name}_fake_joint1" type="revolute">
+			<origin xyz="-0.009 0 0" rpy="0 0 0" />
+			<parent link="${name}_knuckle_link"/>
+			<child link="${name}_fake_link1"/>
+			<axis xyz="0 1 0" />
+			<limit lower="${inner_lb *pi/180}" upper="${inner_ub *pi/180}" effort="${effort}" velocity="${velocity}"/>
+		</joint>
+		<link name="${name}_fake_link1">
+		</link>
 		<!-- end immaginary link-->
 		<!-- abductor joint between palm_link and finger_abd_link - fake between palm and proximal -->
 		<joint name="${name}_inner_joint" type="revolute">
-			<origin xyz="-0.02 0 0" rpy="0 0 0" />
-				<parent link="${name}_fake_link1"/>
+			<origin xyz="-0.013 0 0" rpy="0 0 0" />
+			<parent link="${name}_fake_link1"/>
 			<child link="${name}_proximal_link"/>
-				<axis xyz="0 1 0" />
+			<axis xyz="0 1 0" />
 			<mimic joint="${name}_fake_joint1" multiplier="1" />
 			<limit lower="${middle_lb *pi/180}" upper="${middle_ub *pi/180}" effort="${effort}" velocity="${velocity}"/>
@@ -58,5 +58,5 @@
 				<origin xyz="0 0 0" rpy="0 0 0" />
 				<geometry>
-					<mesh filename="package://complete_soft_hand/meshes/phalanx_short.stl" scale=" .001 .001 .001" />
+					<mesh filename="package://complete_soft_hand/meshes/phalanx_short_injection.stl" scale=" .001 .001 .001" />
 				</geometry>
 				<material name="DarkGolden" />
@@ -66,16 +66,16 @@
 		<!-- immaginary link-->
 		<!-- joint and link FAKE 2-->
-			<joint name="${name}_fake_joint2" type="revolute">
-					<origin xyz="-0 0 0" rpy="0 0 0" />
-				<parent link="${name}_proximal_link"/>
-				<child link="${name}_fake_link2"/>
-					<axis xyz="0 1 0" />
-				<limit lower="${inner_lb *pi/180}" upper="${inner_ub *pi/180}" effort="${effort}" velocity="${velocity}"/>
-			</joint>
-			<link name="${name}_fake_link2">
-			</link>
-		<!-- end immaginary link-->
-	    <joint name="${name}_middle_joint" type="revolute">
-			<origin xyz="-0.02 0 0" rpy="0 0 0" />
+		<joint name="${name}_fake_joint2" type="revolute">
+			<origin xyz="-0.009 0 0" rpy="0 0 0" />
+			<parent link="${name}_proximal_link"/>
+			<child link="${name}_fake_link2"/>
+			<axis xyz="0 1 0" />
+			<limit lower="${inner_lb *pi/180}" upper="${inner_ub *pi/180}" effort="${effort}" velocity="${velocity}"/>
+		</joint>
+		<link name="${name}_fake_link2">
+		</link>
+		<!-- end immaginary link-->
+		<joint name="${name}_middle_joint" type="revolute">
+			<origin xyz="-0.013 0 0" rpy="0 0 0" />
 			<parent link="${name}_fake_link2"/>
 			<child link="${name}_middle_link"/>
@@ -88,7 +88,7 @@
 				<origin xyz="0 0 0" rpy="0 0 0" />
 				<geometry>
-					<mesh filename="package://complete_soft_hand/meshes/phalanx_short.stl" scale=" .001 .001 .001" />
-				</geometry>
-			<material name="DarkGolden" />
+					<mesh filename="package://complete_soft_hand/meshes/phalanx_short_injection.stl" scale=" .001 .001 .001" />
+				</geometry>
+				<material name="DarkGolden" />
 			</visual>
 		</link>
@@ -96,16 +96,16 @@
 		<!-- immaginary link-->
 		<!-- joint and link FAKE 3-->
-			<joint name="${name}_fake_joint3" type="revolute">
-					<origin xyz="0 0 0" rpy="0 0 0" />
-				<parent link="${name}_middle_link"/>
-				<child link="${name}_fake_link3"/>
-					<axis xyz="0 1 0" />
-				<limit lower="${inner_lb *pi/180}" upper="${inner_ub *pi/180}" effort="${effort}" velocity="${velocity}"/>
-			</joint>
-			<link name="${name}_fake_link3">
-			</link>
+		<joint name="${name}_fake_joint3" type="revolute">
+			<origin xyz="-0.009 0 0" rpy="0 0 0" />
+			<parent link="${name}_middle_link"/>
+			<child link="${name}_fake_link3"/>
+			<axis xyz="0 1 0" />
+			<limit lower="${inner_lb *pi/180}" upper="${inner_ub *pi/180}" effort="${effort}" velocity="${velocity}"/>
+		</joint>
+		<link name="${name}_fake_link3">
+		</link>
 		<!-- end immaginary link-->
 		<joint name="${name}_outer_joint" type="revolute">
-			<origin xyz="-0.02 0 0" rpy="0 0 0" />
+			<origin xyz="-0.013 0 0" rpy="0 0 0" />
 			<parent link="${name}_fake_link3"/>
 			<child link="${name}_distal_link"/>
@@ -120,5 +120,117 @@
 					<mesh filename="package://complete_soft_hand/meshes/phalanx_distal_out_no_ati.stl" scale=" .001 .001 .001" />
 				</geometry>
-			<material name="DarkGolden" />
+				<material name="DarkGolden" />
+			</visual>
+		</link>
+		<!-- end BABY PHALANGE -->
+	</xacro:macro>
+	<xacro:macro name="thumb_finger" params="parent name position orientation">
+		<!-- macro for one finger -->
+		<!-- abductor joint between palm_link and finger_abd_link - fake between palm and proximal -->
+		<joint name="${name}_abd_joint" type="revolute">
+			<origin xyz="${position}" rpy="${orientation}" />
+			<parent link="${parent}"/>
+			<child link="${name}_knuckle_link"/>
+			<axis xyz="0 1 0" />
+			<limit lower="${-2*inner_ub *pi/180}" upper="${inner_lb *pi/180}" effort="${effort}" velocity="${velocity}"/>
+		</joint>
+		<link name="${name}_knuckle_link">
+			<visual>
+				<origin xyz="0 0 0" rpy="0 0 0" />
+				<geometry>
+					<mesh filename="package://complete_soft_hand/meshes/phalanx_thumb_injection.stl" scale=" .001 .001 .001" />
+				</geometry>
+				<material name="DarkGolden" />
+			</visual>
+		</link>
+		<!-- PHALANGE -->
+		<!-- immaginary link-->
+		<!-- joint and link FAKE 1-->
+		<joint name="${name}_fake_joint1" type="revolute">
+			<origin xyz="-0.0225 0 -0.0033" rpy="-1.9974238811 0 0" />
+			<parent link="${name}_knuckle_link"/>
+			<child link="${name}_fake_link1"/>
+			<axis xyz="0 1 0" />
+			<limit lower="${inner_lb *pi/180}" upper="${inner_ub *pi/180}" effort="${effort}" velocity="${velocity}"/>
+		</joint>
+		<link name="${name}_fake_link1">
+		</link>
+		<!-- end immaginary link-->
+		<!-- abductor joint between palm_link and finger_abd_link - fake between palm and proximal -->
+		<joint name="${name}_inner_joint" type="revolute">
+			<origin xyz="-0.013 0 0" rpy="0 0 0" />
+			<parent link="${name}_fake_link1"/>
+			<child link="${name}_proximal_link"/>
+			<axis xyz="0 1 0" />
+			<mimic joint="${name}_fake_joint1" multiplier="1" />
+			<limit lower="${middle_lb *pi/180}" upper="${middle_ub *pi/180}" effort="${effort}" velocity="${velocity}"/>
+		</joint>
+		<link name="${name}_proximal_link">
+			<visual>
+				<origin xyz="0 0 0" rpy="0 0 0" />
+				<geometry>
+					<mesh filename="package://complete_soft_hand/meshes/phalanx_short_injection.stl" scale=" .001 .001 .001" />
+				</geometry>
+				<material name="DarkGolden" />
+			</visual>
+		</link>
+		<!-- LITTLE PHALANGE -->
+		<!-- immaginary link-->
+		<!-- joint and link FAKE 2-->
+		<joint name="${name}_fake_joint2" type="revolute">
+			<origin xyz="-0.009 0 0" rpy="0 0 0" />
+			<parent link="${name}_proximal_link"/>
+			<child link="${name}_fake_link2"/>
+			<axis xyz="0 1 0" />
+			<limit lower="${inner_lb *pi/180}" upper="${inner_ub *pi/180}" effort="${effort}" velocity="${velocity}"/>
+		</joint>
+		<link name="${name}_fake_link2">
+		</link>
+		<!-- end immaginary link-->
+		<joint name="${name}_middle_joint" type="revolute">
+			<origin xyz="-0.013 0 0" rpy="0 0 0" />
+			<parent link="${name}_fake_link2"/>
+			<child link="${name}_middle_link"/>
+			<axis xyz="0 1 0" />
+			<mimic joint="${name}_fake_joint2" multiplier="1" />
+			<limit lower="${outer_lb *pi/180}" upper="${outer_ub *pi/180}" effort="${effort}" velocity="${velocity}"/>
+		</joint>
+		<link name="${name}_middle_link">
+			<visual>
+				<origin xyz="0 0 0" rpy="0 0 0" />
+				<geometry>
+					<mesh filename="package://complete_soft_hand/meshes/phalanx_short_injection.stl" scale=" .001 .001 .001" />
+				</geometry>
+				<material name="DarkGolden" />
+			</visual>
+		</link>
+		<!-- BABY PHALANGE -->
+		<!-- immaginary link-->
+		<!-- joint and link FAKE 3-->
+		<joint name="${name}_fake_joint3" type="revolute">
+			<origin xyz="-0.009 0 0.0" rpy="0 0 0" />
+			<parent link="${name}_middle_link"/>
+			<child link="${name}_fake_link3"/>
+			<axis xyz="0 1 0" />
+			<limit lower="${inner_lb *pi/180}" upper="${inner_ub *pi/180}" effort="${effort}" velocity="${velocity}"/>
+		</joint>
+		<link name="${name}_fake_link3">
+		</link>
+		<!-- end immaginary link-->
+		<joint name="${name}_outer_joint" type="revolute">
+			<origin xyz="-0.013 0 0" rpy="0 0 0" />
+			<parent link="${name}_fake_link3"/>
+			<child link="${name}_distal_link"/>
+			<axis xyz="0 1 0" />
+			<mimic joint="${name}_fake_joint3" multiplier="1" />
+			<limit lower="${inner_lb *pi/180}" upper="${inner_ub *pi/180}" effort="${effort}" velocity="${velocity}"/>
+		</joint>
+		<link name="${name}_distal_link">
+			<visual>
+				<origin xyz="0 0 0" rpy="0 0 0" />
+				<geometry>
+					<mesh filename="package://complete_soft_hand/meshes/phalanx_distal_out_no_ati.stl" scale=" .001 .001 .001" />
+				</geometry>
+				<material name="DarkGolden" />
 			</visual>
 		</link>
@@ -131,6 +243,6 @@
 			<parent link="${parent}" />
 			<child link="${name}_palm_link" />
-			<axis xyz="0 1 0" />
-			<limit lower="${-90*pi/180}" upper="${90*pi/180}" effort="${effort}" velocity="${velocity}"/>
+			<!-- <axis xyz="0 1 0" /> -->
+			<!-- <limit lower="${-90*pi/180}" upper="${90*pi/180}" effort="${effort}" velocity="${velocity}"/> -->
 		</joint>
 		<link name="${name}_palm_link">
@@ -138,5 +250,5 @@
 				<origin xyz="0 0 0" rpy="0 0 0" />
 				<geometry>
-					<mesh filename="package://complete_soft_hand/meshes/palmo.stl" scale=" .001 .001 .001" />
+					<mesh filename="package://complete_soft_hand/meshes/palm_hand.stl" scale=" .001 .001 .001" />
 				</geometry>
 				<material name="LightGrey" />
@@ -144,6 +256,9 @@
 		</link>
 		<!-- macro for each finger -->
-		<xacro:soft_finger parent="${name}_palm_link" name="${name}_thumb" position="-0.0245 0.024 0.039" orientation="0 ${50*pi/180} 0" />
-		<xacro:soft_finger parent="${name}_palm_link" name="${name}_index" position="0.0275 0.024 0.039" orientation="0 ${45*pi/180} ${pi}" />
+		<xacro:soft_finger parent="${name}_palm_link" name="${name}_index" position="-0.0285 0.0943918 0.00205" orientation="${180*pi/180} 0 ${-90*pi/180}" />
+		<xacro:soft_finger parent="${name}_palm_link" name="${name}_middle" position="-0.009 0.107892 0.00205" orientation="${180*pi/180} 0 ${-90*pi/180}" />
+		<xacro:soft_finger parent="${name}_palm_link" name="${name}_ring" position="0.0105 0.0943918 0.00205" orientation="${180*pi/180} 0 ${-90*pi/180}" />
+		<xacro:soft_finger parent="${name}_palm_link" name="${name}_little" position="0.030 0.0808918 0.00205" orientation="${180*pi/180} 0 ${-90*pi/180}" />
+		<xacro:thumb_finger parent="${name}_palm_link" name="${name}_thumb" position="-0.0418769 0.0538740 -0.00691972	" orientation="0 0 -0.43633181" />
 	</xacro:macro>
 </robot>

File: robot/hand_in_world.urdf.xacro (robot description, xacro)
@@ -3,10 +3,10 @@
   <xacro:include filename="$(find complete_soft_hand)/model/complete_soft_hand.urdf.xacro"/>
   <link name="world">
-    <visual>
+<!--     <visual>
       <origin xyz="0 0 0" rpy="0 0 0"/>
       <geometry>
         <box size="1 1 1.0"/>
       </geometry>
-    </visual>
+    </visual> -->
   </link>
   <xacro:complete_soft_hand parent="world" name="hand">

Commit message: updateing hand model

File: model/complete_soft_hand.urdf.xacro (robot description, xacro)
@@ -3,4 +3,6 @@
 	<xacro:include filename="$(find complete_soft_hand)/model/materials.urdf.xacro"/>
 	<xacro:property name="pi" value="3.1415926535897931" />
+	<xacro:property name="abd_lb" value="-30" />
+	<xacro:property name="abd_ub" value="30" />
 	<xacro:property name="inner_lb" value="0" />
 	<xacro:property name="inner_ub" value="45" />
@@ -12,8 +14,9 @@
 	<xacro:property name="effort" value="100" />
 	<!-- Declaration of single finger that we can replicate in another position -->
-	<!-- We suppose that all fingers are equal -->
+	<!-- We suppose that 4th fingers are equal (index, middle, ring, little) -->
 	<xacro:macro name="soft_finger" params="parent name position orientation">
 		<!-- macro for one finger -->
 		<!-- abductor joint between palm_link and finger_abd_link - fake between palm and proximal -->
+		<!-- KNUCKLE -->
 		<joint name="${name}_abd_joint" type="revolute">
 			<origin xyz="${position}" rpy="${orientation}" />
@@ -21,5 +24,5 @@
 			<child link="${name}_knuckle_link"/>
 			<axis xyz="0 0 1" />
-			<limit lower="${inner_lb *pi/180}" upper="${inner_ub *pi/180}" effort="${effort}" velocity="${velocity}"/>
+			<limit lower="${abd_lb *pi/180}" upper="${abd_ub *pi/180}" effort="${effort}" velocity="${velocity}"/>
 		</joint>
 		<link name="${name}_knuckle_link">
@@ -32,4 +35,5 @@
 			</visual>
 		</link>
+		<!-- end KNUCKLE -->
 		<!-- PHALANGE -->
 		<!-- immaginary link-->
@@ -63,4 +67,5 @@
 			</visual>
 		</link>
+		<!-- end PHALANGE -->
 		<!-- LITTLE PHALANGE -->
 		<!-- immaginary link-->
@@ -93,4 +98,5 @@
 			</visual>
 		</link>
+		<!-- end LITTLE PHALANGE -->
 		<!-- BABY PHALANGE -->
 		<!-- immaginary link-->
@@ -125,7 +131,10 @@
 		<!-- end BABY PHALANGE -->
 	</xacro:macro>
+	<!-- end FINGER model -->
+	<!-- THUMB model -->
 	<xacro:macro name="thumb_finger" params="parent name position orientation">
 		<!-- macro for one finger -->
-		<!-- abductor joint between palm_link and finger_abd_link - fake between palm and proximal -->
+		<!-- abductor joint between palm_link and thumb_abd_link - fake between palm and proximal -->
+		<!-- THUMB KNUCKLE -->
 		<joint name="${name}_abd_joint" type="revolute">
 			<origin xyz="${position}" rpy="${orientation}" />
@@ -144,5 +153,6 @@
 			</visual>
 		</link>
-		<!-- PHALANGE -->
+		<!-- end KNUCKLE -->
+		<!-- THUMB PHALANGE -->
 		<!-- immaginary link-->
 		<!-- joint and link FAKE 1-->
@@ -175,5 +185,6 @@
 			</visual>
 		</link>
-		<!-- LITTLE PHALANGE -->
+		<!-- end PHALANGE -->
+		<!-- THUMB LITTLE PHALANGE -->
 		<!-- immaginary link-->
 		<!-- joint and link FAKE 2-->
@@ -205,5 +216,5 @@
 			</visual>
 		</link>
-		<!-- BABY PHALANGE -->
+		<!-- THUMB BABY PHALANGE -->
 		<!-- immaginary link-->
 		<!-- joint and link FAKE 3-->
@@ -237,6 +248,8 @@
 		<!-- end BABY PHALANGE -->
 	</xacro:macro>
+	<!-- end THUMB model -->
 	<xacro:macro name="complete_soft_hand" params="parent name *origin">
 		<!-- macro for the hand -->
+		<!-- PALM -->
 		<joint name="${name}_palm_joint" type="fixed" >
 			<origin xyz="0 0 0" rpy="0 0 0" />
@@ -255,10 +268,11 @@
 			</visual>
 		</link>
+		<!-- end PALM -->
 		<!-- macro for each finger -->
-		<xacro:soft_finger parent="${name}_palm_link" name="${name}_index" position="-0.0285 0.0943918 0.00205" orientation="${180*pi/180} 0 ${-90*pi/180}" />
+		<xacro:thumb_finger parent="${name}_palm_link" name="${name}_thumb" position="-0.0418769 0.0538740 -0.00691972	" orientation="0 0 -0.43633181" />
+		<xacro:soft_finger parent="${name}_palm_link" name="${name}_index" position="-0.0285 0.0943918 0.00205" orientation="${180*pi/180} 0 ${(-90+20)*pi/180}" />
 		<xacro:soft_finger parent="${name}_palm_link" name="${name}_middle" position="-0.009 0.107892 0.00205" orientation="${180*pi/180} 0 ${-90*pi/180}" />
-		<xacro:soft_finger parent="${name}_palm_link" name="${name}_ring" position="0.0105 0.0943918 0.00205" orientation="${180*pi/180} 0 ${-90*pi/180}" />
-		<xacro:soft_finger parent="${name}_palm_link" name="${name}_little" position="0.030 0.0808918 0.00205" orientation="${180*pi/180} 0 ${-90*pi/180}" />
-		<xacro:thumb_finger parent="${name}_palm_link" name="${name}_thumb" position="-0.0418769 0.0538740 -0.00691972	" orientation="0 0 -0.43633181" />
+		<xacro:soft_finger parent="${name}_palm_link" name="${name}_ring" position="0.0105 0.0943918 0.00205" orientation="${180*pi/180} 0 ${(-90-10)*pi/180}" />
+		<xacro:soft_finger parent="${name}_palm_link" name="${name}_little" position="0.030 0.0808918 0.00205" orientation="${180*pi/180} 0 ${(-90-20)*pi/180}" />
 	</xacro:macro>
 </robot>

Commit message: rename fingers joint

File: model/complete_soft_hand.urdf.xacro (robot description, xacro)
@@ -24,5 +24,5 @@
 			<child link="${name}_knuckle_link"/>
 			<axis xyz="0 0 1" />
-			<limit lower="${abd_lb *pi/180}" upper="${abd_ub *pi/180}" effort="${effort}" velocity="${velocity}"/>
+			<limit lower="${abd_lb *pi/180}" upper="${inner_ub *pi/180}" effort="${effort}" velocity="${velocity}"/>
 		</joint>
 		<link name="${name}_knuckle_link">
@@ -39,12 +39,15 @@
 		<!-- immaginary link-->
 		<!-- joint and link FAKE 1-->
-		<joint name="${name}_fake_joint1" type="revolute">
+		<joint name="${name}_inner_joint
+" type="revolute">
 			<origin xyz="-0.009 0 0" rpy="0 0 0" />
 			<parent link="${name}_knuckle_link"/>
-			<child link="${name}_fake_link1"/>
-			<axis xyz="0 1 0" />
-			<limit lower="${inner_lb *pi/180}" upper="${inner_ub *pi/180}" effort="${effort}" velocity="${velocity}"/>
-		</joint>
-		<link name="${name}_fake_link1">
+			<child link="${name}_inner_link
+"/>
+			<axis xyz="0 1 0" />
+			<limit lower="${inner_lb *pi/180}" upper="${inner_ub *pi/180}" effort="${effort}" velocity="${velocity}"/>
+		</joint>
+		<link name="${name}_inner_link
+">
 		</link>
 		<!-- end immaginary link-->
@@ -52,8 +55,10 @@
 		<joint name="${name}_inner_joint" type="revolute">
 			<origin xyz="-0.013 0 0" rpy="0 0 0" />
-			<parent link="${name}_fake_link1"/>
+			<parent link="${name}_inner_link
+"/>
 			<child link="${name}_proximal_link"/>
 			<axis xyz="0 1 0" />
-			<mimic joint="${name}_fake_joint1" multiplier="1" />
+			<mimic joint="${name}_inner_joint
+" multiplier="1" />
 			<limit lower="${middle_lb *pi/180}" upper="${middle_ub *pi/180}" effort="${effort}" velocity="${velocity}"/>
 		</joint>
@@ -71,5 +76,6 @@
 		<!-- immaginary link-->
 		<!-- joint and link FAKE 2-->
-		<joint name="${name}_fake_joint2" type="revolute">
+		<joint name="${name}_middle_joint
+" type="revolute">
 			<origin xyz="-0.009 0 0" rpy="0 0 0" />
 			<parent link="${name}_proximal_link"/>
@@ -86,5 +92,6 @@
 			<child link="${name}_middle_link"/>
 			<axis xyz="0 1 0" />
-			<mimic joint="${name}_fake_joint2" multiplier="1" />
+			<mimic joint="${name}_middle_joint
+" multiplier="1" />
 			<limit lower="${outer_lb *pi/180}" upper="${outer_ub *pi/180}" effort="${effort}" velocity="${velocity}"/>
 		</joint>
@@ -102,5 +109,6 @@
 		<!-- immaginary link-->
 		<!-- joint and link FAKE 3-->
-		<joint name="${name}_fake_joint3" type="revolute">
+		<joint name="${name}_outer_joint
+" type="revolute">
 			<origin xyz="-0.009 0 0" rpy="0 0 0" />
 			<parent link="${name}_middle_link"/>
@@ -117,5 +125,6 @@
 			<child link="${name}_distal_link"/>
 			<axis xyz="0 1 0" />
-			<mimic joint="${name}_fake_joint3" multiplier="1" />
+			<mimic joint="${name}_outer_joint
+" multiplier="1" />
 			<limit lower="${inner_lb *pi/180}" upper="${inner_ub *pi/180}" effort="${effort}" velocity="${velocity}"/>
 		</joint>
@@ -157,12 +166,15 @@
 		<!-- immaginary link-->
 		<!-- joint and link FAKE 1-->
-		<joint name="${name}_fake_joint1" type="revolute">
+		<joint name="${name}_inner_joint
+" type="revolute">
 			<origin xyz="-0.0225 0 -0.0033" rpy="-1.9974238811 0 0" />
 			<parent link="${name}_knuckle_link"/>
-			<child link="${name}_fake_link1"/>
-			<axis xyz="0 1 0" />
-			<limit lower="${inner_lb *pi/180}" upper="${inner_ub *pi/180}" effort="${effort}" velocity="${velocity}"/>
-		</joint>
-		<link name="${name}_fake_link1">
+			<child link="${name}_inner_link
+"/>
+			<axis xyz="0 1 0" />
+			<limit lower="${inner_lb *pi/180}" upper="${inner_ub *pi/180}" effort="${effort}" velocity="${velocity}"/>
+		</joint>
+		<link name="${name}_inner_link
+">
 		</link>
 		<!-- end immaginary link-->
@@ -170,8 +182,10 @@
 		<joint name="${name}_inner_joint" type="revolute">
 			<origin xyz="-0.013 0 0" rpy="0 0 0" />
-			<parent link="${name}_fake_link1"/>
+			<parent link="${name}_inner_link
+"/>
 			<child link="${name}_proximal_link"/>
 			<axis xyz="0 1 0" />
-			<mimic joint="${name}_fake_joint1" multiplier="1" />
+			<mimic joint="${name}_inner_joint
+" multiplier="1" />
 			<limit lower="${middle_lb *pi/180}" upper="${middle_ub *pi/180}" effort="${effort}" velocity="${velocity}"/>
 		</joint>
@@ -189,5 +203,6 @@
 		<!-- immaginary link-->
 		<!-- joint and link FAKE 2-->
-		<joint name="${name}_fake_joint2" type="revolute">
+		<joint name="${name}_middle_joint
+" type="revolute">
 			<origin xyz="-0.009 0 0" rpy="0 0 0" />
 			<parent link="${name}_proximal_link"/>
@@ -204,5 +219,6 @@
 			<child link="${name}_middle_link"/>
 			<axis xyz="0 1 0" />
-			<mimic joint="${name}_fake_joint2" multiplier="1" />
+			<mimic joint="${name}_middle_joint
+" multiplier="1" />
 			<limit lower="${outer_lb *pi/180}" upper="${outer_ub *pi/180}" effort="${effort}" velocity="${velocity}"/>
 		</joint>
@@ -219,5 +235,6 @@
 		<!-- immaginary link-->
 		<!-- joint and link FAKE 3-->
-		<joint name="${name}_fake_joint3" type="revolute">
+		<joint name="${name}_outer_joint
+" type="revolute">
 			<origin xyz="-0.009 0 0.0" rpy="0 0 0" />
 			<parent link="${name}_middle_link"/>
@@ -234,5 +251,6 @@
 			<child link="${name}_distal_link"/>
 			<axis xyz="0 1 0" />
-			<mimic joint="${name}_fake_joint3" multiplier="1" />
+			<mimic joint="${name}_outer_joint
+" multiplier="1" />
 			<limit lower="${inner_lb *pi/180}" upper="${inner_ub *pi/180}" effort="${effort}" velocity="${velocity}"/>
 		</joint>
