Commit message: new structure and renames of macros

File: soft_hand/soft_hand_description/model/materials.urdf.xacro (robot description, xacro)
@@ -1,20 +1,20 @@
 <?xml version="1.0"?>
 <robot>
-	<material name="LightGrey">
+	<material name="SoftHand/LightGrey">
 		<color rgba="0.7 0.7 0.7 1.0"/>
 	</material>
-	<material name="DarkGrey">
+	<material name="SoftHand/DarkGrey">
 		<color rgba="0.4 0.4 0.4 1.0"/>
 	</material>
-	<material name="Black">
+	<material name="SoftHand/Black">
 		<color rgba="0.0 0.0 0.0 1.0"/>
 	</material>
-	<material name="DarkGolden">
+	<material name="SoftHand/DarkGolden">
 		<color rgba="0.4 0.4 0.3 1.0"/>
 	</material>
-	<material name="Blue">
+	<material name="SoftHand/Blue">
 		<color rgba="0.0 0.0 0.8 0.9"/>
 	</material>
-	<material name="LightBlue">
+	<material name="SoftHand/LightBlue">
 		<color rgba="0.0 0.4 1.0 0.5"/>
 	</material>

File: soft_hand/soft_hand_description/model/soft_hand.urdf.xacro (robot description, xacro)
@@ -1,5 +1,5 @@
 <?xml version="1.0"?>
 <robot xmlns:xacro="http://ros.org/wiki/xacro">
-	<xacro:include filename="$(find complete_soft_hand)/model/materials.urdf.xacro"/>
+	<xacro:include filename="$(find soft_hand_description)/model/materials.urdf.xacro"/>
 	<xacro:property name="pi" value="3.1415926535897931" />
 	<xacro:property name="abd_lb" value="-30" />
@@ -30,7 +30,7 @@
 				<origin xyz="0 0 0" rpy="0 0 0" />
 				<geometry>
-					<mesh filename="package://complete_soft_hand/meshes/phalanx_prossimal_injection.stl" scale=" .001 .001 .001" />
-				</geometry>
-				<material name="DarkGolden" />
+					<mesh filename="package://soft_hand_description/meshes/phalanx_prossimal_injection.stl" scale=" .001 .001 .001" />
+				</geometry>
+				<material name="SoftHand/DarkGolden" />
 			</visual>
 		</link>
@@ -39,26 +39,21 @@
 		<!-- immaginary link-->
 		<!-- joint and link FAKE 1-->
-		<joint name="${name}_inner_joint
-" type="revolute">
+		<joint name="${name}_inner_joint" type="revolute">
 			<origin xyz="-0.009 0 0" rpy="0 0 0" />
 			<parent link="${name}_knuckle_link"/>
-			<child link="${name}_inner_link
-"/>
-			<axis xyz="0 1 0" />
-			<limit lower="${inner_lb *pi/180}" upper="${inner_ub *pi/180}" effort="${effort}" velocity="${velocity}"/>
-		</joint>
-		<link name="${name}_inner_link
-">
+			<child link="${name}_inner_link"/>
+			<axis xyz="0 1 0" />
+			<limit lower="${inner_lb *pi/180}" upper="${inner_ub *pi/180}" effort="${effort}" velocity="${velocity}"/>
+		</joint>
+		<link name="${name}_inner_link">
 		</link>
 		<!-- end immaginary link-->
 		<!-- abductor joint between palm_link and finger_abd_link - fake between palm and proximal -->
-		<joint name="${name}_inner_joint" type="revolute">
-			<origin xyz="-0.013 0 0" rpy="0 0 0" />
-			<parent link="${name}_inner_link
-"/>
+		<joint name="${name}_inner_joint_mimic" type="revolute">
+			<origin xyz="-0.013 0 0" rpy="0 0 0" />
+			<parent link="${name}_inner_link"/>
 			<child link="${name}_proximal_link"/>
 			<axis xyz="0 1 0" />
-			<mimic joint="${name}_inner_joint
-" multiplier="1" />
+			<mimic joint="${name}_inner_joint" multiplier="1" />
 			<limit lower="${middle_lb *pi/180}" upper="${middle_ub *pi/180}" effort="${effort}" velocity="${velocity}"/>
 		</joint>
@@ -67,7 +62,7 @@
 				<origin xyz="0 0 0" rpy="0 0 0" />
 				<geometry>
-					<mesh filename="package://complete_soft_hand/meshes/phalanx_short_injection.stl" scale=" .001 .001 .001" />
-				</geometry>
-				<material name="DarkGolden" />
+					<mesh filename="package://soft_hand_description/meshes/phalanx_short_injection.stl" scale=" .001 .001 .001" />
+				</geometry>
+				<material name="SoftHand/DarkGolden" />
 			</visual>
 		</link>
@@ -76,6 +71,5 @@
 		<!-- immaginary link-->
 		<!-- joint and link FAKE 2-->
-		<joint name="${name}_middle_joint
-" type="revolute">
+		<joint name="${name}_middle_joint" type="revolute">
 			<origin xyz="-0.009 0 0" rpy="0 0 0" />
 			<parent link="${name}_proximal_link"/>
@@ -87,11 +81,10 @@
 		</link>
 		<!-- end immaginary link-->
-		<joint name="${name}_middle_joint" type="revolute">
+		<joint name="${name}_middle_joint_mimic" type="revolute">
 			<origin xyz="-0.013 0 0" rpy="0 0 0" />
 			<parent link="${name}_fake_link2"/>
 			<child link="${name}_middle_link"/>
 			<axis xyz="0 1 0" />
-			<mimic joint="${name}_middle_joint
-" multiplier="1" />
+			<mimic joint="${name}_middle_joint" multiplier="1" />
 			<limit lower="${outer_lb *pi/180}" upper="${outer_ub *pi/180}" effort="${effort}" velocity="${velocity}"/>
 		</joint>
@@ -100,7 +93,7 @@
 				<origin xyz="0 0 0" rpy="0 0 0" />
 				<geometry>
-					<mesh filename="package://complete_soft_hand/meshes/phalanx_short_injection.stl" scale=" .001 .001 .001" />
-				</geometry>
-				<material name="DarkGolden" />
+					<mesh filename="package://soft_hand_description/meshes/phalanx_short_injection.stl" scale=" .001 .001 .001" />
+				</geometry>
+				<material name="SoftHand/DarkGolden" />
 			</visual>
 		</link>
@@ -109,6 +102,5 @@
 		<!-- immaginary link-->
 		<!-- joint and link FAKE 3-->
-		<joint name="${name}_outer_joint
-" type="revolute">
+		<joint name="${name}_outer_joint" type="revolute">
 			<origin xyz="-0.009 0 0" rpy="0 0 0" />
 			<parent link="${name}_middle_link"/>
@@ -120,11 +112,10 @@
 		</link>
 		<!-- end immaginary link-->
-		<joint name="${name}_outer_joint" type="revolute">
+		<joint name="${name}_outer_joint_mimic" type="revolute">
 			<origin xyz="-0.013 0 0" rpy="0 0 0" />
 			<parent link="${name}_fake_link3"/>
 			<child link="${name}_distal_link"/>
 			<axis xyz="0 1 0" />
-			<mimic joint="${name}_outer_joint
-" multiplier="1" />
+			<mimic joint="${name}_outer_joint" multiplier="1" />
 			<limit lower="${inner_lb *pi/180}" upper="${inner_ub *pi/180}" effort="${effort}" velocity="${velocity}"/>
 		</joint>
@@ -133,7 +124,7 @@
 				<origin xyz="0 0 0" rpy="0 0 0" />
 				<geometry>
-					<mesh filename="package://complete_soft_hand/meshes/phalanx_distal_out_no_ati.stl" scale=" .001 .001 .001" />
-				</geometry>
-				<material name="DarkGolden" />
+					<mesh filename="package://soft_hand_description/meshes/phalanx_distal_out_no_ati.stl" scale=" .001 .001 .001" />
+				</geometry>
+				<material name="SoftHand/DarkGolden" />
 			</visual>
 		</link>
@@ -142,5 +133,5 @@
 	<!-- end FINGER model -->
 	<!-- THUMB model -->
-	<xacro:macro name="thumb_finger" params="parent name position orientation">
+	<xacro:macro name="soft_thumb" params="parent name position orientation">
 		<!-- macro for one finger -->
 		<!-- abductor joint between palm_link and thumb_abd_link - fake between palm and proximal -->
@@ -157,7 +148,7 @@
 				<origin xyz="0 0 0" rpy="0 0 0" />
 				<geometry>
-					<mesh filename="package://complete_soft_hand/meshes/phalanx_thumb_injection.stl" scale=" .001 .001 .001" />
-				</geometry>
-				<material name="DarkGolden" />
+					<mesh filename="package://soft_hand_description/meshes/phalanx_thumb_injection.stl" scale=" .001 .001 .001" />
+				</geometry>
+				<material name="SoftHand/DarkGolden" />
 			</visual>
 		</link>
@@ -166,26 +157,21 @@
 		<!-- immaginary link-->
 		<!-- joint and link FAKE 1-->
-		<joint name="${name}_inner_joint
-" type="revolute">
+		<joint name="${name}_inner_joint" type="revolute">
 			<origin xyz="-0.0225 0 -0.0033" rpy="-1.9974238811 0 0" />
 			<parent link="${name}_knuckle_link"/>
-			<child link="${name}_inner_link
-"/>
-			<axis xyz="0 1 0" />
-			<limit lower="${inner_lb *pi/180}" upper="${inner_ub *pi/180}" effort="${effort}" velocity="${velocity}"/>
-		</joint>
-		<link name="${name}_inner_link
-">
+			<child link="${name}_inner_link"/>
+			<axis xyz="0 1 0" />
+			<limit lower="${inner_lb *pi/180}" upper="${inner_ub *pi/180}" effort="${effort}" velocity="${velocity}"/>
+		</joint>
+		<link name="${name}_inner_link">
 		</link>
 		<!-- end immaginary link-->
 		<!-- abductor joint between palm_link and finger_abd_link - fake between palm and proximal -->
-		<joint name="${name}_inner_joint" type="revolute">
-			<origin xyz="-0.013 0 0" rpy="0 0 0" />
-			<parent link="${name}_inner_link
-"/>
+		<joint name="${name}_inner_joint_mimic" type="revolute">
+			<origin xyz="-0.013 0 0" rpy="0 0 0" />
+			<parent link="${name}_inner_link"/>
 			<child link="${name}_proximal_link"/>
 			<axis xyz="0 1 0" />
-			<mimic joint="${name}_inner_joint
-" multiplier="1" />
+			<mimic joint="${name}_inner_joint" multiplier="1" />
 			<limit lower="${middle_lb *pi/180}" upper="${middle_ub *pi/180}" effort="${effort}" velocity="${velocity}"/>
 		</joint>
@@ -194,7 +180,7 @@
 				<origin xyz="0 0 0" rpy="0 0 0" />
 				<geometry>
-					<mesh filename="package://complete_soft_hand/meshes/phalanx_short_injection.stl" scale=" .001 .001 .001" />
-				</geometry>
-				<material name="DarkGolden" />
+					<mesh filename="package://soft_hand_description/meshes/phalanx_short_injection.stl" scale=" .001 .001 .001" />
+				</geometry>
+				<material name="SoftHand/DarkGolden" />
 			</visual>
 		</link>
@@ -203,6 +189,5 @@
 		<!-- immaginary link-->
 		<!-- joint and link FAKE 2-->
-		<joint name="${name}_middle_joint
-" type="revolute">
+		<joint name="${name}_middle_joint" type="revolute">
 			<origin xyz="-0.009 0 0" rpy="0 0 0" />
 			<parent link="${name}_proximal_link"/>
@@ -214,11 +199,10 @@
 		</link>
 		<!-- end immaginary link-->
-		<joint name="${name}_middle_joint" type="revolute">
+		<joint name="${name}_middle_joint_mimic" type="revolute">
 			<origin xyz="-0.013 0 0" rpy="0 0 0" />
 			<parent link="${name}_fake_link2"/>
 			<child link="${name}_middle_link"/>
 			<axis xyz="0 1 0" />
-			<mimic joint="${name}_middle_joint
-" multiplier="1" />
+			<mimic joint="${name}_middle_joint" multiplier="1" />
 			<limit lower="${outer_lb *pi/180}" upper="${outer_ub *pi/180}" effort="${effort}" velocity="${velocity}"/>
 		</joint>
@@ -227,7 +211,7 @@
 				<origin xyz="0 0 0" rpy="0 0 0" />
 				<geometry>
-					<mesh filename="package://complete_soft_hand/meshes/phalanx_short_injection.stl" scale=" .001 .001 .001" />
-				</geometry>
-				<material name="DarkGolden" />
+					<mesh filename="package://soft_hand_description/meshes/phalanx_short_injection.stl" scale=" .001 .001 .001" />
+				</geometry>
+				<material name="SoftHand/DarkGolden" />
 			</visual>
 		</link>
@@ -235,6 +219,5 @@
 		<!-- immaginary link-->
 		<!-- joint and link FAKE 3-->
-		<joint name="${name}_outer_joint
-" type="revolute">
+		<joint name="${name}_outer_joint" type="revolute">
 			<origin xyz="-0.009 0 0.0" rpy="0 0 0" />
 			<parent link="${name}_middle_link"/>
@@ -246,11 +229,10 @@
 		</link>
 		<!-- end immaginary link-->
-		<joint name="${name}_outer_joint" type="revolute">
+		<joint name="${name}_outer_joint_mimic" type="revolute">
 			<origin xyz="-0.013 0 0" rpy="0 0 0" />
 			<parent link="${name}_fake_link3"/>
 			<child link="${name}_distal_link"/>
 			<axis xyz="0 1 0" />
-			<mimic joint="${name}_outer_joint
-" multiplier="1" />
+			<mimic joint="${name}_outer_joint" multiplier="1" />
 			<limit lower="${inner_lb *pi/180}" upper="${inner_ub *pi/180}" effort="${effort}" velocity="${velocity}"/>
 		</joint>
@@ -259,7 +241,7 @@
 				<origin xyz="0 0 0" rpy="0 0 0" />
 				<geometry>
-					<mesh filename="package://complete_soft_hand/meshes/phalanx_distal_out_no_ati.stl" scale=" .001 .001 .001" />
-				</geometry>
-				<material name="DarkGolden" />
+					<mesh filename="package://soft_hand_description/meshes/phalanx_distal_out_no_ati.stl" scale=" .001 .001 .001" />
+				</geometry>
+				<material name="SoftHand/DarkGolden" />
 			</visual>
 		</link>
@@ -267,5 +249,5 @@
 	</xacro:macro>
 	<!-- end THUMB model -->
-	<xacro:macro name="complete_soft_hand" params="parent name *origin">
+	<xacro:macro name="soft_hand" params="parent name *origin">
 		<!-- macro for the hand -->
 		<!-- PALM -->
@@ -281,12 +263,12 @@
 				<origin xyz="0 0 0" rpy="0 0 0" />
 				<geometry>
-					<mesh filename="package://complete_soft_hand/meshes/palm_hand.stl" scale=" .001 .001 .001" />
-				</geometry>
-				<material name="LightGrey" />
+					<mesh filename="package://soft_hand_description/meshes/palm_hand.stl" scale=" .001 .001 .001" />
+				</geometry>
+				<material name="SoftHand/LightGrey" />
 			</visual>
 		</link>
 		<!-- end PALM -->
 		<!-- macro for each finger -->
-		<xacro:thumb_finger parent="${name}_palm_link" name="${name}_thumb" position="-0.0418769 0.0538740 -0.00691972	" orientation="0 0 -0.43633181" />
+		<xacro:soft_thumb parent="${name}_palm_link" name="${name}_thumb" position="-0.0418769 0.0538740 -0.00691972	" orientation="0 0 -0.43633181" />
 		<xacro:soft_finger parent="${name}_palm_link" name="${name}_index" position="-0.0285 0.0943918 0.00205" orientation="${180*pi/180} 0 ${(-90+20)*pi/180}" />
 		<xacro:soft_finger parent="${name}_palm_link" name="${name}_middle" position="-0.009 0.107892 0.00205" orientation="${180*pi/180} 0 ${-90*pi/180}" />
