Commit message: palm + coupler separated, right and left hand models, it required remeshing and now the gazebo simulation stopped working

File: soft_hand/soft_hand_description/robot/soft_hand_adaptive.urdf.xacro (robot description, xacro)
@@ -2,5 +2,5 @@
 <robot xmlns:xacro="http://www.ros.org/wiki/xacro" name="soft_hand">
 	<xacro:include filename="$(find soft_hand_description)/model/soft_hand.urdf.xacro"/>
-	<link name="wrist">
+	<link name="box">
 		<inertial>
 			<mass value="50.0"/>
@@ -20,31 +20,29 @@
 		</collision>
 	</link>
-	<!-- comment or uncomment depending if you want to simulate a fixed or a flying hand -->
-	<gazebo reference="wrist">
+	<gazebo reference="box">
 		<static>true</static>
 	</gazebo>
-	<xacro:soft_hand parent="wrist" name="soft_hand" withAdaptiveTransmission="true" useMimicTag="$(arg use_mimic_tag)">
-		<origin xyz="0 0 1" rpy="1.570796 0 0"/>
+	<xacro:soft_hand parent="box" name="soft_hand" withAdaptiveTransmission="true" useMimicTag="$(arg use_mimic_tag)" left="false">
+		<origin xyz="0.0 0.0 1.02" rpy="0 0 0"/>
 	</xacro:soft_hand>
-	<!-- a wall to test the adaptivity -->
-	<joint name="wrist_object_joint" type="fixed">
-		<origin xyz="0 0.06 1.15" rpy="0 0 0" />
-		<parent link="wrist"/>
+	<!-- a wall to test the adaptivity
+	<joint name="box_object_joint" type="fixed">
+		<origin xyz="0.06 0 1.15" rpy="0 0 0" />
+		<parent link="box"/>
 		<child link="object"/>
 	</joint>
 	<link name="object">
 		<inertial>
-			<insert_block name="negligible_inertia"/>
+			<mass value="50.0"/>
+			<inertia  ixx="1" ixy="0.00"  ixz="0.00" iyy="1" iyz="0.00" izz="1" />
 		</inertial>
 		<visual>
-			<origin xyz="0 0 0" rpy="0 0 0"/>
 			<geometry>
-				<box size="0.07 0.05 0.25"/>
+				<box size="0.05 0.07 0.25"/>
 			</geometry>
 		</visual>
 		<collision>
-			<origin xyz="0 0 0" rpy="0 0 0"/>
 			<geometry>
-				<box size="0.07 0.05 0.25"/>
+				<box size="0.05 0.07 0.25"/>
 			</geometry>
 		</collision>
@@ -53,3 +51,4 @@
 		<selfCollide>True</selfCollide>
 	</gazebo>
+	-->
 </robot>

File: soft_hand/soft_hand_description/robot/soft_hand_full_actuation.urdf.xacro (robot description, xacro)
@@ -2,5 +2,5 @@
 <robot xmlns:xacro="http://www.ros.org/wiki/xacro" name="soft_hand">
 	<xacro:include filename="$(find soft_hand_description)/model/soft_hand.urdf.xacro"/>
-	<link name="wrist">
+	<link name="box">
 		<inertial>
 			<mass value="50.0"/>
@@ -20,10 +20,56 @@
 		</collision>
 	</link>
-	<!-- comment or uncomment depending if you want to simulate a fixed or a flying hand -->
-	<gazebo reference="wrist">
+	<gazebo reference="box">
 		<static>true</static>
 	</gazebo>
-	<xacro:soft_hand parent="wrist" name="hand" withAdaptiveTransmission="false" useMimicTag="$(arg use_mimic_tag)">
-		<origin xyz="0 0 1" rpy="1.570796 0 0"/>
+	<joint name="box_wrist_joint" type="fixed">
+		<origin xyz="0 0 1.02" rpy="0 0 0" />
+		<parent link="box"/>
+		<child link="wrist"/>
+	</joint>
+	<link name="wrist">
+		<inertial>
+			<insert_block name="negligible_inertia"/>
+		</inertial>
+		<visual>
+			<geometry>
+				<mesh filename="package://soft_hand_description/meshes/coman_coupler.stl" scale=" .001 .001 .001" />
+			</geometry>
+			<material name="SoftHand/LightBlue" />
+		</visual>
+		<collision>
+			<geometry>
+				<mesh filename="package://soft_hand_description/meshes/coman_coupler.stl" scale=" .001 .001 .001" />
+			</geometry>
+		</collision>
+	</link>
+	<xacro:soft_hand parent="wrist" name="soft_hand" left="false" withAdaptiveTransmission="false" useMimicTag="$(arg use_mimic_tag)">
+		<origin xyz="0.002 0.009 0.038" rpy="0 0 0"/>
 	</xacro:soft_hand>
+	<!-- a wall to test the adaptivity
+	<joint name="box_object_joint" type="fixed">
+		<origin xyz="0.06 0 1.15" rpy="0 0 0" />
+		<parent link="box"/>
+		<child link="object"/>
+	</joint>
+	<link name="object">
+		<inertial>
+			<mass value="50.0"/>
+			<inertia  ixx="1" ixy="0.00"  ixz="0.00" iyy="1" iyz="0.00" izz="1" />
+		</inertial>
+		<visual>
+			<geometry>
+				<box size="0.05 0.07 0.25"/>
+			</geometry>
+		</visual>
+		<collision>
+			<geometry>
+				<box size="0.05 0.07 0.25"/>
+			</geometry>
+		</collision>
+	</link>
+	<gazebo reference="object">
+		<selfCollide>True</selfCollide>
+	</gazebo>
+	-->
 </robot>
