Commit message: added the synergistic joint, useful to tune the synergy vector only

File: soft_hand/soft_hand_description/model/soft_hand.urdf.xacro (robot description, xacro)
@@ -4,5 +4,5 @@
 	<xacro:include filename="$(find soft_hand_description)/model/soft_hand.transmission.xacro"/>
 	<xacro:include filename="$(find soft_hand_description)/model/soft_hand.gazebo.xacro"/>
-	<xacro:include filename="$(find soft_hand_description)/model/soft_hand.inertias.xacro"/>
+	<xacro:include filename="$(find soft_hand_description)/model/soft_hand.inertia.xacro"/>
 	<xacro:property name="pi" value="3.1415926535897931" />
 	<!-- joint properties -->
@@ -21,15 +21,35 @@
 	<xacro:property name="damping" value="0.0" />
 	<xacro:property name="friction" value="0.0" />
-	<!-- actuator properties -->
-	<xacro:property name="actuator_lb" value="0" />
-	<xacro:property name="actuator_ub" value="359" />
-	<xacro:property name="max_actuator_velocity" value="100" />
-	<xacro:property name="max_actuator_effort" value="100" />
-	<xacro:property name="actuator_damping" value="0.0" />
-	<xacro:property name="actuator_friction" value="0.0" />
+	<!-- synergy vector -->
+	<xacro:property name="thumb_abd_R" value="1.3" />
+	<xacro:property name="thumb_inner_R" value="1.3" />
+	<xacro:property name="thumb_outer_R" value="1.0" />
+	<xacro:property name="index_abd_R" value="-0.2" />
+	<xacro:property name="index_inner_R" value="1.0" />
+	<xacro:property name="index_middle_R" value="1.0" />
+	<xacro:property name="index_outer_R" value="1.0" />
+	<xacro:property name="middle_abd_R" value="0.0" />
+	<xacro:property name="middle_inner_R" value="1.0" />
+	<xacro:property name="middle_middle_R" value="1.0" />
+	<xacro:property name="middle_outer_R" value="1.0" />
+	<xacro:property name="ring_abd_R" value="0.2" />
+	<xacro:property name="ring_inner_R" value="1.0" />
+	<xacro:property name="ring_middle_R" value="1.0" />
+	<xacro:property name="ring_outer_R" value="1.0" />
+	<xacro:property name="little_abd_R" value="0.4" />
+	<xacro:property name="little_inner_R" value="1.0" />
+	<xacro:property name="little_middle_R" value="1.0" />
+	<xacro:property name="little_outer_R" value="1.0" />
+	<!-- synergy joint properties -->
+	<xacro:property name="synergy_lb" value="0.0" />
+	<xacro:property name="synergy_ub" value="1.0" />
+	<xacro:property name="max_synergy_velocity" value="100" />
+	<xacro:property name="max_synergy_effort" value="100" />
+	<xacro:property name="synergy_damping" value="0.0" />
+	<xacro:property name="synergy_friction" value="0.0" />
 	<!-- HAND MODEL v.? Material: ABS -->
 	<!-- SOFT FINGER model -->
 	<!-- 4 fingers are equal (index, middle, ring, little) -->
-	<xacro:macro name="soft_finger" params="parent name position orientation">
+	<xacro:macro name="soft_finger" params="parent name position orientation abd_R inner_R middle_R outer_R">
 		<!-- KNUCKLE -->
 		<joint name="${name}_abd_joint" type="revolute">
@@ -38,6 +58,7 @@
 			<child link="${name}_knuckle_link"/>
 			<axis xyz="0 0 1" />
-			<limit lower="${abd_lb *pi/180}" upper="${inner_ub *pi/180}" effort="${effort}" velocity="${velocity}"/>
-			<dynamics damping="${damping}" friction="${friction}"/>
+			<limit lower="${abd_lb *pi/180}" upper="${abd_ub *pi/180}" effort="${effort}" velocity="${velocity}"/>
+			<dynamics damping="${damping}" friction="${friction}"/>
+			<mimic joint="synergy_joint" multiplier="${abd_R}"/>
 		</joint>
 		<link name="${name}_knuckle_link">
@@ -68,4 +89,5 @@
 			<limit lower="${inner_lb *pi/180}" upper="${inner_ub *pi/180}" effort="${effort}" velocity="${velocity}"/>
 			<dynamics damping="${damping}" friction="${friction}"/>
+			<mimic joint="synergy_joint" multiplier="${inner_R}"/>
 		</joint>
 		<link name="${name}_fake_link1">
@@ -79,7 +101,7 @@
 			<child link="${name}_proximal_link"/>
 			<axis xyz="0 1 0" />
-			<mimic joint="${name}_inner_joint" multiplier="1" />
-			<limit lower="${middle_lb *pi/180}" upper="${middle_ub *pi/180}" effort="${effort}" velocity="${velocity}"/>
-			<dynamics damping="${damping}" friction="${friction}"/>
+			<limit lower="${inner_lb *pi/180}" upper="${inner_ub *pi/180}" effort="${effort}" velocity="${velocity}"/>
+			<dynamics damping="${damping}" friction="${friction}"/>
+			<mimic joint="synergy_joint" multiplier="${inner_R}" />
 		</joint>
 		<link name="${name}_proximal_link">
@@ -108,6 +130,7 @@
 			<child link="${name}_fake_link2"/>
 			<axis xyz="0 1 0" />
-			<limit lower="${inner_lb *pi/180}" upper="${inner_ub *pi/180}" effort="${effort}" velocity="${velocity}"/>
-			<dynamics damping="${damping}" friction="${friction}"/>
+			<limit lower="${middle_lb *pi/180}" upper="${middle_ub *pi/180}" effort="${effort}" velocity="${velocity}"/>
+			<dynamics damping="${damping}" friction="${friction}"/>
+			<mimic joint="synergy_joint" multiplier="${middle_R}"/>
 		</joint>
 		<link name="${name}_fake_link2">
@@ -121,7 +144,7 @@
 			<child link="${name}_middle_link"/>
 			<axis xyz="0 1 0" />
-			<mimic joint="${name}_middle_joint" multiplier="1" />
-			<limit lower="${outer_lb *pi/180}" upper="${outer_ub *pi/180}" effort="${effort}" velocity="${velocity}"/>
-			<dynamics damping="${damping}" friction="${friction}"/>
+			<limit lower="${middle_lb *pi/180}" upper="${middle_ub *pi/180}" effort="${effort}" velocity="${velocity}"/>
+			<dynamics damping="${damping}" friction="${friction}"/>
+			<mimic joint="synergy_joint" multiplier="${middle_R}"/>
 		</joint>
 		<link name="${name}_middle_link">
@@ -148,6 +171,7 @@
 			<child link="${name}_fake_link3"/>
 			<axis xyz="0 1 0" />
-			<limit lower="${inner_lb *pi/180}" upper="${inner_ub *pi/180}" effort="${effort}" velocity="${velocity}"/>
-			<dynamics damping="${damping}" friction="${friction}"/>
+			<limit lower="${outer_lb *pi/180}" upper="${outer_ub *pi/180}" effort="${effort}" velocity="${velocity}"/>
+			<dynamics damping="${damping}" friction="${friction}"/>
+			<mimic joint="synergy_joint" multiplier="${outer_R}"/>
 		</joint>
 		<link name="${name}_fake_link3">
@@ -161,7 +185,7 @@
 			<child link="${name}_distal_link"/>
 			<axis xyz="0 1 0" />
-			<mimic joint="${name}_outer_joint" multiplier="1" />
-			<limit lower="${inner_lb *pi/180}" upper="${inner_ub *pi/180}" effort="${effort}" velocity="${velocity}"/>
-			<dynamics damping="${damping}" friction="${friction}"/>
+			<limit lower="${outer_lb *pi/180}" upper="${outer_ub *pi/180}" effort="${effort}" velocity="${velocity}"/>
+			<dynamics damping="${damping}" friction="${friction}"/>
+			<mimic joint="synergy_joint" multiplier="${outer_R}"/>
 		</joint>
 		<link name="${name}_distal_link">
@@ -185,5 +209,5 @@
 	<!-- THUMB MODEL -->
 	<!-- It has one joint less than rest of fingers -->
-	<xacro:macro name="soft_thumb" params="parent name position orientation">
+	<xacro:macro name="soft_thumb" params="parent name position orientation abd_R inner_R outer_R">
 		<!-- KNUCKLE -->
 		<joint name="${name}_abd_joint" type="revolute">
@@ -194,4 +218,5 @@
 			<limit lower="${thumb_abd_lb *pi/180}" upper="${thumb_abd_ub *pi/180}" effort="${effort}" velocity="${velocity}"/>
 			<dynamics damping="${damping}" friction="${friction}"/>
+			<mimic joint="synergy_joint" multiplier="${abd_R}"/>
 		</joint>
 		<link name="${name}_knuckle_link">
@@ -220,4 +245,5 @@
 			<limit lower="${inner_lb *pi/180}" upper="${inner_ub *pi/180}" effort="${effort}" velocity="${velocity}"/>
 			<dynamics damping="${damping}" friction="${friction}"/>
+			<mimic joint="synergy_joint" multiplier="${inner_R}"/>
 		</joint>
 		<link name="${name}_fake_link1">
@@ -231,7 +257,7 @@
 			<child link="${name}_proximal_link"/>
 			<axis xyz="0 1 0" />
-			<mimic joint="${name}_inner_joint" multiplier="1" />
-			<limit lower="${middle_lb *pi/180}" upper="${middle_ub *pi/180}" effort="${effort}" velocity="${velocity}"/>
-			<dynamics damping="${damping}" friction="${friction}"/>
+			<limit lower="${inner_lb *pi/180}" upper="${inner_ub *pi/180}" effort="${effort}" velocity="${velocity}"/>
+			<dynamics damping="${damping}" friction="${friction}"/>
+			<mimic joint="synergy_joint" multiplier="${inner_R}" />
 		</joint>
 		<link name="${name}_proximal_link">
@@ -258,6 +284,7 @@
 			<child link="${name}_fake_link3"/>
 			<axis xyz="0 1 0" />
-			<limit lower="${inner_lb *pi/180}" upper="${inner_ub *pi/180}" effort="${effort}" velocity="${velocity}"/>
-			<dynamics damping="${damping}" friction="${friction}"/>
+			<limit lower="${outer_lb *pi/180}" upper="${outer_ub *pi/180}" effort="${effort}" velocity="${velocity}"/>
+			<dynamics damping="${damping}" friction="${friction}"/>
+			<mimic joint="synergy_joint" multiplier="${outer_R}"/>
 		</joint>
 		<link name="${name}_fake_link3">
@@ -271,7 +298,7 @@
 			<child link="${name}_distal_link"/>
 			<axis xyz="0 1 0" />
-			<mimic joint="${name}_outer_joint" multiplier="1" />
-			<limit lower="${inner_lb *pi/180}" upper="${inner_ub *pi/180}" effort="${effort}" velocity="${velocity}"/>
-			<dynamics damping="${damping}" friction="${friction}"/>
+			<limit lower="${outer_lb *pi/180}" upper="${outer_ub *pi/180}" effort="${effort}" velocity="${velocity}"/>
+			<dynamics damping="${damping}" friction="${friction}"/>
+			<mimic joint="synergy_joint" multiplier="${outer_R}" />
 		</joint>
 		<link name="${name}_distal_link">
@@ -294,16 +321,14 @@
 	</xacro:macro>
 	<!-- SOFT HAND MODEL -->
-	<xacro:macro name="soft_hand" params="parent name *origin">
+	<xacro:macro name="soft_hand" params="parent name withAdaptiveTransmission *origin">
 		<!-- MOTOR JOINT -->
-		<!--
-		<joint name="${name}a_actuator" type="revolute" >
+		<joint name="synergy_joint" type="revolute" >
 			<parent link="${parent}" />
-			<child link="${name}_invisible_wire_link"/>
+			<child link="invisible_wire_link"/>
 			<axis xyz="0 0 1" />
-			<limit lower="${actuator_lb *pi/180}" upper="${actuator_ub *pi/180}" effort="${actuator_max_effort}" velocity="${actuator_max_velocity}"/>
-			<dynamics damping="${actuator_damping}" friction="${actuator_friction}"/>
-		</joint>
-		<link name="${name}_invisible_wire_link"/>
-		-->
+			<limit lower="${synergy_lb}" upper="${synergy_ub}" effort="${max_synergy_effort}" velocity="${max_synergy_velocity}"/>
+			<dynamics damping="${synergy_damping}" friction="${synergy_friction}"/>
+		</joint>
+		<link name="invisible_wire_link"/>
 		<!-- PALM -->
 		<joint name="${name}_palm_joint" type="fixed" >
@@ -329,12 +354,12 @@
 			</collision>
 		</link>
-		<!-- FINGERS AND THUMB -->
-		<xacro:soft_thumb parent="${name}_palm_link" name="${name}_thumb" position="-0.0418769 0.0538740 -0.00691972" orientation="0 0 -0.43633181" />
-		<xacro:soft_finger parent="${name}_palm_link" name="${name}_index" position="-0.0285 0.0943918 0.00205" orientation="${180*pi/180} 0 ${(-90+20)*pi/180}" />
-		<xacro:soft_finger parent="${name}_palm_link" name="${name}_middle" position="-0.009 0.107892 0.00205" orientation="${180*pi/180} 0 ${-90*pi/180}" />
-		<xacro:soft_finger parent="${name}_palm_link" name="${name}_ring" position="0.0105 0.0943918 0.00205" orientation="${180*pi/180} 0 ${(-90-10)*pi/180}" />
-		<xacro:soft_finger parent="${name}_palm_link" name="${name}_little" position="0.030 0.0808918 0.00205" orientation="${180*pi/180} 0 ${(-90-20)*pi/180}" />
-		<xacro:soft_hand_transmission name="${name}"/>
-		<xacro:soft_hand_gazebo name="${name}"/>
+		<!-- THUMB AND FINGERS -->
+		<xacro:soft_thumb parent="${name}_palm_link" name="${name}_thumb" position="-0.0418769 0.0538740 -0.00691972" orientation="0 0 -0.43633181" abd_R="${thumb_abd_R *(thumb_abd_ub - thumb_abd_lb)*pi/180}" inner_R="${thumb_inner_R *(inner_ub - inner_lb)*pi/180}" outer_R="${thumb_outer_R *(outer_ub - outer_lb)*pi/180}"/>
+		<xacro:soft_finger parent="${name}_palm_link" name="${name}_index" position="-0.0285 0.0943918 0.00205" orientation="${180*pi/180} 0 ${(-90+20)*pi/180}" abd_R="${index_abd_R}" inner_R="${index_inner_R *(inner_ub - inner_lb)*pi/180}" middle_R="${index_middle_R *(middle_ub - middle_lb)*pi/180}" outer_R="${index_outer_R *(outer_ub - outer_lb)*pi/180}" />
+		<xacro:soft_finger parent="${name}_palm_link" name="${name}_middle" position="-0.009 0.107892 0.00205" orientation="${180*pi/180} 0 ${-90*pi/180}" abd_R="${middle_abd_R}" inner_R="${middle_inner_R *(inner_ub - inner_lb)*pi/180}" middle_R="${middle_middle_R *(middle_ub - middle_lb)*pi/180}" outer_R="${middle_outer_R *(outer_ub - outer_lb)*pi/180}" />
+		<xacro:soft_finger parent="${name}_palm_link" name="${name}_ring" position="0.0105 0.0943918 0.00205" orientation="${180*pi/180} 0 ${(-90-10)*pi/180}" abd_R="${ring_abd_R}" inner_R="${ring_inner_R *(inner_ub - inner_lb)*pi/180}" middle_R="${ring_middle_R *(middle_ub - middle_lb)*pi/180}" outer_R="${ring_outer_R *(outer_ub - outer_lb)*pi/180}" />
+		<xacro:soft_finger parent="${name}_palm_link" name="${name}_little" position="0.030 0.0808918 0.00205" orientation="${180*pi/180} 0 ${(-90-20)*pi/180}" abd_R="${little_abd_R}" inner_R="${little_inner_R *(inner_ub - inner_lb)*pi/180}" middle_R="${little_middle_R *(middle_ub - middle_lb)*pi/180}" outer_R="${little_outer_R *(outer_ub - outer_lb)*pi/180}" />
+		<xacro:soft_hand_transmission name="${name}" withAdaptiveTransmission="${withAdaptiveTransmission}"/>
+		<xacro:soft_hand_gazebo name="${name}" withAdaptiveTransmission="${withAdaptiveTransmission}"/>
 	</xacro:macro>
 </robot>

File: soft_hand/soft_hand_description/robot/soft_hand_full_actuation.urdf.xacro (robot description, xacro)
@@ -24,5 +24,5 @@
 		<static>true</static>
 	</gazebo>
-	<xacro:soft_hand parent="wrist" name="hand">
+	<xacro:soft_hand parent="wrist" name="hand" withAdaptiveTransmission="false">
 		<origin xyz="0 0 1" rpy="1.570796 0 0"/>
 	</xacro:soft_hand>
