Commit message: update, control over the synergy joint and move the rest with pure kinematics

File: soft_hand/soft_hand_description/model/soft_hand.gazebo.xacro (robot description, xacro)
@@ -38,11 +38,12 @@
 		<!-- PLUGINS -->
 		<xacro:if value="${withAdaptiveTransmission}">
-			<!-- work in progess
+			<!-- work in progess -->
 			<gazebo>
 				<plugin name="gazebo_ros_soft_hand" filename="libgazebo_ros_soft_hand.so">
 					<robotNamespace>soft_hand</robotNamespace>
+					<!-- the joint that rule them all -->
+					<synergyJoint>hand_synergy_joint</synergyJoint>
 				</plugin>
 			</gazebo>
-			-->
 		</xacro:if>
 		<xacro:unless value="${withAdaptiveTransmission}">

File: soft_hand/soft_hand_description/model/soft_hand.transmission.xacro (robot description, xacro)
@@ -131,5 +131,16 @@
     </xacro:unless>
     <xacro:if value="${withAdaptiveTransmission}">
-      <!--
+      <!-- work in progress -->
+      <transmission name="synergy_trans">
+          <type>transmission_interface/SimpleTransmission</type>
+          <joint name="synergy_joint">
+            <hardwareInterface>EffortJointInterface</hardwareInterface>
+          </joint>
+          <actuator name="synergy_motor">
+            <hardwareInterface>EffortJointInterface</hardwareInterface>
+            <mechanicalReduction>1</mechanicalReduction>
+          </actuator>
+      </transmission>
+<!--
       <transmission name="${name}">
         <type>transmission_interface/AdaptiveSynergyTransmission</type>
@@ -139,5 +150,5 @@
             <mechanicalReduction>2</mechanicalReduction>
             <mechanicalElasticity>3</mechanicalElasticity>
-            <hardwareInterface>hardware_interface/EffortJointInterface</hardwareInterface>
+            <hardwareInterface>EffortJointInterface</hardwareInterface>
           </joint>
           <joint name="${name}_thumb_inner_joint">
@@ -146,5 +157,5 @@
             <mechanicalReduction>2</mechanicalReduction>
             <mechanicalElasticity>3</mechanicalElasticity>
-            <hardwareInterface>hardware_interface/EffortJointInterface</hardwareInterface>
+            <hardwareInterface>EffortJointInterface</hardwareInterface>
           </joint>
           <joint name="${name}_thumb_outer_joint">
@@ -153,5 +164,5 @@
             <mechanicalReduction>2</mechanicalReduction>
             <mechanicalElasticity>3</mechanicalElasticity>
-            <hardwareInterface>hardware_interface/EffortJointInterface</hardwareInterface>
+            <hardwareInterface>EffortJointInterface</hardwareInterface>
           </joint>
           <joint name="${name}_index_abd_joint">
@@ -160,5 +171,5 @@
             <mechanicalReduction>2</mechanicalReduction>
             <mechanicalElasticity>3</mechanicalElasticity>
-            <hardwareInterface>hardware_interface/EffortJointInterface</hardwareInterface>
+            <hardwareInterface>EffortJointInterface</hardwareInterface>
           </joint>
           <joint name="${name}_index_inner_joint">
@@ -167,5 +178,5 @@
             <mechanicalReduction>2</mechanicalReduction>
             <mechanicalElasticity>3</mechanicalElasticity>
-            <hardwareInterface>hardware_interface/EffortJointInterface</hardwareInterface>
+            <hardwareInterface>EffortJointInterface</hardwareInterface>
           </joint>
           <joint name="${name}_index_middle_joint">
@@ -174,5 +185,5 @@
             <mechanicalReduction>2</mechanicalReduction>
             <mechanicalElasticity>3</mechanicalElasticity>
-            <hardwareInterface>hardware_interface/EffortJointInterface</hardwareInterface>
+            <hardwareInterface>EffortJointInterface</hardwareInterface>
           </joint>
           <joint name="${name}_index_distal_joint">
@@ -181,5 +192,5 @@
             <mechanicalReduction>2</mechanicalReduction>
             <mechanicalElasticity>3</mechanicalElasticity>
-            <hardwareInterface>hardware_interface/EffortJointInterface</hardwareInterface>
+            <hardwareInterface>EffortJointInterface</hardwareInterface>
           </joint>
           <joint name="${name}_middle_abd_joint">
@@ -188,5 +199,5 @@
             <mechanicalReduction>2</mechanicalReduction>
             <mechanicalElasticity>3</mechanicalElasticity>
-            <hardwareInterface>hardware_interface/EffortJointInterface</hardwareInterface>
+            <hardwareInterface>EffortJointInterface</hardwareInterface>
           </joint>
           <joint name="${name}_middle_inner_joint">
@@ -195,5 +206,5 @@
             <mechanicalReduction>2</mechanicalReduction>
             <mechanicalElasticity>3</mechanicalElasticity>
-            <hardwareInterface>hardware_interface/EffortJointInterface</hardwareInterface>
+            <hardwareInterface>EffortJointInterface</hardwareInterface>
           </joint>
           <joint name="${name}_middle_middle_joint">
@@ -202,5 +213,5 @@
             <mechanicalReduction>2</mechanicalReduction>
             <mechanicalElasticity>3</mechanicalElasticity>
-            <hardwareInterface>hardware_interface/EffortJointInterface</hardwareInterface>
+            <hardwareInterface>EffortJointInterface</hardwareInterface>
           </joint>
           <joint name="${name}_middle_distal_joint">
@@ -209,5 +220,5 @@
             <mechanicalReduction>2</mechanicalReduction>
             <mechanicalElasticity>3</mechanicalElasticity>
-            <hardwareInterface>hardware_interface/EffortJointInterface</hardwareInterface>
+            <hardwareInterface>EffortJointInterface</hardwareInterface>
           </joint>
           <joint name="${name}_ring_abd_joint">
@@ -216,5 +227,5 @@
             <mechanicalReduction>2</mechanicalReduction>
             <mechanicalElasticity>3</mechanicalElasticity>
-            <hardwareInterface>hardware_interface/EffortJointInterface</hardwareInterface>
+            <hardwareInterface>EffortJointInterface</hardwareInterface>
           </joint>
           <joint name="${name}_ring_inner_joint">
@@ -223,5 +234,5 @@
             <mechanicalReduction>2</mechanicalReduction>
             <mechanicalElasticity>3</mechanicalElasticity>
-            <hardwareInterface>hardware_interface/EffortJointInterface</hardwareInterface>
+            <hardwareInterface>EffortJointInterface</hardwareInterface>
           </joint>
           <joint name="${name}_ring_middle_joint">
@@ -230,5 +241,5 @@
             <mechanicalReduction>2</mechanicalReduction>
             <mechanicalElasticity>3</mechanicalElasticity>
-            <hardwareInterface>hardware_interface/EffortJointInterface</hardwareInterface>
+            <hardwareInterface>EffortJointInterface</hardwareInterface>
           </joint>
           <joint name="${name}_ring_distal_joint">
@@ -237,5 +248,5 @@
             <mechanicalReduction>2</mechanicalReduction>
             <mechanicalElasticity>3</mechanicalElasticity>
-            <hardwareInterface>hardware_interface/EffortJointInterface</hardwareInterface>
+            <hardwareInterface>EffortJointInterface</hardwareInterface>
           </joint>
           <joint name="${name}_little_abd_joint">
@@ -244,5 +255,5 @@
             <mechanicalReduction>2</mechanicalReduction>
             <mechanicalElasticity>3</mechanicalElasticity>
-            <hardwareInterface>hardware_interface/EffortJointInterface</hardwareInterface>
+            <hardwareInterface>EffortJointInterface</hardwareInterface>
           </joint>
           <joint name="${name}_little_inner_joint">
@@ -251,5 +262,5 @@
             <mechanicalReduction>2</mechanicalReduction>
             <mechanicalElasticity>3</mechanicalElasticity>
-            <hardwareInterface>hardware_interface/EffortJointInterface</hardwareInterface>
+            <hardwareInterface>EffortJointInterface</hardwareInterface>
           </joint>
           <joint name="${name}_little_middle_joint">
@@ -258,5 +269,5 @@
             <mechanicalReduction>2</mechanicalReduction>
             <mechanicalElasticity>3</mechanicalElasticity>
-            <hardwareInterface>hardware_interface/EffortJointInterface</hardwareInterface>
+            <hardwareInterface>EffortJointInterface</hardwareInterface>
           </joint>
           <joint name="${name}_little_distal_joint">
@@ -265,12 +276,13 @@
             <mechanicalReduction>2</mechanicalReduction>
             <mechanicalElasticity>3</mechanicalElasticity>
-            <hardwareInterface>hardware_interface/EffortJointInterface</hardwareInterface>
+            <hardwareInterface>EffortJointInterface</hardwareInterface>
           </joint>
           <actuator name="${name}_actuator">
             <role>actuator</role>
-            <hardwareInterface>hardware_interface/EffortJointInterface</hardwareInterface>
-          </actuator>
-      </transmission>
-      -->
+            <mechanicalReduction>2</mechanicalReduction>
+            <hardwareInterface>EffortJointInterface</hardwareInterface>
+          </actuator>
+      </transmission>
+-->
     </xacro:if>
   </xacro:macro>

File: soft_hand/soft_hand_description/model/soft_hand.urdf.xacro (robot description, xacro)
@@ -51,5 +51,5 @@
 	<!-- SOFT FINGER model -->
 	<!-- 4 fingers are equal (index, middle, ring, little) -->
-	<xacro:macro name="soft_finger" params="parent name position orientation abd_R inner_R middle_R outer_R">
+	<xacro:macro name="soft_finger" params="parent name position orientation useMimicTag abd_R inner_R middle_R outer_R">
 		<!-- KNUCKLE -->
 		<joint name="${name}_abd_joint" type="revolute">
@@ -60,5 +60,7 @@
 			<limit lower="${abd_lb *pi/180}" upper="${abd_ub *pi/180}" effort="${effort}" velocity="${velocity}"/>
 			<dynamics damping="${damping}" friction="${friction}"/>
-			<mimic joint="synergy_joint" multiplier="${abd_R}"/>
+			<xacro:if value="${useMimicTag}">
+				<mimic joint="synergy_joint" multiplier="${abd_R}"/>
+			</xacro:if>
 		</joint>
 		<link name="${name}_knuckle_link">
@@ -89,5 +91,7 @@
 			<limit lower="${inner_lb *pi/180}" upper="${inner_ub *pi/180}" effort="${effort}" velocity="${velocity}"/>
 			<dynamics damping="${damping}" friction="${friction}"/>
-			<mimic joint="synergy_joint" multiplier="${inner_R}"/>
+			<xacro:if value="${useMimicTag}">
+				<mimic joint="synergy_joint" multiplier="${inner_R}"/>
+			</xacro:if>
 		</joint>
 		<link name="${name}_fake_link1">
@@ -103,5 +107,7 @@
 			<limit lower="${inner_lb *pi/180}" upper="${inner_ub *pi/180}" effort="${effort}" velocity="${velocity}"/>
 			<dynamics damping="${damping}" friction="${friction}"/>
-			<mimic joint="synergy_joint" multiplier="${inner_R}" />
+			<xacro:if value="${useMimicTag}">
+				<mimic joint="synergy_joint" multiplier="${inner_R}" />
+			</xacro:if>
 		</joint>
 		<link name="${name}_proximal_link">
@@ -132,5 +138,7 @@
 			<limit lower="${middle_lb *pi/180}" upper="${middle_ub *pi/180}" effort="${effort}" velocity="${velocity}"/>
 			<dynamics damping="${damping}" friction="${friction}"/>
-			<mimic joint="synergy_joint" multiplier="${middle_R}"/>
+			<xacro:if value="${useMimicTag}">
+				<mimic joint="synergy_joint" multiplier="${middle_R}"/>
+			</xacro:if>
 		</joint>
 		<link name="${name}_fake_link2">
@@ -146,5 +154,7 @@
 			<limit lower="${middle_lb *pi/180}" upper="${middle_ub *pi/180}" effort="${effort}" velocity="${velocity}"/>
 			<dynamics damping="${damping}" friction="${friction}"/>
-			<mimic joint="synergy_joint" multiplier="${middle_R}"/>
+			<xacro:if value="${useMimicTag}">
+				<mimic joint="synergy_joint" multiplier="${middle_R}"/>
+			</xacro:if>
 		</joint>
 		<link name="${name}_middle_link">
@@ -173,5 +183,7 @@
 			<limit lower="${outer_lb *pi/180}" upper="${outer_ub *pi/180}" effort="${effort}" velocity="${velocity}"/>
 			<dynamics damping="${damping}" friction="${friction}"/>
-			<mimic joint="synergy_joint" multiplier="${outer_R}"/>
+			<xacro:if value="${useMimicTag}">
+				<mimic joint="synergy_joint" multiplier="${outer_R}"/>
+			</xacro:if>
 		</joint>
 		<link name="${name}_fake_link3">
@@ -187,5 +199,7 @@
 			<limit lower="${outer_lb *pi/180}" upper="${outer_ub *pi/180}" effort="${effort}" velocity="${velocity}"/>
 			<dynamics damping="${damping}" friction="${friction}"/>
-			<mimic joint="synergy_joint" multiplier="${outer_R}"/>
+			<xacro:if value="${useMimicTag}">
+				<mimic joint="synergy_joint" multiplier="${outer_R}"/>
+			</xacro:if>
 		</joint>
 		<link name="${name}_distal_link">
@@ -209,5 +223,5 @@
 	<!-- THUMB MODEL -->
 	<!-- It has one joint less than rest of fingers -->
-	<xacro:macro name="soft_thumb" params="parent name position orientation abd_R inner_R outer_R">
+	<xacro:macro name="soft_thumb" params="parent name position orientation useMimicTag abd_R inner_R outer_R">
 		<!-- KNUCKLE -->
 		<joint name="${name}_abd_joint" type="revolute">
@@ -218,5 +232,7 @@
 			<limit lower="${thumb_abd_lb *pi/180}" upper="${thumb_abd_ub *pi/180}" effort="${effort}" velocity="${velocity}"/>
 			<dynamics damping="${damping}" friction="${friction}"/>
-			<mimic joint="synergy_joint" multiplier="${abd_R}"/>
+			<xacro:if value="${useMimicTag}">
+				<mimic joint="synergy_joint" multiplier="${abd_R}"/>
+			</xacro:if>
 		</joint>
 		<link name="${name}_knuckle_link">
@@ -245,5 +261,7 @@
 			<limit lower="${inner_lb *pi/180}" upper="${inner_ub *pi/180}" effort="${effort}" velocity="${velocity}"/>
 			<dynamics damping="${damping}" friction="${friction}"/>
-			<mimic joint="synergy_joint" multiplier="${inner_R}"/>
+			<xacro:if value="${useMimicTag}">
+				<mimic joint="synergy_joint" multiplier="${inner_R}"/>
+			</xacro:if>
 		</joint>
 		<link name="${name}_fake_link1">
@@ -259,5 +277,7 @@
 			<limit lower="${inner_lb *pi/180}" upper="${inner_ub *pi/180}" effort="${effort}" velocity="${velocity}"/>
 			<dynamics damping="${damping}" friction="${friction}"/>
-			<mimic joint="synergy_joint" multiplier="${inner_R}" />
+			<xacro:if value="${useMimicTag}">
+				<mimic joint="synergy_joint" multiplier="${inner_R}" />
+			</xacro:if>
 		</joint>
 		<link name="${name}_proximal_link">
@@ -286,5 +306,7 @@
 			<limit lower="${outer_lb *pi/180}" upper="${outer_ub *pi/180}" effort="${effort}" velocity="${velocity}"/>
 			<dynamics damping="${damping}" friction="${friction}"/>
-			<mimic joint="synergy_joint" multiplier="${outer_R}"/>
+			<xacro:if value="${useMimicTag}">
+				<mimic joint="synergy_joint" multiplier="${outer_R}"/>
+			</xacro:if>
 		</joint>
 		<link name="${name}_fake_link3">
@@ -300,5 +322,7 @@
 			<limit lower="${outer_lb *pi/180}" upper="${outer_ub *pi/180}" effort="${effort}" velocity="${velocity}"/>
 			<dynamics damping="${damping}" friction="${friction}"/>
-			<mimic joint="synergy_joint" multiplier="${outer_R}" />
+			<xacro:if value="${useMimicTag}">
+				<mimic joint="synergy_joint" multiplier="${outer_R}" />
+			</xacro:if>
 		</joint>
 		<link name="${name}_distal_link">
@@ -321,5 +345,5 @@
 	</xacro:macro>
 	<!-- SOFT HAND MODEL -->
-	<xacro:macro name="soft_hand" params="parent name withAdaptiveTransmission *origin">
+	<xacro:macro name="soft_hand" params="parent name withAdaptiveTransmission useMimicTag *origin">
 		<!-- MOTOR JOINT -->
 		<joint name="synergy_joint" type="revolute" >
@@ -330,5 +354,9 @@
 			<dynamics damping="${synergy_damping}" friction="${synergy_friction}"/>
 		</joint>
-		<link name="invisible_wire_link"/>
+		<link name="invisible_wire_link">
+			<inertial>
+				<insert_block name="negligible_inertia"/>
+			</inertial>
+		</link>
 		<!-- PALM -->
 		<joint name="${name}_palm_joint" type="fixed" >
@@ -355,9 +383,9 @@
 		</link>
 		<!-- THUMB AND FINGERS -->
-		<xacro:soft_thumb parent="${name}_palm_link" name="${name}_thumb" position="-0.0418769 0.0538740 -0.00691972" orientation="0 0 -0.43633181" abd_R="${thumb_abd_R *(thumb_abd_ub - thumb_abd_lb)*pi/180}" inner_R="${thumb_inner_R *(inner_ub - inner_lb)*pi/180}" outer_R="${thumb_outer_R *(outer_ub - outer_lb)*pi/180}"/>
-		<xacro:soft_finger parent="${name}_palm_link" name="${name}_index" position="-0.0285 0.0943918 0.00205" orientation="${180*pi/180} 0 ${(-90+20)*pi/180}" abd_R="${index_abd_R}" inner_R="${index_inner_R *(inner_ub - inner_lb)*pi/180}" middle_R="${index_middle_R *(middle_ub - middle_lb)*pi/180}" outer_R="${index_outer_R *(outer_ub - outer_lb)*pi/180}" />
-		<xacro:soft_finger parent="${name}_palm_link" name="${name}_middle" position="-0.009 0.107892 0.00205" orientation="${180*pi/180} 0 ${-90*pi/180}" abd_R="${middle_abd_R}" inner_R="${middle_inner_R *(inner_ub - inner_lb)*pi/180}" middle_R="${middle_middle_R *(middle_ub - middle_lb)*pi/180}" outer_R="${middle_outer_R *(outer_ub - outer_lb)*pi/180}" />
-		<xacro:soft_finger parent="${name}_palm_link" name="${name}_ring" position="0.0105 0.0943918 0.00205" orientation="${180*pi/180} 0 ${(-90-10)*pi/180}" abd_R="${ring_abd_R}" inner_R="${ring_inner_R *(inner_ub - inner_lb)*pi/180}" middle_R="${ring_middle_R *(middle_ub - middle_lb)*pi/180}" outer_R="${ring_outer_R *(outer_ub - outer_lb)*pi/180}" />
-		<xacro:soft_finger parent="${name}_palm_link" name="${name}_little" position="0.030 0.0808918 0.00205" orientation="${180*pi/180} 0 ${(-90-20)*pi/180}" abd_R="${little_abd_R}" inner_R="${little_inner_R *(inner_ub - inner_lb)*pi/180}" middle_R="${little_middle_R *(middle_ub - middle_lb)*pi/180}" outer_R="${little_outer_R *(outer_ub - outer_lb)*pi/180}" />
+		<xacro:soft_thumb parent="${name}_palm_link" name="${name}_thumb" position="-0.0418769 0.0538740 -0.00691972" orientation="0 0 -0.43633181" useMimicTag="${useMimicTag}" abd_R="${thumb_abd_R *(thumb_abd_ub - thumb_abd_lb)*pi/180}" inner_R="${thumb_inner_R *(inner_ub - inner_lb)*pi/180}" outer_R="${thumb_outer_R *(outer_ub - outer_lb)*pi/180}"/>
+		<xacro:soft_finger parent="${name}_palm_link" name="${name}_index" position="-0.0285 0.0943918 0.00205" orientation="${180*pi/180} 0 ${(-90+20)*pi/180}" useMimicTag="${useMimicTag}" abd_R="${index_abd_R}" inner_R="${index_inner_R *(inner_ub - inner_lb)*pi/180}" middle_R="${index_middle_R *(middle_ub - middle_lb)*pi/180}" outer_R="${index_outer_R *(outer_ub - outer_lb)*pi/180}" />
+		<xacro:soft_finger parent="${name}_palm_link" name="${name}_middle" position="-0.009 0.107892 0.00205" orientation="${180*pi/180} 0 ${-90*pi/180}" useMimicTag="${useMimicTag}" abd_R="${middle_abd_R}" inner_R="${middle_inner_R *(inner_ub - inner_lb)*pi/180}" middle_R="${middle_middle_R *(middle_ub - middle_lb)*pi/180}" outer_R="${middle_outer_R *(outer_ub - outer_lb)*pi/180}" />
+		<xacro:soft_finger parent="${name}_palm_link" name="${name}_ring" position="0.0105 0.0943918 0.00205" orientation="${180*pi/180} 0 ${(-90-10)*pi/180}" useMimicTag="${useMimicTag}" abd_R="${ring_abd_R}" inner_R="${ring_inner_R *(inner_ub - inner_lb)*pi/180}" middle_R="${ring_middle_R *(middle_ub - middle_lb)*pi/180}" outer_R="${ring_outer_R *(outer_ub - outer_lb)*pi/180}" />
+		<xacro:soft_finger parent="${name}_palm_link" name="${name}_little" position="0.030 0.0808918 0.00205" orientation="${180*pi/180} 0 ${(-90-20)*pi/180}" useMimicTag="${useMimicTag}" abd_R="${little_abd_R}" inner_R="${little_inner_R *(inner_ub - inner_lb)*pi/180}" middle_R="${little_middle_R *(middle_ub - middle_lb)*pi/180}" outer_R="${little_outer_R *(outer_ub - outer_lb)*pi/180}" />
 		<xacro:soft_hand_transmission name="${name}" withAdaptiveTransmission="${withAdaptiveTransmission}"/>
 		<xacro:soft_hand_gazebo name="${name}" withAdaptiveTransmission="${withAdaptiveTransmission}"/>
