Commit message: adaptive model almost ready, gazebo crashes when the transmission propagates, still looking at it

File: soft_hand/soft_hand_description/model/soft_hand.gazebo.xacro (robot description, xacro)
@@ -3,5 +3,5 @@
 	<!-- configure how all bodies will behave in gazebo (particular behavior can be set at each link as well) -->
 	<xacro:property name="gazebo_body_elements">
-		<material>Gazebo/Black</material>
+		<!-- material>Gazebo/FlatBlack</material -->
 		<gravity>true</gravity>
 		<mu1>0.2</mu1>
@@ -25,4 +25,5 @@
 	<!-- configure how all joints will behave in gazebo (particular behavior can be set at each joint as well) -->
 	<xacro:property name="gazebo_joint_elements">
+		<provideFeedback>True</provideFeedback>
 		<!--
 		<kp> </kp>
@@ -30,5 +31,4 @@
 		<stopCfm> </stopCfm>
 		<stopErp> </stopErp>
-		<provideFeedback> </provideFeedback>
 		<cfmDamping> </cfmDamping>
 		<fudgeFactor> </fudgeFactor>
@@ -42,6 +42,4 @@
 				<plugin name="gazebo_ros_soft_hand" filename="libgazebo_ros_soft_hand.so">
 					<robotNamespace>soft_hand</robotNamespace>
-					<!-- the joint that rule them all -->
-					<synergyJoint>hand_synergy_joint</synergyJoint>
 				</plugin>
 			</gazebo>

File: soft_hand/soft_hand_description/model/soft_hand.transmission.xacro (robot description, xacro)
@@ -8,5 +8,4 @@
         </joint>
         <actuator name="${name}_${finger}_abd_motor">
-          <hardwareInterface>EffortJointInterface</hardwareInterface>
           <mechanicalReduction>1</mechanicalReduction>
         </actuator>
@@ -18,5 +17,4 @@
         </joint>
         <actuator name="${name}_${finger}_inner_motor">
-          <hardwareInterface>EffortJointInterface</hardwareInterface>
           <mechanicalReduction>1</mechanicalReduction>
         </actuator>
@@ -28,5 +26,4 @@
         </joint>
         <actuator name="${name}_${finger}_inner_motor">
-          <hardwareInterface>EffortJointInterface</hardwareInterface>
           <mechanicalReduction>1</mechanicalReduction>
         </actuator>
@@ -38,5 +35,4 @@
         </joint>
         <actuator name="${name}_${finger}_middle_motor">
-          <hardwareInterface>EffortJointInterface</hardwareInterface>
           <mechanicalReduction>1</mechanicalReduction>
         </actuator>
@@ -48,5 +44,4 @@
         </joint>
         <actuator name="${name}_${finger}_middle_motor">
-          <hardwareInterface>EffortJointInterface</hardwareInterface>
           <mechanicalReduction>1</mechanicalReduction>
         </actuator>
@@ -58,5 +53,4 @@
         </joint>
         <actuator name="${name}_${finger}_outer_motor">
-          <hardwareInterface>EffortJointInterface</hardwareInterface>
           <mechanicalReduction>1</mechanicalReduction>
         </actuator>
@@ -68,5 +62,4 @@
         </joint>
         <actuator name="${name}_${finger}_outer_motor">
-          <hardwareInterface>EffortJointInterface</hardwareInterface>
           <mechanicalReduction>1</mechanicalReduction>
         </actuator>
@@ -81,5 +74,4 @@
           </joint>
           <actuator name="${name}_thumb_abd_motor">
-            <hardwareInterface>EffortJointInterface</hardwareInterface>
             <mechanicalReduction>1</mechanicalReduction>
           </actuator>
@@ -91,5 +83,4 @@
           </joint>
           <actuator name="${name}_thumb_inner_motor">
-            <hardwareInterface>EffortJointInterface</hardwareInterface>
             <mechanicalReduction>1</mechanicalReduction>
           </actuator>
@@ -101,5 +92,4 @@
           </joint>
           <actuator name="${name}_thumb_inner_motor">
-            <hardwareInterface>EffortJointInterface</hardwareInterface>
             <mechanicalReduction>1</mechanicalReduction>
           </actuator>
@@ -111,5 +101,4 @@
           </joint>
           <actuator name="${name}_thumb_outer_motor">
-            <hardwareInterface>EffortJointInterface</hardwareInterface>
             <mechanicalReduction>1</mechanicalReduction>
           </actuator>
@@ -121,5 +110,4 @@
           </joint>
           <actuator name="${name}_thumb_outer_motor">
-            <hardwareInterface>EffortJointInterface</hardwareInterface>
             <mechanicalReduction>1</mechanicalReduction>
           </actuator>
@@ -138,151 +126,149 @@
           </joint>
           <actuator name="synergy_motor">
-            <hardwareInterface>EffortJointInterface</hardwareInterface>
-            <mechanicalReduction>1</mechanicalReduction>
-          </actuator>
-      </transmission>
-<!--
+            <mechanicalReduction>1</mechanicalReduction>
+          </actuator>
+      </transmission>
       <transmission name="${name}">
         <type>transmission_interface/AdaptiveSynergyTransmission</type>
           <joint name="${name}_thumb_abd_joint">
             <role>joint1</role>
-            <offset>-0.5</offset>
-            <mechanicalReduction>2</mechanicalReduction>
-            <mechanicalElasticity>3</mechanicalElasticity>
-            <hardwareInterface>EffortJointInterface</hardwareInterface>
+            <offset>-0.0</offset>
+            <mechanicalReduction>1</mechanicalReduction>
+            <mechanicalElasticity>1</mechanicalElasticity>
+            <!-- in this transmission type, this value depend on teh causality chosen in the plugin -->
+            <!-- ToDo: parametrize! -->
+            <hardwareInterface>PositionJointInterface</hardwareInterface>
           </joint>
           <joint name="${name}_thumb_inner_joint">
             <role>joint2</role>
-            <offset>-0.5</offset>
-            <mechanicalReduction>2</mechanicalReduction>
-            <mechanicalElasticity>3</mechanicalElasticity>
-            <hardwareInterface>EffortJointInterface</hardwareInterface>
+            <offset>-0.0</offset>
+            <mechanicalReduction>1</mechanicalReduction>
+            <mechanicalElasticity>1</mechanicalElasticity>
+            <hardwareInterface>PositionJointInterface</hardwareInterface>
           </joint>
           <joint name="${name}_thumb_outer_joint">
             <role>joint3</role>
-            <offset>-0.5</offset>
-            <mechanicalReduction>2</mechanicalReduction>
-            <mechanicalElasticity>3</mechanicalElasticity>
-            <hardwareInterface>EffortJointInterface</hardwareInterface>
+            <offset>-0.0</offset>
+            <mechanicalReduction>1</mechanicalReduction>
+            <mechanicalElasticity>1</mechanicalElasticity>
+            <hardwareInterface>PositionJointInterface</hardwareInterface>
           </joint>
           <joint name="${name}_index_abd_joint">
             <role>joint4</role>
-            <offset>-0.5</offset>
-            <mechanicalReduction>2</mechanicalReduction>
-            <mechanicalElasticity>3</mechanicalElasticity>
-            <hardwareInterface>EffortJointInterface</hardwareInterface>
+            <offset>-0.0</offset>
+            <mechanicalReduction>1</mechanicalReduction>
+            <mechanicalElasticity>1</mechanicalElasticity>
+            <hardwareInterface>PositionJointInterface</hardwareInterface>
           </joint>
           <joint name="${name}_index_inner_joint">
             <role>joint5</role>
-            <offset>-0.5</offset>
-            <mechanicalReduction>2</mechanicalReduction>
-            <mechanicalElasticity>3</mechanicalElasticity>
-            <hardwareInterface>EffortJointInterface</hardwareInterface>
+            <offset>-0.0</offset>
+            <mechanicalReduction>1</mechanicalReduction>
+            <mechanicalElasticity>1</mechanicalElasticity>
+            <hardwareInterface>PositionJointInterface</hardwareInterface>
           </joint>
           <joint name="${name}_index_middle_joint">
             <role>joint6</role>
-            <offset>-0.5</offset>
-            <mechanicalReduction>2</mechanicalReduction>
-            <mechanicalElasticity>3</mechanicalElasticity>
-            <hardwareInterface>EffortJointInterface</hardwareInterface>
-          </joint>
-          <joint name="${name}_index_distal_joint">
+            <offset>-0.0</offset>
+            <mechanicalReduction>1</mechanicalReduction>
+            <mechanicalElasticity>1</mechanicalElasticity>
+            <hardwareInterface>PositionJointInterface</hardwareInterface>
+          </joint>
+          <joint name="${name}_index_outer_joint">
             <role>joint7</role>
-            <offset>-0.5</offset>
-            <mechanicalReduction>2</mechanicalReduction>
-            <mechanicalElasticity>3</mechanicalElasticity>
-            <hardwareInterface>EffortJointInterface</hardwareInterface>
+            <offset>-0.0</offset>
+            <mechanicalReduction>1</mechanicalReduction>
+            <mechanicalElasticity>1</mechanicalElasticity>
+            <hardwareInterface>PositionJointInterface</hardwareInterface>
           </joint>
           <joint name="${name}_middle_abd_joint">
             <role>joint8</role>
-            <offset>-0.5</offset>
-            <mechanicalReduction>2</mechanicalReduction>
-            <mechanicalElasticity>3</mechanicalElasticity>
-            <hardwareInterface>EffortJointInterface</hardwareInterface>
+            <offset>-0.0</offset>
+            <mechanicalReduction>1</mechanicalReduction>
+            <mechanicalElasticity>1</mechanicalElasticity>
+            <hardwareInterface>PositionJointInterface</hardwareInterface>
           </joint>
           <joint name="${name}_middle_inner_joint">
             <role>joint9</role>
-            <offset>-0.5</offset>
-            <mechanicalReduction>2</mechanicalReduction>
-            <mechanicalElasticity>3</mechanicalElasticity>
-            <hardwareInterface>EffortJointInterface</hardwareInterface>
+            <offset>-0.0</offset>
+            <mechanicalReduction>1</mechanicalReduction>
+            <mechanicalElasticity>1</mechanicalElasticity>
+            <hardwareInterface>PositionJointInterface</hardwareInterface>
           </joint>
           <joint name="${name}_middle_middle_joint">
             <role>joint10</role>
-            <offset>-0.5</offset>
-            <mechanicalReduction>2</mechanicalReduction>
-            <mechanicalElasticity>3</mechanicalElasticity>
-            <hardwareInterface>EffortJointInterface</hardwareInterface>
-          </joint>
-          <joint name="${name}_middle_distal_joint">
+            <offset>-0.0</offset>
+            <mechanicalReduction>1</mechanicalReduction>
+            <mechanicalElasticity>1</mechanicalElasticity>
+            <hardwareInterface>PositionJointInterface</hardwareInterface>
+          </joint>
+          <joint name="${name}_middle_outer_joint">
             <role>joint11</role>
-            <offset>-0.5</offset>
-            <mechanicalReduction>2</mechanicalReduction>
-            <mechanicalElasticity>3</mechanicalElasticity>
-            <hardwareInterface>EffortJointInterface</hardwareInterface>
+            <offset>-0.0</offset>
+            <mechanicalReduction>1</mechanicalReduction>
+            <mechanicalElasticity>1</mechanicalElasticity>
+            <hardwareInterface>PositionJointInterface</hardwareInterface>
           </joint>
           <joint name="${name}_ring_abd_joint">
             <role>joint12</role>
-            <offset>-0.5</offset>
-            <mechanicalReduction>2</mechanicalReduction>
-            <mechanicalElasticity>3</mechanicalElasticity>
-            <hardwareInterface>EffortJointInterface</hardwareInterface>
+            <offset>-0.0</offset>
+            <mechanicalReduction>1</mechanicalReduction>
+            <mechanicalElasticity>1</mechanicalElasticity>
+            <hardwareInterface>PositionJointInterface</hardwareInterface>
           </joint>
           <joint name="${name}_ring_inner_joint">
             <role>joint13</role>
-            <offset>-0.5</offset>
-            <mechanicalReduction>2</mechanicalReduction>
-            <mechanicalElasticity>3</mechanicalElasticity>
-            <hardwareInterface>EffortJointInterface</hardwareInterface>
+            <offset>-0.0</offset>
+            <mechanicalReduction>1</mechanicalReduction>
+            <mechanicalElasticity>1</mechanicalElasticity>
+            <hardwareInterface>PositionJointInterface</hardwareInterface>
           </joint>
           <joint name="${name}_ring_middle_joint">
             <role>joint14</role>
-            <offset>-0.5</offset>
-            <mechanicalReduction>2</mechanicalReduction>
-            <mechanicalElasticity>3</mechanicalElasticity>
-            <hardwareInterface>EffortJointInterface</hardwareInterface>
-          </joint>
-          <joint name="${name}_ring_distal_joint">
+            <offset>-0.0</offset>
+            <mechanicalReduction>1</mechanicalReduction>
+            <mechanicalElasticity>1</mechanicalElasticity>
+            <hardwareInterface>PositionJointInterface</hardwareInterface>
+          </joint>
+          <joint name="${name}_ring_outer_joint">
             <role>joint15</role>
-            <offset>-0.5</offset>
-            <mechanicalReduction>2</mechanicalReduction>
-            <mechanicalElasticity>3</mechanicalElasticity>
-            <hardwareInterface>EffortJointInterface</hardwareInterface>
+            <offset>-0.0</offset>
+            <mechanicalReduction>1</mechanicalReduction>
+            <mechanicalElasticity>1</mechanicalElasticity>
+            <hardwareInterface>PositionJointInterface</hardwareInterface>
           </joint>
           <joint name="${name}_little_abd_joint">
             <role>joint16</role>
-            <offset>-0.5</offset>
-            <mechanicalReduction>2</mechanicalReduction>
-            <mechanicalElasticity>3</mechanicalElasticity>
-            <hardwareInterface>EffortJointInterface</hardwareInterface>
+            <offset>-0.0</offset>
+            <mechanicalReduction>1</mechanicalReduction>
+            <mechanicalElasticity>1</mechanicalElasticity>
+            <hardwareInterface>PositionJointInterface</hardwareInterface>
           </joint>
           <joint name="${name}_little_inner_joint">
             <role>joint17</role>
-            <offset>-0.5</offset>
-            <mechanicalReduction>2</mechanicalReduction>
-            <mechanicalElasticity>3</mechanicalElasticity>
-            <hardwareInterface>EffortJointInterface</hardwareInterface>
+            <offset>-0.0</offset>
+            <mechanicalReduction>1</mechanicalReduction>
+            <mechanicalElasticity>1</mechanicalElasticity>
+            <hardwareInterface>PositionJointInterface</hardwareInterface>
           </joint>
           <joint name="${name}_little_middle_joint">
             <role>joint18</role>
-            <offset>-0.5</offset>
-            <mechanicalReduction>2</mechanicalReduction>
-            <mechanicalElasticity>3</mechanicalElasticity>
-            <hardwareInterface>EffortJointInterface</hardwareInterface>
-          </joint>
-          <joint name="${name}_little_distal_joint">
+            <offset>-0.0</offset>
+            <mechanicalReduction>1</mechanicalReduction>
+            <mechanicalElasticity>1</mechanicalElasticity>
+            <hardwareInterface>PositionJointInterface</hardwareInterface>
+          </joint>
+          <joint name="${name}_little_outer_joint">
             <role>joint19</role>
-            <offset>-0.5</offset>
-            <mechanicalReduction>2</mechanicalReduction>
-            <mechanicalElasticity>3</mechanicalElasticity>
-            <hardwareInterface>EffortJointInterface</hardwareInterface>
+            <offset>-0.0</offset>
+            <mechanicalReduction>1</mechanicalReduction>
+            <mechanicalElasticity>1</mechanicalElasticity>
+            <hardwareInterface>PositionJointInterface</hardwareInterface>
           </joint>
           <actuator name="${name}_actuator">
-            <role>actuator</role>
-            <mechanicalReduction>2</mechanicalReduction>
-            <hardwareInterface>EffortJointInterface</hardwareInterface>
-          </actuator>
-      </transmission>
--->
+            <role>actuator1</role>
+            <mechanicalReduction>1</mechanicalReduction>
+          </actuator>
+      </transmission>
     </xacro:if>
   </xacro:macro>

File: soft_hand/soft_hand_description/model/soft_hand.urdf.xacro (robot description, xacro)
@@ -1,4 +1,9 @@
 <?xml version="1.0"?>
 <robot xmlns:xacro="http://ros.org/wiki/xacro">
+	<!--
+		HAND MODEL v.01
+		Material: ABS
+		CAD model available at: http://www.naturalmachinemotioninitiative.com/#!softhand/c24r2
+	-->
 	<xacro:include filename="$(find soft_hand_description)/model/materials.urdf.xacro"/>
 	<xacro:include filename="$(find soft_hand_description)/model/soft_hand.transmission.xacro"/>
@@ -48,5 +53,4 @@
 	<xacro:property name="synergy_damping" value="0.0" />
 	<xacro:property name="synergy_friction" value="0.0" />
-	<!-- HAND MODEL v.? Material: ABS -->
 	<!-- SOFT FINGER model -->
 	<!-- 4 fingers are equal (index, middle, ring, little) -->

File: soft_hand/soft_hand_description/robot/soft_hand_full_actuation.urdf.xacro (robot description, xacro)
@@ -24,5 +24,5 @@
 		<static>true</static>
 	</gazebo>
-	<xacro:soft_hand parent="wrist" name="hand" withAdaptiveTransmission="false">
+	<xacro:soft_hand parent="wrist" name="hand" withAdaptiveTransmission="false" useMimicTag="$(arg use_mimic_tag)">
 		<origin xyz="0 0 1" rpy="1.570796 0 0"/>
 	</xacro:soft_hand>
