Commit message: - gazebo soft hand plugin works in position control for the underactuated joints - deleting the transmission interface files, now in forked ros_control - added disable link and mimic joint gazebo plugins, but not used so far.

File: soft_hand/soft_hand_description/model/soft_hand.gazebo.xacro (robot description, xacro)
@@ -7,5 +7,5 @@
 		<mu1>0.2</mu1>
     	<mu2>0.2</mu2>
-    	<!-- <selfCollide>True</selfCollide> -->
+    	<!-- selfCollide>True</selfCollide -->
 		<!--
 		<dampingFactor> </dampingFactor>
@@ -35,5 +35,5 @@
 		-->
 	</xacro:property>
-	<xacro:macro name="soft_hand_gazebo" params="name withAdaptiveTransmission">
+	<xacro:macro name="soft_hand_gazebo" params="name withAdaptiveTransmission useMimicTag">
 		<!-- PLUGINS -->
 		<xacro:if value="${withAdaptiveTransmission}">
@@ -42,4 +42,12 @@
 				<plugin name="gazebo_ros_soft_hand" filename="libgazebo_ros_soft_hand.so">
 					<robotNamespace>soft_hand</robotNamespace>
+					<!-- select which type of hardware simulation you want:
+					     - DefatulSoftHandHWSim: underactuated with adaptivity
+					     - KinematicCtrlSoftHandHWSim: underactuation with pure kinematic
+					       control over joints (if you enable mimic tags, this one is automatically loaded)
+					-->
+					<xacro:if value="${useMimicTag}">
+						<robotSimType>gazebo_ros_soft_hand/KinematicCtrlSoftHandHWSim</robotSimType>
+					</xacro:if>
 				</plugin>
 			</gazebo>

File: soft_hand/soft_hand_description/model/soft_hand.transmission.xacro (robot description, xacro)
@@ -8,5 +8,5 @@
         </joint>
         <actuator name="${name}_${finger}_abd_motor">
-          <mechanicalReduction>1</mechanicalReduction>
+          <mechanicalReduction>1.0</mechanicalReduction>
         </actuator>
         </transmission>
@@ -17,5 +17,5 @@
         </joint>
         <actuator name="${name}_${finger}_inner_motor">
-          <mechanicalReduction>1</mechanicalReduction>
+          <mechanicalReduction>1.0</mechanicalReduction>
         </actuator>
         </transmission>
@@ -26,5 +26,5 @@
         </joint>
         <actuator name="${name}_${finger}_inner_motor">
-          <mechanicalReduction>1</mechanicalReduction>
+          <mechanicalReduction>1.0</mechanicalReduction>
         </actuator>
         </transmission>
@@ -35,5 +35,5 @@
         </joint>
         <actuator name="${name}_${finger}_middle_motor">
-          <mechanicalReduction>1</mechanicalReduction>
+          <mechanicalReduction>1.0</mechanicalReduction>
         </actuator>
         </transmission>
@@ -44,5 +44,5 @@
         </joint>
         <actuator name="${name}_${finger}_middle_motor">
-          <mechanicalReduction>1</mechanicalReduction>
+          <mechanicalReduction>1.0</mechanicalReduction>
         </actuator>
         </transmission>
@@ -53,5 +53,5 @@
         </joint>
         <actuator name="${name}_${finger}_outer_motor">
-          <mechanicalReduction>1</mechanicalReduction>
+          <mechanicalReduction>1.0</mechanicalReduction>
         </actuator>
         </transmission>
@@ -62,5 +62,5 @@
         </joint>
         <actuator name="${name}_${finger}_outer_motor">
-          <mechanicalReduction>1</mechanicalReduction>
+          <mechanicalReduction>1.0</mechanicalReduction>
         </actuator>
         </transmission>
@@ -74,5 +74,5 @@
           </joint>
           <actuator name="${name}_thumb_abd_motor">
-            <mechanicalReduction>1</mechanicalReduction>
+            <mechanicalReduction>1.0</mechanicalReduction>
           </actuator>
       </transmission>
@@ -83,5 +83,5 @@
           </joint>
           <actuator name="${name}_thumb_inner_motor">
-            <mechanicalReduction>1</mechanicalReduction>
+            <mechanicalReduction>1.0</mechanicalReduction>
           </actuator>
       </transmission>
@@ -92,5 +92,5 @@
           </joint>
           <actuator name="${name}_thumb_inner_motor">
-            <mechanicalReduction>1</mechanicalReduction>
+            <mechanicalReduction>1.0</mechanicalReduction>
           </actuator>
       </transmission>
@@ -101,5 +101,5 @@
           </joint>
           <actuator name="${name}_thumb_outer_motor">
-            <mechanicalReduction>1</mechanicalReduction>
+            <mechanicalReduction>1.0</mechanicalReduction>
           </actuator>
       </transmission>
@@ -110,5 +110,5 @@
           </joint>
           <actuator name="${name}_thumb_outer_motor">
-            <mechanicalReduction>1</mechanicalReduction>
+            <mechanicalReduction>1.0</mechanicalReduction>
           </actuator>
       </transmission>
@@ -126,5 +126,5 @@
           </joint>
           <actuator name="synergy_motor">
-            <mechanicalReduction>1</mechanicalReduction>
+            <mechanicalReduction>1.0</mechanicalReduction>
           </actuator>
       </transmission>
@@ -134,8 +134,6 @@
             <role>joint1</role>
             <offset>-0.0</offset>
-            <mechanicalReduction>1</mechanicalReduction>
-            <mechanicalElasticity>1</mechanicalElasticity>
-            <!-- in this transmission type, this value depend on teh causality chosen in the plugin -->
-            <!-- ToDo: parametrize! -->
+            <mechanicalReduction>1.3</mechanicalReduction>
+            <mechanicalElasticity>1.0</mechanicalElasticity>
             <hardwareInterface>PositionJointInterface</hardwareInterface>
           </joint>
@@ -143,6 +141,6 @@
             <role>joint2</role>
             <offset>-0.0</offset>
-            <mechanicalReduction>1</mechanicalReduction>
-            <mechanicalElasticity>1</mechanicalElasticity>
+            <mechanicalReduction>1.0</mechanicalReduction>
+            <mechanicalElasticity>1.0</mechanicalElasticity>
             <hardwareInterface>PositionJointInterface</hardwareInterface>
           </joint>
@@ -150,6 +148,6 @@
             <role>joint3</role>
             <offset>-0.0</offset>
-            <mechanicalReduction>1</mechanicalReduction>
-            <mechanicalElasticity>1</mechanicalElasticity>
+            <mechanicalReduction>1.0</mechanicalReduction>
+            <mechanicalElasticity>1.0</mechanicalElasticity>
             <hardwareInterface>PositionJointInterface</hardwareInterface>
           </joint>
@@ -157,6 +155,6 @@
             <role>joint4</role>
             <offset>-0.0</offset>
-            <mechanicalReduction>1</mechanicalReduction>
-            <mechanicalElasticity>1</mechanicalElasticity>
+            <mechanicalReduction>-0.2</mechanicalReduction>
+            <mechanicalElasticity>1.0</mechanicalElasticity>
             <hardwareInterface>PositionJointInterface</hardwareInterface>
           </joint>
@@ -164,6 +162,6 @@
             <role>joint5</role>
             <offset>-0.0</offset>
-            <mechanicalReduction>1</mechanicalReduction>
-            <mechanicalElasticity>1</mechanicalElasticity>
+            <mechanicalReduction>1.0</mechanicalReduction>
+            <mechanicalElasticity>1.0</mechanicalElasticity>
             <hardwareInterface>PositionJointInterface</hardwareInterface>
           </joint>
@@ -171,6 +169,6 @@
             <role>joint6</role>
             <offset>-0.0</offset>
-            <mechanicalReduction>1</mechanicalReduction>
-            <mechanicalElasticity>1</mechanicalElasticity>
+            <mechanicalReduction>1.0</mechanicalReduction>
+            <mechanicalElasticity>1.0</mechanicalElasticity>
             <hardwareInterface>PositionJointInterface</hardwareInterface>
           </joint>
@@ -178,6 +176,6 @@
             <role>joint7</role>
             <offset>-0.0</offset>
-            <mechanicalReduction>1</mechanicalReduction>
-            <mechanicalElasticity>1</mechanicalElasticity>
+            <mechanicalReduction>1.0</mechanicalReduction>
+            <mechanicalElasticity>1.0</mechanicalElasticity>
             <hardwareInterface>PositionJointInterface</hardwareInterface>
           </joint>
@@ -185,6 +183,6 @@
             <role>joint8</role>
             <offset>-0.0</offset>
-            <mechanicalReduction>1</mechanicalReduction>
-            <mechanicalElasticity>1</mechanicalElasticity>
+            <mechanicalReduction>0.001</mechanicalReduction>
+            <mechanicalElasticity>1.0</mechanicalElasticity>
             <hardwareInterface>PositionJointInterface</hardwareInterface>
           </joint>
@@ -192,6 +190,6 @@
             <role>joint9</role>
             <offset>-0.0</offset>
-            <mechanicalReduction>1</mechanicalReduction>
-            <mechanicalElasticity>1</mechanicalElasticity>
+            <mechanicalReduction>1.0</mechanicalReduction>
+            <mechanicalElasticity>1.0</mechanicalElasticity>
             <hardwareInterface>PositionJointInterface</hardwareInterface>
           </joint>
@@ -199,6 +197,6 @@
             <role>joint10</role>
             <offset>-0.0</offset>
-            <mechanicalReduction>1</mechanicalReduction>
-            <mechanicalElasticity>1</mechanicalElasticity>
+            <mechanicalReduction>1.0</mechanicalReduction>
+            <mechanicalElasticity>1.0</mechanicalElasticity>
             <hardwareInterface>PositionJointInterface</hardwareInterface>
           </joint>
@@ -206,6 +204,6 @@
             <role>joint11</role>
             <offset>-0.0</offset>
-            <mechanicalReduction>1</mechanicalReduction>
-            <mechanicalElasticity>1</mechanicalElasticity>
+            <mechanicalReduction>1.0</mechanicalReduction>
+            <mechanicalElasticity>1.0</mechanicalElasticity>
             <hardwareInterface>PositionJointInterface</hardwareInterface>
           </joint>
@@ -213,6 +211,6 @@
             <role>joint12</role>
             <offset>-0.0</offset>
-            <mechanicalReduction>1</mechanicalReduction>
-            <mechanicalElasticity>1</mechanicalElasticity>
+            <mechanicalReduction>0.2</mechanicalReduction>
+            <mechanicalElasticity>1.0</mechanicalElasticity>
             <hardwareInterface>PositionJointInterface</hardwareInterface>
           </joint>
@@ -220,6 +218,6 @@
             <role>joint13</role>
             <offset>-0.0</offset>
-            <mechanicalReduction>1</mechanicalReduction>
-            <mechanicalElasticity>1</mechanicalElasticity>
+            <mechanicalReduction>1.0</mechanicalReduction>
+            <mechanicalElasticity>1.0</mechanicalElasticity>
             <hardwareInterface>PositionJointInterface</hardwareInterface>
           </joint>
@@ -227,6 +225,6 @@
             <role>joint14</role>
             <offset>-0.0</offset>
-            <mechanicalReduction>1</mechanicalReduction>
-            <mechanicalElasticity>1</mechanicalElasticity>
+            <mechanicalReduction>1.0</mechanicalReduction>
+            <mechanicalElasticity>1.0</mechanicalElasticity>
             <hardwareInterface>PositionJointInterface</hardwareInterface>
           </joint>
@@ -234,6 +232,6 @@
             <role>joint15</role>
             <offset>-0.0</offset>
-            <mechanicalReduction>1</mechanicalReduction>
-            <mechanicalElasticity>1</mechanicalElasticity>
+            <mechanicalReduction>1.0</mechanicalReduction>
+            <mechanicalElasticity>1.0</mechanicalElasticity>
             <hardwareInterface>PositionJointInterface</hardwareInterface>
           </joint>
@@ -241,6 +239,6 @@
             <role>joint16</role>
             <offset>-0.0</offset>
-            <mechanicalReduction>1</mechanicalReduction>
-            <mechanicalElasticity>1</mechanicalElasticity>
+            <mechanicalReduction>0.4</mechanicalReduction>
+            <mechanicalElasticity>1.0</mechanicalElasticity>
             <hardwareInterface>PositionJointInterface</hardwareInterface>
           </joint>
@@ -248,6 +246,6 @@
             <role>joint17</role>
             <offset>-0.0</offset>
-            <mechanicalReduction>1</mechanicalReduction>
-            <mechanicalElasticity>1</mechanicalElasticity>
+            <mechanicalReduction>1.0</mechanicalReduction>
+            <mechanicalElasticity>1.0</mechanicalElasticity>
             <hardwareInterface>PositionJointInterface</hardwareInterface>
           </joint>
@@ -255,6 +253,6 @@
             <role>joint18</role>
             <offset>-0.0</offset>
-            <mechanicalReduction>1</mechanicalReduction>
-            <mechanicalElasticity>1</mechanicalElasticity>
+            <mechanicalReduction>1.0</mechanicalReduction>
+            <mechanicalElasticity>1.0</mechanicalElasticity>
             <hardwareInterface>PositionJointInterface</hardwareInterface>
           </joint>
@@ -262,11 +260,11 @@
             <role>joint19</role>
             <offset>-0.0</offset>
-            <mechanicalReduction>1</mechanicalReduction>
-            <mechanicalElasticity>1</mechanicalElasticity>
+            <mechanicalReduction>1.0</mechanicalReduction>
+            <mechanicalElasticity>1.0</mechanicalElasticity>
             <hardwareInterface>PositionJointInterface</hardwareInterface>
           </joint>
           <actuator name="${name}_actuator">
             <role>actuator1</role>
-            <mechanicalReduction>1</mechanicalReduction>
+            <mechanicalReduction>0.1</mechanicalReduction>
           </actuator>
       </transmission>

File: soft_hand/soft_hand_description/model/soft_hand.urdf.xacro (robot description, xacro)
@@ -393,5 +393,5 @@
 		<xacro:soft_finger parent="${name}_palm_link" name="${name}_little" position="0.030 0.0808918 0.00205" orientation="${180*pi/180} 0 ${(-90-20)*pi/180}" useMimicTag="${useMimicTag}" abd_R="${little_abd_R}" inner_R="${little_inner_R *(inner_ub - inner_lb)*pi/180}" middle_R="${little_middle_R *(middle_ub - middle_lb)*pi/180}" outer_R="${little_outer_R *(outer_ub - outer_lb)*pi/180}" />
 		<xacro:soft_hand_transmission name="${name}" withAdaptiveTransmission="${withAdaptiveTransmission}"/>
-		<xacro:soft_hand_gazebo name="${name}" withAdaptiveTransmission="${withAdaptiveTransmission}"/>
+		<xacro:soft_hand_gazebo name="${name}" withAdaptiveTransmission="${withAdaptiveTransmission}" useMimicTag="${useMimicTag}"/>
 	</xacro:macro>
 </robot>

File: soft_hand/soft_hand_description/robot/soft_hand_adaptive.urdf.xacro (robot description, xacro)
@@ -24,6 +24,32 @@
 		<static>true</static>
 	</gazebo>
-	<xacro:soft_hand parent="wrist" name="hand" withAdaptiveTransmission="true" useMimicTag="$(arg use_mimic_tag)">
+	<xacro:soft_hand parent="wrist" name="soft_hand" withAdaptiveTransmission="true" useMimicTag="$(arg use_mimic_tag)">
 		<origin xyz="0 0 1" rpy="1.570796 0 0"/>
 	</xacro:soft_hand>
+	<joint name="wrist_object_joint" type="fixed">
+		<origin xyz="0 0.05 1.1" rpy="0 0 0" />
+		<parent link="wrist"/>
+		<child link="object"/>
+	</joint>
+	<link name="object">
+		<inertial>
+			<insert_block name="negligible_inertia"/>
+		</inertial>
+		<visual>
+			<origin xyz="0 0 0" rpy="0 0 0"/>
+			<geometry>
+				<box size="0.05 0.05 0.05"/>
+			</geometry>
+		</visual>
+		<collision>
+			<origin xyz="0 0 0" rpy="0 0 0"/>
+			<geometry>
+				<box size="0.05 0.05 0.05"/>
+			</geometry>
+		</collision>
+	</link>
+	<gazebo reference="object">
+		<static>true</static>
+		<selfCollide>True</selfCollide>
+	</gazebo>
 </robot>
