Commit message: adaptive synergy working with contact force and kinematic information

File: soft_hand/soft_hand_description/model/soft_hand.transmission.xacro (robot description, xacro)
@@ -136,5 +136,6 @@
             <mechanicalReduction>1.3</mechanicalReduction>
             <mechanicalElasticity>1.0</mechanicalElasticity>
-            <hardwareInterface>PositionJointInterface</hardwareInterface>
+            <!-- hardwareInterface>PositionJointInterface</hardwareInterface -->
+            <hardwareInterface>EffortJointInterface</hardwareInterface>
           </joint>
           <joint name="${name}_thumb_inner_joint">
@@ -143,5 +144,6 @@
             <mechanicalReduction>1.0</mechanicalReduction>
             <mechanicalElasticity>1.0</mechanicalElasticity>
-            <hardwareInterface>PositionJointInterface</hardwareInterface>
+            <!-- hardwareInterface>PositionJointInterface</hardwareInterface -->
+            <hardwareInterface>EffortJointInterface</hardwareInterface>
           </joint>
           <joint name="${name}_thumb_outer_joint">
@@ -150,5 +152,6 @@
             <mechanicalReduction>1.0</mechanicalReduction>
             <mechanicalElasticity>1.0</mechanicalElasticity>
-            <hardwareInterface>PositionJointInterface</hardwareInterface>
+            <!-- hardwareInterface>PositionJointInterface</hardwareInterface -->
+            <hardwareInterface>EffortJointInterface</hardwareInterface>
           </joint>
           <joint name="${name}_index_abd_joint">
@@ -157,5 +160,6 @@
             <mechanicalReduction>-0.2</mechanicalReduction>
             <mechanicalElasticity>1.0</mechanicalElasticity>
-            <hardwareInterface>PositionJointInterface</hardwareInterface>
+            <!-- hardwareInterface>PositionJointInterface</hardwareInterface -->
+            <hardwareInterface>EffortJointInterface</hardwareInterface>
           </joint>
           <joint name="${name}_index_inner_joint">
@@ -164,5 +168,6 @@
             <mechanicalReduction>1.0</mechanicalReduction>
             <mechanicalElasticity>1.0</mechanicalElasticity>
-            <hardwareInterface>PositionJointInterface</hardwareInterface>
+            <!-- hardwareInterface>PositionJointInterface</hardwareInterface -->
+            <hardwareInterface>EffortJointInterface</hardwareInterface>
           </joint>
           <joint name="${name}_index_middle_joint">
@@ -171,5 +176,6 @@
             <mechanicalReduction>1.0</mechanicalReduction>
             <mechanicalElasticity>1.0</mechanicalElasticity>
-            <hardwareInterface>PositionJointInterface</hardwareInterface>
+            <!-- hardwareInterface>PositionJointInterface</hardwareInterface -->
+            <hardwareInterface>EffortJointInterface</hardwareInterface>
           </joint>
           <joint name="${name}_index_outer_joint">
@@ -178,5 +184,6 @@
             <mechanicalReduction>1.0</mechanicalReduction>
             <mechanicalElasticity>1.0</mechanicalElasticity>
-            <hardwareInterface>PositionJointInterface</hardwareInterface>
+            <!-- hardwareInterface>PositionJointInterface</hardwareInterface -->
+            <hardwareInterface>EffortJointInterface</hardwareInterface>
           </joint>
           <joint name="${name}_middle_abd_joint">
@@ -185,5 +192,6 @@
             <mechanicalReduction>0.001</mechanicalReduction>
             <mechanicalElasticity>1.0</mechanicalElasticity>
-            <hardwareInterface>PositionJointInterface</hardwareInterface>
+            <!-- hardwareInterface>PositionJointInterface</hardwareInterface -->
+            <hardwareInterface>EffortJointInterface</hardwareInterface>
           </joint>
           <joint name="${name}_middle_inner_joint">
@@ -192,5 +200,6 @@
             <mechanicalReduction>1.0</mechanicalReduction>
             <mechanicalElasticity>1.0</mechanicalElasticity>
-            <hardwareInterface>PositionJointInterface</hardwareInterface>
+            <!-- hardwareInterface>PositionJointInterface</hardwareInterface -->
+            <hardwareInterface>EffortJointInterface</hardwareInterface>
           </joint>
           <joint name="${name}_middle_middle_joint">
@@ -199,5 +208,6 @@
             <mechanicalReduction>1.0</mechanicalReduction>
             <mechanicalElasticity>1.0</mechanicalElasticity>
-            <hardwareInterface>PositionJointInterface</hardwareInterface>
+            <!-- hardwareInterface>PositionJointInterface</hardwareInterface -->
+            <hardwareInterface>EffortJointInterface</hardwareInterface>
           </joint>
           <joint name="${name}_middle_outer_joint">
@@ -206,5 +216,6 @@
             <mechanicalReduction>1.0</mechanicalReduction>
             <mechanicalElasticity>1.0</mechanicalElasticity>
-            <hardwareInterface>PositionJointInterface</hardwareInterface>
+            <!-- hardwareInterface>PositionJointInterface</hardwareInterface -->
+            <hardwareInterface>EffortJointInterface</hardwareInterface>
           </joint>
           <joint name="${name}_ring_abd_joint">
@@ -213,5 +224,6 @@
             <mechanicalReduction>0.2</mechanicalReduction>
             <mechanicalElasticity>1.0</mechanicalElasticity>
-            <hardwareInterface>PositionJointInterface</hardwareInterface>
+            <!-- hardwareInterface>PositionJointInterface</hardwareInterface -->
+            <hardwareInterface>EffortJointInterface</hardwareInterface>
           </joint>
           <joint name="${name}_ring_inner_joint">
@@ -220,5 +232,6 @@
             <mechanicalReduction>1.0</mechanicalReduction>
             <mechanicalElasticity>1.0</mechanicalElasticity>
-            <hardwareInterface>PositionJointInterface</hardwareInterface>
+            <!-- hardwareInterface>PositionJointInterface</hardwareInterface -->
+            <hardwareInterface>EffortJointInterface</hardwareInterface>
           </joint>
           <joint name="${name}_ring_middle_joint">
@@ -227,5 +240,6 @@
             <mechanicalReduction>1.0</mechanicalReduction>
             <mechanicalElasticity>1.0</mechanicalElasticity>
-            <hardwareInterface>PositionJointInterface</hardwareInterface>
+            <!-- hardwareInterface>PositionJointInterface</hardwareInterface -->
+            <hardwareInterface>EffortJointInterface</hardwareInterface>
           </joint>
           <joint name="${name}_ring_outer_joint">
@@ -234,5 +248,6 @@
             <mechanicalReduction>1.0</mechanicalReduction>
             <mechanicalElasticity>1.0</mechanicalElasticity>
-            <hardwareInterface>PositionJointInterface</hardwareInterface>
+            <!-- hardwareInterface>PositionJointInterface</hardwareInterface -->
+            <hardwareInterface>EffortJointInterface</hardwareInterface>
           </joint>
           <joint name="${name}_little_abd_joint">
@@ -241,5 +256,6 @@
             <mechanicalReduction>0.4</mechanicalReduction>
             <mechanicalElasticity>1.0</mechanicalElasticity>
-            <hardwareInterface>PositionJointInterface</hardwareInterface>
+            <!-- hardwareInterface>PositionJointInterface</hardwareInterface -->
+            <hardwareInterface>EffortJointInterface</hardwareInterface>
           </joint>
           <joint name="${name}_little_inner_joint">
@@ -248,5 +264,6 @@
             <mechanicalReduction>1.0</mechanicalReduction>
             <mechanicalElasticity>1.0</mechanicalElasticity>
-            <hardwareInterface>PositionJointInterface</hardwareInterface>
+            <!-- hardwareInterface>PositionJointInterface</hardwareInterface -->
+            <hardwareInterface>EffortJointInterface</hardwareInterface>
           </joint>
           <joint name="${name}_little_middle_joint">
@@ -255,5 +272,6 @@
             <mechanicalReduction>1.0</mechanicalReduction>
             <mechanicalElasticity>1.0</mechanicalElasticity>
-            <hardwareInterface>PositionJointInterface</hardwareInterface>
+            <!-- hardwareInterface>PositionJointInterface</hardwareInterface -->
+            <hardwareInterface>EffortJointInterface</hardwareInterface>
           </joint>
           <joint name="${name}_little_outer_joint">
@@ -262,9 +280,14 @@
             <mechanicalReduction>1.0</mechanicalReduction>
             <mechanicalElasticity>1.0</mechanicalElasticity>
-            <hardwareInterface>PositionJointInterface</hardwareInterface>
-          </joint>
+            <!-- hardwareInterface>PositionJointInterface</hardwareInterface -->
+            <hardwareInterface>EffortJointInterface</hardwareInterface>
+          </joint>
+          <!-- IMPORTANT: if you change the elasticity or reduction at the joints, this value must be calibrated again to
+                          ensure that the joints don't go after the limits -->
+          <!-- ToDO: autocalibration using the joint limits. When the synergy goes to 1, they must be at the upper limirt
+                    and to 0, they must be at the lower limit -->
           <actuator name="${name}_actuator">
             <role>actuator1</role>
-            <mechanicalReduction>0.1</mechanicalReduction>
+            <mechanicalReduction>4.5</mechanicalReduction>
           </actuator>
       </transmission>

File: soft_hand/soft_hand_description/robot/soft_hand_adaptive.urdf.xacro (robot description, xacro)
@@ -27,6 +27,7 @@
 		<origin xyz="0 0 1" rpy="1.570796 0 0"/>
 	</xacro:soft_hand>
+	<!-- a wall to test the adaptivity -->
 	<joint name="wrist_object_joint" type="fixed">
-		<origin xyz="0 0.05 1.1" rpy="0 0 0" />
+		<origin xyz="0 0.06 1.15" rpy="0 0 0" />
 		<parent link="wrist"/>
 		<child link="object"/>
@@ -39,5 +40,5 @@
 			<origin xyz="0 0 0" rpy="0 0 0"/>
 			<geometry>
-				<box size="0.05 0.05 0.05"/>
+				<box size="0.07 0.05 0.25"/>
 			</geometry>
 		</visual>
@@ -45,10 +46,9 @@
 			<origin xyz="0 0 0" rpy="0 0 0"/>
 			<geometry>
-				<box size="0.05 0.05 0.05"/>
+				<box size="0.07 0.05 0.25"/>
 			</geometry>
 		</collision>
 	</link>
 	<gazebo reference="object">
-		<static>true</static>
 		<selfCollide>True</selfCollide>
 	</gazebo>

Commit message: update

File: soft_hand/soft_hand_description/model/soft_hand.gazebo.xacro (robot description, xacro)
@@ -53,8 +53,8 @@
 					<frameName>${name}_palm_link</frameName>
 					<updateRate>100.0</updateRate>
-					<bumperTopicName>contacts/${name}_palm_link</bumperTopicName>
-				</plugin>
-			</sensor>
-			<!-- selfCollide>true</selfCollide -->
+					<bumperTopicName>/contacts/${name}_palm_link</bumperTopicName>
+				</plugin>
+			</sensor>
+			<!--selfCollide>true</selfCollide-->
 			<gravity>true</gravity>
 			<mu1>500.0</mu1>
@@ -77,8 +77,8 @@
 					<frameName>${name}_thumb_knuckle_link</frameName>
 					<updateRate>100.0</updateRate>
-					<bumperTopicName>contacts/${name}_thumb_knuckle_link</bumperTopicName>
-				</plugin>
-			</sensor>
-			<!-- selfCollide>true</selfCollide -->
+					<bumperTopicName>/contacts/${name}_thumb_knuckle_link</bumperTopicName>
+				</plugin>
+			</sensor>
+			<!--selfCollide>true</selfCollide-->
 			<gravity>true</gravity>
 			<mu1>500.0</mu1>
@@ -101,8 +101,8 @@
 					<frameName>${name}_thumb_proximal_link</frameName>
 					<updateRate>100.0</updateRate>
-					<bumperTopicName>contacts/${name}_thumb_proximal_link</bumperTopicName>
-				</plugin>
-			</sensor>
-			<!-- selfCollide>true</selfCollide -->
+					<bumperTopicName>/contacts/${name}_thumb_proximal_link</bumperTopicName>
+				</plugin>
+			</sensor>
+			<!--selfCollide>true</selfCollide-->
 			<gravity>true</gravity>
 			<mu1>500.0</mu1>
@@ -125,8 +125,8 @@
 					<frameName>${name}_thumb_distal_link</frameName>
 					<updateRate>100.0</updateRate>
-					<bumperTopicName>contacts/${name}_thumb_distal_link</bumperTopicName>
-				</plugin>
-			</sensor>
-			<!-- selfCollide>true</selfCollide -->
+					<bumperTopicName>/contacts/${name}_thumb_distal_link</bumperTopicName>
+				</plugin>
+			</sensor>
+			<!-- selfCollide>true</selfCollide-->
 			<gravity>true</gravity>
 			<mu1>500.0</mu1>
@@ -149,8 +149,8 @@
 					<frameName>${name}_index_knuckle_link</frameName>
 					<updateRate>100.0</updateRate>
-					<bumperTopicName>contacts/${name}_index_knuckle_link</bumperTopicName>
-				</plugin>
-			</sensor>
-			<!-- selfCollide>true</selfCollide -->
+					<bumperTopicName>/contacts/${name}_index_knuckle_link</bumperTopicName>
+				</plugin>
+			</sensor>
+			<!--selfCollide>true</selfCollide-->
 			<gravity>true</gravity>
 			<mu1>500.0</mu1>
@@ -173,8 +173,8 @@
 					<frameName>${name}_index_proximal_link</frameName>
 					<updateRate>100.0</updateRate>
-					<bumperTopicName>contacts/${name}_index_proximal_link</bumperTopicName>
-				</plugin>
-			</sensor>
-			<!-- selfCollide>true</selfCollide -->
+					<bumperTopicName>/contacts/${name}_index_proximal_link</bumperTopicName>
+				</plugin>
+			</sensor>
+			<!--selfCollide>true</selfCollide-->
 			<gravity>true</gravity>
 			<mu1>500.0</mu1>
@@ -197,8 +197,8 @@
 					<frameName>${name}_index_middle_link</frameName>
 					<updateRate>100.0</updateRate>
-					<bumperTopicName>contacts/${name}_index_middle_link</bumperTopicName>
-				</plugin>
-			</sensor>
-			<!-- selfCollide>true</selfCollide -->
+					<bumperTopicName>/contacts/${name}_index_middle_link</bumperTopicName>
+				</plugin>
+			</sensor>
+			<!--selfCollide>true</selfCollide-->
 			<gravity>true</gravity>
 			<mu1>500.0</mu1>
@@ -221,8 +221,8 @@
 					<frameName>${name}_index_distal_link</frameName>
 					<updateRate>100.0</updateRate>
-					<bumperTopicName>contacts/${name}_index_distal_link</bumperTopicName>
-				</plugin>
-			</sensor>
-			<!-- selfCollide>true</selfCollide -->
+					<bumperTopicName>/contacts/${name}_index_distal_link</bumperTopicName>
+				</plugin>
+			</sensor>
+			<!-- selfCollide>true</selfCollide-->
 			<gravity>true</gravity>
 			<mu1>500.0</mu1>
@@ -245,8 +245,8 @@
 					<frameName>${name}_middle_knuckle_link</frameName>
 					<updateRate>100.0</updateRate>
-					<bumperTopicName>contacts/${name}_middle_knuckle_link</bumperTopicName>
-				</plugin>
-			</sensor>
-			<!-- selfCollide>true</selfCollide -->
+					<bumperTopicName>/contacts/${name}_middle_knuckle_link</bumperTopicName>
+				</plugin>
+			</sensor>
+			<!--selfCollide>true</selfCollide-->
 			<gravity>true</gravity>
 			<mu1>500.0</mu1>
@@ -269,8 +269,8 @@
 					<frameName>${name}_middle_proximal_link</frameName>
 					<updateRate>100.0</updateRate>
-					<bumperTopicName>contacts/${name}_middle_proximal_link</bumperTopicName>
-				</plugin>
-			</sensor>
-			<!-- selfCollide>true</selfCollide -->
+					<bumperTopicName>/contacts/${name}_middle_proximal_link</bumperTopicName>
+				</plugin>
+			</sensor>
+			<!--selfCollide>true</selfCollide-->
 			<gravity>true</gravity>
 			<mu1>500.0</mu1>
@@ -293,8 +293,8 @@
 					<frameName>${name}_middle_middle_link</frameName>
 					<updateRate>100.0</updateRate>
-					<bumperTopicName>contacts/${name}_middle_middle_link</bumperTopicName>
-				</plugin>
-			</sensor>
-			<!-- selfCollide>true</selfCollide -->
+					<bumperTopicName>/contacts/${name}_middle_middle_link</bumperTopicName>
+				</plugin>
+			</sensor>
+			<!--selfCollide>true</selfCollide-->
 			<gravity>true</gravity>
 			<mu1>500.0</mu1>
@@ -317,8 +317,8 @@
 					<frameName>${name}_middle_distal_link</frameName>
 					<updateRate>100.0</updateRate>
-					<bumperTopicName>contacts/${name}_middle_distal_link</bumperTopicName>
-				</plugin>
-			</sensor>
-			<!-- selfCollide>true</selfCollide -->
+					<bumperTopicName>/contacts/${name}_middle_distal_link</bumperTopicName>
+				</plugin>
+			</sensor>
+			<!-- selfCollide>true</selfCollide-->
 			<gravity>true</gravity>
 			<mu1>500.0</mu1>
@@ -341,8 +341,8 @@
 					<frameName>${name}_ring_knuckle_link</frameName>
 					<updateRate>100.0</updateRate>
-					<bumperTopicName>contacts/${name}_ring_knuckle_link</bumperTopicName>
-				</plugin>
-			</sensor>
-			<!-- selfCollide>true</selfCollide -->
+					<bumperTopicName>/contacts/${name}_ring_knuckle_link</bumperTopicName>
+				</plugin>
+			</sensor>
+			<!--selfCollide>true</selfCollide-->
 			<gravity>true</gravity>
 			<mu1>500.0</mu1>
@@ -365,8 +365,8 @@
 					<frameName>${name}_ring_proximal_link</frameName>
 					<updateRate>100.0</updateRate>
-					<bumperTopicName>contacts/${name}_ring_proximal_link</bumperTopicName>
-				</plugin>
-			</sensor>
-			<!-- selfCollide>true</selfCollide -->
+					<bumperTopicName>/contacts/${name}_ring_proximal_link</bumperTopicName>
+				</plugin>
+			</sensor>
+			<!--selfCollide>true</selfCollide-->
 			<gravity>true</gravity>
 			<mu1>500.0</mu1>
@@ -389,8 +389,8 @@
 					<frameName>${name}_ring_middle_link</frameName>
 					<updateRate>100.0</updateRate>
-					<bumperTopicName>contacts/${name}_ring_middle_link</bumperTopicName>
-				</plugin>
-			</sensor>
-			<!-- selfCollide>true</selfCollide -->
+					<bumperTopicName>/contacts/${name}_ring_middle_link</bumperTopicName>
+				</plugin>
+			</sensor>
+			<!--selfCollide>true</selfCollide-->
 			<gravity>true</gravity>
 			<mu1>500.0</mu1>
@@ -413,8 +413,8 @@
 					<frameName>${name}_ring_distal_link</frameName>
 					<updateRate>100.0</updateRate>
-					<bumperTopicName>contacts/${name}_ring_distal_link</bumperTopicName>
-				</plugin>
-			</sensor>
-			<!-- selfCollide>true</selfCollide -->
+					<bumperTopicName>/contacts/${name}_ring_distal_link</bumperTopicName>
+				</plugin>
+			</sensor>
+			<!-- selfCollide>true</selfCollide-->
 			<gravity>true</gravity>
 			<mu1>500.0</mu1>
@@ -437,8 +437,8 @@
 					<frameName>${name}_little_knuckle_link</frameName>
 					<updateRate>100.0</updateRate>
-					<bumperTopicName>contacts/${name}_little_knuckle_link</bumperTopicName>
-				</plugin>
-			</sensor>
-			<!-- selfCollide>true</selfCollide -->
+					<bumperTopicName>/contacts/${name}_little_knuckle_link</bumperTopicName>
+				</plugin>
+			</sensor>
+			<!--selfCollide>true</selfCollide-->
 			<gravity>true</gravity>
 			<mu1>500.0</mu1>
@@ -461,8 +461,8 @@
 					<frameName>${name}_little_proximal_link</frameName>
 					<updateRate>100.0</updateRate>
-					<bumperTopicName>contacts/${name}_little_proximal_link</bumperTopicName>
-				</plugin>
-			</sensor>
-			<!-- selfCollide>true</selfCollide -->
+					<bumperTopicName>/contacts/${name}_little_proximal_link</bumperTopicName>
+				</plugin>
+			</sensor>
+			<!--selfCollide>true</selfCollide-->
 			<gravity>true</gravity>
 			<mu1>500.0</mu1>
@@ -485,8 +485,8 @@
 					<frameName>${name}_little_middle_link</frameName>
 					<updateRate>100.0</updateRate>
-					<bumperTopicName>contacts/${name}_little_middle_link</bumperTopicName>
-				</plugin>
-			</sensor>
-			<!-- selfCollide>true</selfCollide -->
+					<bumperTopicName>/contacts/${name}_little_middle_link</bumperTopicName>
+				</plugin>
+			</sensor>
+			<!--selfCollide>true</selfCollide-->
 			<gravity>true</gravity>
 			<mu1>500.0</mu1>
@@ -509,8 +509,8 @@
 					<frameName>${name}_little_distal_link</frameName>
 					<updateRate>100.0</updateRate>
-					<bumperTopicName>contacts/${name}_little_distal_link</bumperTopicName>
-				</plugin>
-			</sensor>
-			<!-- selfCollide>true</selfCollide -->
+					<bumperTopicName>/contacts/${name}_little_distal_link</bumperTopicName>
+				</plugin>
+			</sensor>
+			<!-- selfCollide>true</selfCollide-->
 			<gravity>true</gravity>
 			<mu1>500.0</mu1>

File: soft_hand/soft_hand_description/robot/soft_hand_adaptive.urdf.xacro (robot description, xacro)
@@ -26,29 +26,3 @@
 		<origin xyz="0.0 0.0 1.02" rpy="0 0 0"/>
 	</xacro:soft_hand>
-	<!-- a wall to test the adaptivity
-	<joint name="box_object_joint" type="fixed">
-		<origin xyz="0.06 0 1.15" rpy="0 0 0" />
-		<parent link="box"/>
-		<child link="object"/>
-	</joint>
-	<link name="object">
-		<inertial>
-			<mass value="50.0"/>
-			<inertia  ixx="1" ixy="0.00"  ixz="0.00" iyy="1" iyz="0.00" izz="1" />
-		</inertial>
-		<visual>
-			<geometry>
-				<box size="0.05 0.07 0.25"/>
-			</geometry>
-		</visual>
-		<collision>
-			<geometry>
-				<box size="0.05 0.07 0.25"/>
-			</geometry>
-		</collision>
-	</link>
-	<gazebo reference="object">
-		<selfCollide>True</selfCollide>
-	</gazebo>
-	-->
 </robot>
