Commit message: modified the synergy joint to allow multiple instances of the hand, always right hand

File: soft_hand/soft_hand_description/model/soft_hand.transmission.xacro (robot description, xacro)
@@ -122,5 +122,5 @@
       <transmission name="synergy_trans">
           <type>transmission_interface/SimpleTransmission</type>
-          <joint name="synergy_joint">
+          <joint name="${name}_synergy_joint">
             <hardwareInterface>EffortJointInterface</hardwareInterface>
           </joint>

File: soft_hand/soft_hand_description/model/soft_hand.urdf.xacro (robot description, xacro)
@@ -55,5 +55,5 @@
 	<!-- SOFT FINGER model -->
 	<!-- 4 fingers are equal (index, middle, ring, little) -->
-	<xacro:macro name="soft_finger" params="parent name position orientation useMimicTag abd_R inner_R middle_R outer_R">
+	<xacro:macro name="soft_finger" params="parent parent_name name position orientation useMimicTag abd_R inner_R middle_R outer_R">
 		<!-- KNUCKLE -->
 		<joint name="${name}_abd_joint" type="revolute">
@@ -65,5 +65,5 @@
 			<dynamics damping="${damping}" friction="${friction}"/>
 			<xacro:if value="${useMimicTag}">
-				<mimic joint="synergy_joint" multiplier="${abd_R}"/>
+				<mimic joint="${parent_name}_synergy_joint" multiplier="${abd_R}"/>
 			</xacro:if>
 		</joint>
@@ -96,5 +96,5 @@
 			<dynamics damping="${damping}" friction="${friction}"/>
 			<xacro:if value="${useMimicTag}">
-				<mimic joint="synergy_joint" multiplier="${inner_R}"/>
+				<mimic joint="${parent_name}_synergy_joint" multiplier="${inner_R}"/>
 			</xacro:if>
 		</joint>
@@ -112,5 +112,5 @@
 			<dynamics damping="${damping}" friction="${friction}"/>
 			<xacro:if value="${useMimicTag}">
-				<mimic joint="synergy_joint" multiplier="${inner_R}" />
+				<mimic joint="${parent_name}_synergy_joint" multiplier="${inner_R}" />
 			</xacro:if>
 		</joint>
@@ -143,5 +143,5 @@
 			<dynamics damping="${damping}" friction="${friction}"/>
 			<xacro:if value="${useMimicTag}">
-				<mimic joint="synergy_joint" multiplier="${middle_R}"/>
+				<mimic joint="${parent_name}_synergy_joint" multiplier="${middle_R}"/>
 			</xacro:if>
 		</joint>
@@ -159,5 +159,5 @@
 			<dynamics damping="${damping}" friction="${friction}"/>
 			<xacro:if value="${useMimicTag}">
-				<mimic joint="synergy_joint" multiplier="${middle_R}"/>
+				<mimic joint="${parent_name}_synergy_joint" multiplier="${middle_R}"/>
 			</xacro:if>
 		</joint>
@@ -188,5 +188,5 @@
 			<dynamics damping="${damping}" friction="${friction}"/>
 			<xacro:if value="${useMimicTag}">
-				<mimic joint="synergy_joint" multiplier="${outer_R}"/>
+				<mimic joint="${parent_name}_synergy_joint" multiplier="${outer_R}"/>
 			</xacro:if>
 		</joint>
@@ -204,5 +204,5 @@
 			<dynamics damping="${damping}" friction="${friction}"/>
 			<xacro:if value="${useMimicTag}">
-				<mimic joint="synergy_joint" multiplier="${outer_R}"/>
+				<mimic joint="${parent_name}_synergy_joint" multiplier="${outer_R}"/>
 			</xacro:if>
 		</joint>
@@ -227,5 +227,5 @@
 	<!-- THUMB MODEL -->
 	<!-- It has one joint less than rest of fingers -->
-	<xacro:macro name="soft_thumb" params="parent name position orientation useMimicTag abd_R inner_R outer_R">
+	<xacro:macro name="soft_thumb" params="parent parent_name name position orientation useMimicTag abd_R inner_R outer_R">
 		<!-- KNUCKLE -->
 		<joint name="${name}_abd_joint" type="revolute">
@@ -237,5 +237,5 @@
 			<dynamics damping="${damping}" friction="${friction}"/>
 			<xacro:if value="${useMimicTag}">
-				<mimic joint="synergy_joint" multiplier="${abd_R}"/>
+				<mimic joint="${parent_name}_synergy_joint" multiplier="${abd_R}"/>
 			</xacro:if>
 		</joint>
@@ -266,5 +266,5 @@
 			<dynamics damping="${damping}" friction="${friction}"/>
 			<xacro:if value="${useMimicTag}">
-				<mimic joint="synergy_joint" multiplier="${inner_R}"/>
+				<mimic joint="${parent_name}_synergy_joint" multiplier="${inner_R}"/>
 			</xacro:if>
 		</joint>
@@ -282,5 +282,5 @@
 			<dynamics damping="${damping}" friction="${friction}"/>
 			<xacro:if value="${useMimicTag}">
-				<mimic joint="synergy_joint" multiplier="${inner_R}" />
+				<mimic joint="${parent_name}_synergy_joint" multiplier="${inner_R}" />
 			</xacro:if>
 		</joint>
@@ -311,5 +311,5 @@
 			<dynamics damping="${damping}" friction="${friction}"/>
 			<xacro:if value="${useMimicTag}">
-				<mimic joint="synergy_joint" multiplier="${outer_R}"/>
+				<mimic joint="${parent_name}_synergy_joint" multiplier="${outer_R}"/>
 			</xacro:if>
 		</joint>
@@ -327,5 +327,5 @@
 			<dynamics damping="${damping}" friction="${friction}"/>
 			<xacro:if value="${useMimicTag}">
-				<mimic joint="synergy_joint" multiplier="${outer_R}" />
+				<mimic joint="${parent_name}_synergy_joint" multiplier="${outer_R}" />
 			</xacro:if>
 		</joint>
@@ -351,12 +351,12 @@
 	<xacro:macro name="soft_hand" params="parent name withAdaptiveTransmission useMimicTag *origin">
 		<!-- MOTOR JOINT -->
-		<joint name="synergy_joint" type="revolute" >
+		<joint name="${name}_synergy_joint" type="revolute" >
 			<parent link="${parent}" />
-			<child link="invisible_wire_link"/>
+			<child link="${name}_invisible_wire_link"/>
 			<axis xyz="0 0 1" />
 			<limit lower="${synergy_lb}" upper="${synergy_ub}" effort="${max_synergy_effort}" velocity="${max_synergy_velocity}"/>
 			<dynamics damping="${synergy_damping}" friction="${synergy_friction}"/>
 		</joint>
-		<link name="invisible_wire_link">
+		<link name="${name}_invisible_wire_link">
 			<inertial>
 				<insert_block name="negligible_inertia"/>
@@ -387,9 +387,9 @@
 		</link>
 		<!-- THUMB AND FINGERS -->
-		<xacro:soft_thumb parent="${name}_palm_link" name="${name}_thumb" position="-0.0418769 0.0538740 -0.00691972" orientation="0 0 -0.43633181" useMimicTag="${useMimicTag}" abd_R="${thumb_abd_R *(thumb_abd_ub - thumb_abd_lb)*pi/180}" inner_R="${thumb_inner_R *(inner_ub - inner_lb)*pi/180}" outer_R="${thumb_outer_R *(outer_ub - outer_lb)*pi/180}"/>
-		<xacro:soft_finger parent="${name}_palm_link" name="${name}_index" position="-0.0285 0.0943918 0.00205" orientation="${180*pi/180} 0 ${(-90+20)*pi/180}" useMimicTag="${useMimicTag}" abd_R="${index_abd_R}" inner_R="${index_inner_R *(inner_ub - inner_lb)*pi/180}" middle_R="${index_middle_R *(middle_ub - middle_lb)*pi/180}" outer_R="${index_outer_R *(outer_ub - outer_lb)*pi/180}" />
-		<xacro:soft_finger parent="${name}_palm_link" name="${name}_middle" position="-0.009 0.107892 0.00205" orientation="${180*pi/180} 0 ${-90*pi/180}" useMimicTag="${useMimicTag}" abd_R="${middle_abd_R}" inner_R="${middle_inner_R *(inner_ub - inner_lb)*pi/180}" middle_R="${middle_middle_R *(middle_ub - middle_lb)*pi/180}" outer_R="${middle_outer_R *(outer_ub - outer_lb)*pi/180}" />
-		<xacro:soft_finger parent="${name}_palm_link" name="${name}_ring" position="0.0105 0.0943918 0.00205" orientation="${180*pi/180} 0 ${(-90-10)*pi/180}" useMimicTag="${useMimicTag}" abd_R="${ring_abd_R}" inner_R="${ring_inner_R *(inner_ub - inner_lb)*pi/180}" middle_R="${ring_middle_R *(middle_ub - middle_lb)*pi/180}" outer_R="${ring_outer_R *(outer_ub - outer_lb)*pi/180}" />
-		<xacro:soft_finger parent="${name}_palm_link" name="${name}_little" position="0.030 0.0808918 0.00205" orientation="${180*pi/180} 0 ${(-90-20)*pi/180}" useMimicTag="${useMimicTag}" abd_R="${little_abd_R}" inner_R="${little_inner_R *(inner_ub - inner_lb)*pi/180}" middle_R="${little_middle_R *(middle_ub - middle_lb)*pi/180}" outer_R="${little_outer_R *(outer_ub - outer_lb)*pi/180}" />
+		<xacro:soft_thumb parent="${name}_palm_link" parent_name="${name}" name="${name}_thumb" position="-0.0418769 0.0538740 -0.00691972" orientation="0 0 -0.43633181" useMimicTag="${useMimicTag}" abd_R="${thumb_abd_R *(thumb_abd_ub - thumb_abd_lb)*pi/180}" inner_R="${thumb_inner_R *(inner_ub - inner_lb)*pi/180}" outer_R="${thumb_outer_R *(outer_ub - outer_lb)*pi/180}"/>
+		<xacro:soft_finger parent="${name}_palm_link" parent_name="${name}" name="${name}_index" position="-0.0285 0.0943918 0.00205" orientation="${180*pi/180} 0 ${(-90+20)*pi/180}" useMimicTag="${useMimicTag}" abd_R="${index_abd_R}" inner_R="${index_inner_R *(inner_ub - inner_lb)*pi/180}" middle_R="${index_middle_R *(middle_ub - middle_lb)*pi/180}" outer_R="${index_outer_R *(outer_ub - outer_lb)*pi/180}" />
+		<xacro:soft_finger parent="${name}_palm_link" parent_name="${name}" name="${name}_middle" position="-0.009 0.107892 0.00205" orientation="${180*pi/180} 0 ${-90*pi/180}" useMimicTag="${useMimicTag}" abd_R="${middle_abd_R}" inner_R="${middle_inner_R *(inner_ub - inner_lb)*pi/180}" middle_R="${middle_middle_R *(middle_ub - middle_lb)*pi/180}" outer_R="${middle_outer_R *(outer_ub - outer_lb)*pi/180}" />
+		<xacro:soft_finger parent="${name}_palm_link" parent_name="${name}" name="${name}_ring" position="0.0105 0.0943918 0.00205" orientation="${180*pi/180} 0 ${(-90-10)*pi/180}" useMimicTag="${useMimicTag}" abd_R="${ring_abd_R}" inner_R="${ring_inner_R *(inner_ub - inner_lb)*pi/180}" middle_R="${ring_middle_R *(middle_ub - middle_lb)*pi/180}" outer_R="${ring_outer_R *(outer_ub - outer_lb)*pi/180}" />
+		<xacro:soft_finger parent="${name}_palm_link" parent_name="${name}" name="${name}_little" position="0.030 0.0808918 0.00205" orientation="${180*pi/180} 0 ${(-90-20)*pi/180}" useMimicTag="${useMimicTag}" abd_R="${little_abd_R}" inner_R="${little_inner_R *(inner_ub - inner_lb)*pi/180}" middle_R="${little_middle_R *(middle_ub - middle_lb)*pi/180}" outer_R="${little_outer_R *(outer_ub - outer_lb)*pi/180}" />
 		<xacro:soft_hand_transmission name="${name}" withAdaptiveTransmission="${withAdaptiveTransmission}"/>
 		<xacro:soft_hand_gazebo name="${name}" withAdaptiveTransmission="${withAdaptiveTransmission}" useMimicTag="${useMimicTag}"/>

Commit message: Update to allow multi-robots in gazebo

File: soft_hand/soft_hand_description/model/soft_hand.transmission.xacro (robot description, xacro)
@@ -2,5 +2,6 @@
 <robot name="robot" xmlns:xacro="http://www.ros.org/wiki/xacro">
     <xacro:macro name="finger_transmission" params="name finger">
-      <transmission name="${name}_${finger}_abd_trans">
+        <transmission name="${name}_${finger}_abd_trans">
+        <robotNamespace>${name}</robotNamespace>
         <type>transmission_interface/SimpleTransmission</type>
         <joint name="${name}_${finger}_abd_joint">
@@ -12,4 +13,5 @@
         </transmission>
         <transmission name="${name}_${finger}_inner_trans">
+        <robotNamespace>${name}</robotNamespace>
         <type>transmission_interface/SimpleTransmission</type>
         <joint name="${name}_${finger}_inner_joint">
@@ -21,4 +23,5 @@
         </transmission>
         <transmission name="${name}_${finger}_inner_mimic_trans">
+        <robotNamespace>${name}</robotNamespace>
         <type>transmission_interface/SimpleTransmission</type>
         <joint name="${name}_${finger}_inner_joint_mimic">
@@ -30,4 +33,5 @@
         </transmission>
         <transmission name="${name}_${finger}_middle_trans">
+        <robotNamespace>${name}</robotNamespace>
         <type>transmission_interface/SimpleTransmission</type>
         <joint name="${name}_${finger}_middle_joint">
@@ -39,4 +43,5 @@
         </transmission>
         <transmission name="${name}_${finger}_middle_mimic_trans">
+        <robotNamespace>${name}</robotNamespace>
         <type>transmission_interface/SimpleTransmission</type>
         <joint name="${name}_${finger}_middle_joint_mimic">
@@ -48,4 +53,5 @@
         </transmission>
         <transmission name="${name}_${finger}_outer_trans">
+        <robotNamespace>${name}</robotNamespace>
         <type>transmission_interface/SimpleTransmission</type>
         <joint name="${name}_${finger}_outer_joint">
@@ -57,4 +63,5 @@
         </transmission>
         <transmission name="${name}_${finger}_outer_mimic_trans">
+        <robotNamespace>${name}</robotNamespace>
         <type>transmission_interface/SimpleTransmission</type>
         <joint name="${name}_${finger}_outer_joint_mimic">
@@ -69,4 +76,5 @@
     <xacro:unless value="${withAdaptiveTransmission}">
       <transmission name="${name}_thumb_abd_trans">
+          <robotNamespace>${name}</robotNamespace>
           <type>transmission_interface/SimpleTransmission</type>
           <joint name="${name}_thumb_abd_joint">
@@ -78,4 +86,5 @@
       </transmission>
       <transmission name="${name}_thumb_inner_trans">
+          <robotNamespace>${name}</robotNamespace>
           <type>transmission_interface/SimpleTransmission</type>
           <joint name="${name}_thumb_inner_joint">
@@ -87,4 +96,5 @@
       </transmission>
       <transmission name="${name}_thumb_inner_mimic_trans">
+          <robotNamespace>${name}</robotNamespace>
           <type>transmission_interface/SimpleTransmission</type>
           <joint name="${name}_thumb_inner_joint_mimic">
@@ -96,4 +106,5 @@
       </transmission>
       <transmission name="${name}_thumb_outer_trans">
+          <robotNamespace>${name}</robotNamespace>
           <type>transmission_interface/SimpleTransmission</type>
           <joint name="${name}_thumb_outer_joint">
@@ -105,4 +116,5 @@
       </transmission>
       <transmission name="${name}_thumb_outer_mimic_trans">
+          <robotNamespace>${name}</robotNamespace>
           <type>transmission_interface/SimpleTransmission</type>
           <joint name="${name}_thumb_outer_joint_mimic">
@@ -121,4 +133,5 @@
       <!-- work in progress -->
       <transmission name="${name}_synergy_trans">
+          <robotNamespace>${name}</robotNamespace>
           <type>transmission_interface/SimpleTransmission</type>
           <joint name="${name}_synergy_joint">
@@ -130,4 +143,5 @@
       </transmission>
       <transmission name="${name}_joint_trans">
+        <robotNamespace>${name}</robotNamespace>
         <type>transmission_interface/AdaptiveSynergyTransmission</type>
           <joint name="${name}_thumb_abd_joint">

File: soft_hand/soft_hand_description/model/soft_hand.urdf.xacro (robot description, xacro)
@@ -27,5 +27,5 @@
 	<xacro:property name="friction" value="0.0" />
 	<!-- synergy vector -->
-	<xacro:property name="syn_amp" value="0.00005555555" /> <!-- 1/18000 -->
+	<xacro:property name="syn_amp" value="1.0"/> <!--0.00005555555" /--> <!-- 1/18000 -->
 	<xacro:property name="thumb_abd_R" value="${1.3*syn_amp}" />
 	<xacro:property name="thumb_inner_R" value="${1.3*syn_amp}" />
@@ -49,5 +49,5 @@
 	<!-- synergy joint properties -->
 	<xacro:property name="synergy_lb" value="0.0" />
-	<xacro:property name="synergy_ub" value="18000.0" />
+	<xacro:property name="synergy_ub" value="1.0"/> <!--18000.0" /-->
 	<xacro:property name="max_synergy_velocity" value="10000" />
 	<xacro:property name="max_synergy_effort" value="100" />

File: soft_hand/soft_hand_description/objects/object.urdf.xacro (robot description, xacro)
@@ -19,6 +19,6 @@
 	</link>
 	<gazebo reference="object">
-		<selfCollide>True</selfCollide>
-		<static>true</static>
+		<!-- <selfCollide>True</selfCollide>
+		<static>true</static> -->
 	</gazebo>
 </robot>
