Commit message: soft hand full actuation model in gazebo, see readme for details

File: soft_hand/soft_hand_description/model/soft_hand.urdf.xacro (robot description, xacro)
@@ -2,7 +2,13 @@
 <robot xmlns:xacro="http://ros.org/wiki/xacro">
 	<xacro:include filename="$(find soft_hand_description)/model/materials.urdf.xacro"/>
+	<xacro:include filename="$(find soft_hand_description)/model/soft_hand.transmission.xacro"/>
+	<xacro:include filename="$(find soft_hand_description)/model/soft_hand.gazebo.xacro"/>
+	<xacro:include filename="$(find soft_hand_description)/model/soft_hand.inertias.xacro"/>
 	<xacro:property name="pi" value="3.1415926535897931" />
+	<!-- joint properties -->
 	<xacro:property name="abd_lb" value="-30" />
 	<xacro:property name="abd_ub" value="30" />
+	<xacro:property name="thumb_abd_lb" value="0" />
+	<xacro:property name="thumb_abd_ub" value="90" />
 	<xacro:property name="inner_lb" value="0" />
 	<xacro:property name="inner_ub" value="45" />
@@ -13,4 +19,14 @@
 	<xacro:property name="velocity" value="100" />
 	<xacro:property name="effort" value="100" />
+	<xacro:property name="damping" value="0.0" />
+	<xacro:property name="friction" value="0.0" />
+	<!-- actuator properties -->
+	<xacro:property name="actuator_lb" value="0" />
+	<xacro:property name="actuator_ub" value="359" />
+	<xacro:property name="max_actuator_velocity" value="100" />
+	<xacro:property name="max_actuator_effort" value="100" />
+	<xacro:property name="actuator_damping" value="0.0" />
+	<xacro:property name="actuator_friction" value="0.0" />
+	<!-- HAND MODEL v.? Material: ABS -->
 	<!-- SOFT FINGER model -->
 	<!-- 4 fingers are equal (index, middle, ring, little) -->
@@ -23,6 +39,10 @@
 			<axis xyz="0 0 1" />
 			<limit lower="${abd_lb *pi/180}" upper="${inner_ub *pi/180}" effort="${effort}" velocity="${velocity}"/>
+			<dynamics damping="${damping}" friction="${friction}"/>
 		</joint>
 		<link name="${name}_knuckle_link">
+			<inertial>
+				<insert_block name="knuckle_inertia"/>
+			</inertial>
 			<visual>
 				<origin xyz="0 0 0" rpy="0 0 0" />
@@ -32,4 +52,11 @@
 				<material name="SoftHand/DarkGolden" />
 			</visual>
+			<collision>
+				<!-- origin xyz="-0.001 0.0 0.001" rpy="0 0 0" /-->
+				<geometry>
+					<!-- box size="0.034 0.014 0.024"/-->
+					<mesh filename="package://soft_hand_description/meshes/knuckle.stl" scale=" .001 .001 .001" />
+				</geometry>
+			</collision>
 		</link>
 		<!-- PROXIMAL PHALANGE -->
@@ -40,6 +67,10 @@
 			<axis xyz="0 1 0" />
 			<limit lower="${inner_lb *pi/180}" upper="${inner_ub *pi/180}" effort="${effort}" velocity="${velocity}"/>
+			<dynamics damping="${damping}" friction="${friction}"/>
 		</joint>
 		<link name="${name}_fake_link1">
+			<inertial>
+				<insert_block name="negligible_inertia"/>
+			</inertial>
 		</link>
 		<joint name="${name}_inner_joint_mimic" type="revolute">
@@ -50,13 +81,24 @@
 			<mimic joint="${name}_inner_joint" multiplier="1" />
 			<limit lower="${middle_lb *pi/180}" upper="${middle_ub *pi/180}" effort="${effort}" velocity="${velocity}"/>
+			<dynamics damping="${damping}" friction="${friction}"/>
 		</joint>
 		<link name="${name}_proximal_link">
-			<visual>
-				<origin xyz="0 0 0" rpy="0 0 0" />
-				<geometry>
-					<mesh filename="package://soft_hand_description/meshes/short_link.stl" scale=" .001 .001 .001" />
-				</geometry>
-				<material name="SoftHand/DarkGolden" />
-			</visual>
+			<inertial>
+				<insert_block name="phalanx_inertia"/>
+			</inertial>
+			<visual>
+				<origin xyz="0 0 0" rpy="0 0 0" />
+				<geometry>
+					<mesh filename="package://soft_hand_description/meshes/phalanx.stl" scale=" .001 .001 .001" />
+				</geometry>
+				<material name="SoftHand/DarkGolden" />
+			</visual>
+			<collision>
+				<!-- origin xyz="-0.005 0.0 0.0 " rpy="0 0 0" /-->
+				<geometry>
+					<!-- box size="0.025 0.014 0.019"/-->
+					<mesh filename="package://soft_hand_description/meshes/phalanx.stl" scale=" .001 .001 .001" />
+				</geometry>
+			</collision>
 		</link>
 		<!-- MIDDLE PHALANGE -->
@@ -67,6 +109,10 @@
 			<axis xyz="0 1 0" />
 			<limit lower="${inner_lb *pi/180}" upper="${inner_ub *pi/180}" effort="${effort}" velocity="${velocity}"/>
+			<dynamics damping="${damping}" friction="${friction}"/>
 		</joint>
 		<link name="${name}_fake_link2">
+			<inertial>
+				<insert_block name="negligible_inertia"/>
+			</inertial>
 		</link>
 		<joint name="${name}_middle_joint_mimic" type="revolute">
@@ -77,13 +123,22 @@
 			<mimic joint="${name}_middle_joint" multiplier="1" />
 			<limit lower="${outer_lb *pi/180}" upper="${outer_ub *pi/180}" effort="${effort}" velocity="${velocity}"/>
+			<dynamics damping="${damping}" friction="${friction}"/>
 		</joint>
 		<link name="${name}_middle_link">
-			<visual>
-				<origin xyz="0 0 0" rpy="0 0 0" />
-				<geometry>
-					<mesh filename="package://soft_hand_description/meshes/short_link.stl" scale=" .001 .001 .001" />
-				</geometry>
-				<material name="SoftHand/DarkGolden" />
-			</visual>
+			<inertial>
+				<insert_block name="phalanx_inertia"/>
+			</inertial>
+			<visual>
+				<origin xyz="0 0 0" rpy="0 0 0" />
+				<geometry>
+					<mesh filename="package://soft_hand_description/meshes/phalanx.stl" scale=" .001 .001 .001" />
+				</geometry>
+				<material name="SoftHand/DarkGolden" />
+			</visual>
+			<collision>
+				<geometry>
+					<mesh filename="package://soft_hand_description/meshes/phalanx.stl" scale=" .001 .001 .001" />
+				</geometry>
+			</collision>
 		</link>
 		<!-- DISTAL PHALANGE -->
@@ -94,6 +149,10 @@
 			<axis xyz="0 1 0" />
 			<limit lower="${inner_lb *pi/180}" upper="${inner_ub *pi/180}" effort="${effort}" velocity="${velocity}"/>
+			<dynamics damping="${damping}" friction="${friction}"/>
 		</joint>
 		<link name="${name}_fake_link3">
+			<inertial>
+				<insert_block name="negligible_inertia"/>
+			</inertial>
 		</link>
 		<joint name="${name}_outer_joint_mimic" type="revolute">
@@ -104,6 +163,10 @@
 			<mimic joint="${name}_outer_joint" multiplier="1" />
 			<limit lower="${inner_lb *pi/180}" upper="${inner_ub *pi/180}" effort="${effort}" velocity="${velocity}"/>
+			<dynamics damping="${damping}" friction="${friction}"/>
 		</joint>
 		<link name="${name}_distal_link">
+			<inertial>
+				<insert_block name="fingertip_inertia"/>
+			</inertial>
 			<visual>
 				<origin xyz="0 0 0" rpy="0 0 0" />
@@ -113,7 +176,13 @@
 				<material name="SoftHand/DarkGolden" />
 			</visual>
+			<collision>
+				<geometry>
+					<mesh filename="package://soft_hand_description/meshes/fingertip.stl" scale=" .001 .001 .001" />
+				</geometry>
+			</collision>
 		</link>
 	</xacro:macro>
-	<!-- THUMB has one joint less -->
+	<!-- THUMB MODEL -->
+	<!-- It has one joint less than rest of fingers -->
 	<xacro:macro name="soft_thumb" params="parent name position orientation">
 		<!-- KNUCKLE -->
@@ -122,8 +191,12 @@
 			<parent link="${parent}"/>
 			<child link="${name}_knuckle_link"/>
-			<axis xyz="0 1 0" />
-			<limit lower="${-2*inner_ub *pi/180}" upper="${inner_lb *pi/180}" effort="${effort}" velocity="${velocity}"/>
+			<axis xyz="0 -1 0" />
+			<limit lower="${thumb_abd_lb *pi/180}" upper="${thumb_abd_ub *pi/180}" effort="${effort}" velocity="${velocity}"/>
+			<dynamics damping="${damping}" friction="${friction}"/>
 		</joint>
 		<link name="${name}_knuckle_link">
+			<inertial>
+				<insert_block name="thumb_knuckle_inertia"/>
+			</inertial>
 			<visual>
 				<origin xyz="0 0 0" rpy="0 0 0" />
@@ -133,4 +206,9 @@
 				<material name="SoftHand/DarkGolden" />
 			</visual>
+			<collision>
+				<geometry>
+					<mesh filename="package://soft_hand_description/meshes/thumb_knuckle.stl" scale=" .001 .001 .001" />
+				</geometry>
+			</collision>
 		</link>
 		<!-- PROXIMAL PHALANGE -->
@@ -138,26 +216,39 @@
 			<origin xyz="-0.0225 0 -0.0033" rpy="-1.9974238811 0 0" />
 			<parent link="${name}_knuckle_link"/>
-			<child link="${name}_inner_link"/>
-			<axis xyz="0 1 0" />
-			<limit lower="${inner_lb *pi/180}" upper="${inner_ub *pi/180}" effort="${effort}" velocity="${velocity}"/>
-		</joint>
-		<link name="${name}_inner_link">
+			<child link="${name}_fake_link1"/>
+			<axis xyz="0 1 0" />
+			<limit lower="${inner_lb *pi/180}" upper="${inner_ub *pi/180}" effort="${effort}" velocity="${velocity}"/>
+			<dynamics damping="${damping}" friction="${friction}"/>
+		</joint>
+		<link name="${name}_fake_link1">
+			<inertial>
+				<insert_block name="negligible_inertia"/>
+			</inertial>
 		</link>
 		<joint name="${name}_inner_joint_mimic" type="revolute">
 			<origin xyz="-0.013 0 0" rpy="0 0 0" />
-			<parent link="${name}_inner_link"/>
+			<parent link="${name}_fake_link1"/>
 			<child link="${name}_proximal_link"/>
 			<axis xyz="0 1 0" />
 			<mimic joint="${name}_inner_joint" multiplier="1" />
 			<limit lower="${middle_lb *pi/180}" upper="${middle_ub *pi/180}" effort="${effort}" velocity="${velocity}"/>
+			<dynamics damping="${damping}" friction="${friction}"/>
 		</joint>
 		<link name="${name}_proximal_link">
-			<visual>
-				<origin xyz="0 0 0" rpy="0 0 0" />
-				<geometry>
-					<mesh filename="package://soft_hand_description/meshes/short_link.stl" scale=" .001 .001 .001" />
-				</geometry>
-				<material name="SoftHand/DarkGolden" />
-			</visual>
+			<inertial>
+				<insert_block name="phalanx_inertia"/>
+			</inertial>
+			<visual>
+				<origin xyz="0 0 0" rpy="0 0 0" />
+				<geometry>
+					<mesh filename="package://soft_hand_description/meshes/phalanx.stl" scale=" .001 .001 .001" />
+				</geometry>
+				<material name="SoftHand/DarkGolden" />
+			</visual>
+			<collision>
+				<geometry>
+					<mesh filename="package://soft_hand_description/meshes/phalanx.stl" scale=" .001 .001 .001" />
+				</geometry>
+			</collision>
 		</link>
 		<!-- DISTAL PHALANGE -->
@@ -168,6 +259,10 @@
 			<axis xyz="0 1 0" />
 			<limit lower="${inner_lb *pi/180}" upper="${inner_ub *pi/180}" effort="${effort}" velocity="${velocity}"/>
+			<dynamics damping="${damping}" friction="${friction}"/>
 		</joint>
 		<link name="${name}_fake_link3">
+			<inertial>
+				<insert_block name="negligible_inertia"/>
+			</inertial>
 		</link>
 		<joint name="${name}_outer_joint_mimic" type="revolute">
@@ -178,6 +273,10 @@
 			<mimic joint="${name}_outer_joint" multiplier="1" />
 			<limit lower="${inner_lb *pi/180}" upper="${inner_ub *pi/180}" effort="${effort}" velocity="${velocity}"/>
+			<dynamics damping="${damping}" friction="${friction}"/>
 		</joint>
 		<link name="${name}_distal_link">
+			<inertial>
+				<insert_block name="fingertip_inertia"/>
+			</inertial>
 			<visual>
 				<origin xyz="0 0 0" rpy="0 0 0" />
@@ -187,15 +286,34 @@
 				<material name="SoftHand/DarkGolden" />
 			</visual>
+			<collision>
+				<geometry>
+					<mesh filename="package://soft_hand_description/meshes/fingertip.stl" scale=" .001 .001 .001" />
+				</geometry>
+			</collision>
 		</link>
 	</xacro:macro>
 	<!-- SOFT HAND MODEL -->
 	<xacro:macro name="soft_hand" params="parent name *origin">
+		<!-- MOTOR JOINT -->
+		<!--
+		<joint name="${name}a_actuator" type="revolute" >
+			<parent link="${parent}" />
+			<child link="${name}_invisible_wire_link"/>
+			<axis xyz="0 0 1" />
+			<limit lower="${actuator_lb *pi/180}" upper="${actuator_ub *pi/180}" effort="${actuator_max_effort}" velocity="${actuator_max_velocity}"/>
+			<dynamics damping="${actuator_damping}" friction="${actuator_friction}"/>
+		</joint>
+		<link name="${name}_invisible_wire_link"/>
+		-->
 		<!-- PALM -->
 		<joint name="${name}_palm_joint" type="fixed" >
-			<origin xyz="0 0 0" rpy="0 0 0" />
+			<insert_block name="origin"/>
 			<parent link="${parent}" />
 			<child link="${name}_palm_link" />
 		</joint>
 		<link name="${name}_palm_link">
+			<inertial>
+				<insert_block name="palm_inertia"/>
+			</inertial>
 			<visual>
 				<origin xyz="0 0 0" rpy="0 0 0" />
@@ -205,4 +323,9 @@
 				<material name="SoftHand/LightGrey" />
 			</visual>
+			<collision>
+				<geometry>
+					<mesh filename="package://soft_hand_description/meshes/palm.stl" scale=" .001 .001 .001" />
+				</geometry>
+			</collision>
 		</link>
 		<!-- FINGERS AND THUMB -->
@@ -212,4 +335,6 @@
 		<xacro:soft_finger parent="${name}_palm_link" name="${name}_ring" position="0.0105 0.0943918 0.00205" orientation="${180*pi/180} 0 ${(-90-10)*pi/180}" />
 		<xacro:soft_finger parent="${name}_palm_link" name="${name}_little" position="0.030 0.0808918 0.00205" orientation="${180*pi/180} 0 ${(-90-20)*pi/180}" />
+		<xacro:soft_hand_transmission name="${name}"/>
+		<xacro:soft_hand_gazebo name="${name}"/>
 	</xacro:macro>
 </robot>

File: soft_hand/soft_hand_description/robot/hand_in_world.urdf.xacro (robot description, xacro)
@@ -1,15 +1,29 @@
 <?xml version="1.0"?>
-<robot xmlns:xacro="http://ros.org/wiki/xacro" name="soft_hand">
-  <xacro:include filename="$(find soft_hand_description)/model/soft_hand.urdf.xacro"/>
-  <link name="world">
-<!--     <visual>
-      <origin xyz="0 0 0" rpy="0 0 0"/>
-      <geometry>
-        <box size="1 1 1.0"/>
-      </geometry>
-    </visual> -->
-  </link>
-  <xacro:soft_hand parent="world" name="hand">
-    <origin xyz="0 0 0" rpy="0 0 0"/>
-  </xacro:soft_hand>
+<robot xmlns:xacro="http://www.ros.org/wiki/xacro" name="soft_hand">
+	<xacro:include filename="$(find soft_hand_description)/model/soft_hand.urdf.xacro"/>
+	<link name="wrist">
+		<inertial>
+			<mass value="50.0"/>
+			<inertia  ixx="1" ixy="0.00"  ixz="0.00" iyy="1" iyz="0.00" izz="1" />
+		</inertial>
+		<visual>
+			<origin xyz="0 0 0.50" rpy="0 0 0"/>
+			<geometry>
+				<box size="1.0 1.0 1.0"/>
+			</geometry>
+		</visual>
+		<collision>
+			<origin xyz="0 0 0.50" rpy="0 0 0"/>
+			<geometry>
+				<box size="1.0 1.0 1.0"/>
+			</geometry>
+		</collision>
+	</link>
+	<!-- comment or uncomment depending if you want to simulate a fixed or a flying hand -->
+	<gazebo reference="wrist">
+		<static>true</static>
+	</gazebo>
+	<xacro:soft_hand parent="wrist" name="hand">
+		<origin xyz="0 0 1" rpy="1.570796 0 0"/>
+	</xacro:soft_hand>
 </robot>

Commit message: adding changes in the handmoveadmin submodule and fix in package.xml

File: soft_hand/soft_hand_description/model/soft_hand.urdf.xacro (robot description, xacro)
@@ -47,6 +47,6 @@
 	<xacro:property name="little_outer_R" value="1.0" />
 	<!-- synergy joint properties -->
-	<xacro:property name="synergy_lb" value="0.0" />
-	<xacro:property name="synergy_ub" value="1.0" />
+	<xacro:property name="synergy_lb" value="-5.0" />
+	<xacro:property name="synergy_ub" value="5.0" />
 	<xacro:property name="max_synergy_velocity" value="100" />
 	<xacro:property name="max_synergy_effort" value="100" />

Commit message: update collision geometry, and upladed the HW interface

File: soft_hand/soft_hand_description/model/soft_hand.urdf.xacro (robot description, xacro)
@@ -27,27 +27,28 @@
 	<xacro:property name="friction" value="0.0" />
 	<!-- synergy vector -->
-	<xacro:property name="thumb_abd_R" value="1.3" />
-	<xacro:property name="thumb_inner_R" value="1.3" />
-	<xacro:property name="thumb_outer_R" value="1.0" />
-	<xacro:property name="index_abd_R" value="-0.2" />
-	<xacro:property name="index_inner_R" value="1.0" />
-	<xacro:property name="index_middle_R" value="1.0" />
-	<xacro:property name="index_outer_R" value="1.0" />
-	<xacro:property name="middle_abd_R" value="0.0" />
-	<xacro:property name="middle_inner_R" value="1.0" />
-	<xacro:property name="middle_middle_R" value="1.0" />
-	<xacro:property name="middle_outer_R" value="1.0" />
-	<xacro:property name="ring_abd_R" value="0.2" />
-	<xacro:property name="ring_inner_R" value="1.0" />
-	<xacro:property name="ring_middle_R" value="1.0" />
-	<xacro:property name="ring_outer_R" value="1.0" />
-	<xacro:property name="little_abd_R" value="0.4" />
-	<xacro:property name="little_inner_R" value="1.0" />
-	<xacro:property name="little_middle_R" value="1.0" />
-	<xacro:property name="little_outer_R" value="1.0" />
+	<xacro:property name="syn_amp" value="0.00005555555" /> <!-- 1/18000 -->
+	<xacro:property name="thumb_abd_R" value="${1.3*syn_amp}" />
+	<xacro:property name="thumb_inner_R" value="${1.3*syn_amp}" />
+	<xacro:property name="thumb_outer_R" value="${1.0*syn_amp}" />
+	<xacro:property name="index_abd_R" value="-${0.2*syn_amp}" />
+	<xacro:property name="index_inner_R" value="${1.0*syn_amp}" />
+	<xacro:property name="index_middle_R" value="${1.0*syn_amp}" />
+	<xacro:property name="index_outer_R" value="${1.0*syn_amp}" />
+	<xacro:property name="middle_abd_R" value="${0.0*syn_amp}" />
+	<xacro:property name="middle_inner_R" value="${1.0*syn_amp}" />
+	<xacro:property name="middle_middle_R" value="${1.0*syn_amp}" />
+	<xacro:property name="middle_outer_R" value="${1.0*syn_amp}" />
+	<xacro:property name="ring_abd_R" value="${0.2*syn_amp}" />
+	<xacro:property name="ring_inner_R" value="${1.0*syn_amp}" />
+	<xacro:property name="ring_middle_R" value="${1.0*syn_amp}" />
+	<xacro:property name="ring_outer_R" value="${1.0*syn_amp}" />
+	<xacro:property name="little_abd_R" value="${0.4*syn_amp}" />
+	<xacro:property name="little_inner_R" value="${1.0*syn_amp}" />
+	<xacro:property name="little_middle_R" value="${1.0*syn_amp}" />
+	<xacro:property name="little_outer_R" value="${1.0*syn_amp}" />
 	<!-- synergy joint properties -->
-	<xacro:property name="synergy_lb" value="-5.0" />
-	<xacro:property name="synergy_ub" value="5.0" />
-	<xacro:property name="max_synergy_velocity" value="100" />
+	<xacro:property name="synergy_lb" value="0.0" />
+	<xacro:property name="synergy_ub" value="18000.0" />
+	<xacro:property name="max_synergy_velocity" value="10000" />
 	<xacro:property name="max_synergy_effort" value="100" />
 	<xacro:property name="synergy_damping" value="0.0" />
@@ -80,5 +81,5 @@
 			<collision>
 				<geometry>
-					<mesh filename="package://soft_hand_description/meshes/knuckle.stl" scale=" .001 .001 .001" />
+					<mesh filename="package://soft_hand_description/meshes/knuckle_collision.stl" scale=" .001 .001 .001" />
 				</geometry>
 			</collision>
@@ -124,5 +125,5 @@
 			<collision>
 				<geometry>
-					<mesh filename="package://soft_hand_description/meshes/phalanx.stl" scale=" .001 .001 .001" />
+					<mesh filename="package://soft_hand_description/meshes/phalanx_collision.stl" scale=" .001 .001 .001" />
 				</geometry>
 			</collision>
@@ -168,5 +169,5 @@
 			<collision>
 				<geometry>
-					<mesh filename="package://soft_hand_description/meshes/phalanx.stl" scale=" .001 .001 .001" />
+					<mesh filename="package://soft_hand_description/meshes/phalanx_collision.stl" scale=" .001 .001 .001" />
 				</geometry>
 			</collision>
@@ -212,5 +213,5 @@
 			<collision>
 				<geometry>
-					<mesh filename="package://soft_hand_description/meshes/fingertip.stl" scale=" .001 .001 .001" />
+					<mesh filename="package://soft_hand_description/meshes/fingertip_collision.stl" scale=" .001 .001 .001" />
 				</geometry>
 			</collision>
@@ -245,5 +246,5 @@
 				<collision>
 					<geometry>
-						<mesh filename="package://soft_hand_description/meshes/thumb_knuckle_left.stl" scale=" .001 .001 .001" />
+						<mesh filename="package://soft_hand_description/meshes/thumb_knuckle_left_collision.stl" scale=" .001 .001 .001" />
 					</geometry>
 				</collision>
@@ -287,5 +288,5 @@
 				<collision>
 					<geometry>
-						<mesh filename="package://soft_hand_description/meshes/thumb_knuckle_right.stl" scale=" .001 .001 .001" />
+						<mesh filename="package://soft_hand_description/meshes/thumb_knuckle_right_collision.stl" scale=" .001 .001 .001" />
 					</geometry>
 				</collision>
@@ -332,5 +333,5 @@
 			<collision>
 				<geometry>
-					<mesh filename="package://soft_hand_description/meshes/phalanx.stl" scale=" .001 .001 .001" />
+					<mesh filename="package://soft_hand_description/meshes/phalanx_collision.stl" scale=" .001 .001 .001" />
 				</geometry>
 			</collision>
@@ -376,5 +377,5 @@
 			<collision>
 				<geometry>
-					<mesh filename="package://soft_hand_description/meshes/fingertip.stl" scale=" .001 .001 .001" />
+					<mesh filename="package://soft_hand_description/meshes/fingertip_collision.stl" scale=" .001 .001 .001" />
 				</geometry>
 			</collision>
@@ -415,5 +416,5 @@
 				<collision>
 					<geometry>
-						<mesh filename="package://soft_hand_description/meshes/palm_left.stl" scale=" .001 .001 .001" />
+						<mesh filename="package://soft_hand_description/meshes/palm_left_collision.stl" scale=" .001 .001 .001" />
 					</geometry>
 				</collision>
@@ -428,5 +429,5 @@
 				<collision>
 					<geometry>
-						<mesh filename="package://soft_hand_description/meshes/palm_right.stl" scale=" .001 .001 .001" />
+						<mesh filename="package://soft_hand_description/meshes/palm_right_collision.stl" scale=" .001 .001 .001" />
 					</geometry>
 				</collision>

Commit message: Resolve #2.

File: soft_hand/soft_hand_description/model/soft_hand.urdf.xacro (robot description, xacro)
@@ -384,17 +384,4 @@
 	<!-- SOFT HAND MODEL -->
 	<xacro:macro name="soft_hand" params="parent name withAdaptiveTransmission useMimicTag left *origin">
-		<!-- MOTOR JOINT -->
-		<joint name="${name}_synergy_joint" type="revolute" >
-			<parent link="${parent}" />
-			<child link="${name}_invisible_wire_link"/>
-			<axis xyz="0 0 1" />
-			<limit lower="${synergy_lb}" upper="${synergy_ub}" effort="${max_synergy_effort}" velocity="${max_synergy_velocity}"/>
-			<dynamics damping="${synergy_damping}" friction="${synergy_friction}"/>
-		</joint>
-		<link name="${name}_invisible_wire_link">
-			<inertial>
-				<insert_block name="negligible_inertia"/>
-			</inertial>
-		</link>
 		<!-- PALM -->
 		<joint name="${name}_palm_joint" type="fixed" >
@@ -433,4 +420,17 @@
 				</collision>
 			</xacro:unless>
+		</link>
+		<!-- MOTOR JOINT -->
+		<joint name="${name}_synergy_joint" type="revolute" >
+			<parent link="${name}_palm_link" />
+			<child link="${name}_invisible_wire_link"/>
+			<axis xyz="0 0 1" />
+			<limit lower="${synergy_lb}" upper="${synergy_ub}" effort="${max_synergy_effort}" velocity="${max_synergy_velocity}"/>
+			<dynamics damping="${synergy_damping}" friction="${synergy_friction}"/>
+		</joint>
+		<link name="${name}_invisible_wire_link">
+			<inertial>
+				<insert_block name="negligible_inertia"/>
+			</inertial>
 		</link>
 		<!-- THUMB AND FINGERS -->
