Commit message: Update to allow multi-robots in gazebo

File: soft_hand/soft_hand_description/model/soft_hand.urdf.xacro (robot description, xacro)
@@ -32,5 +32,5 @@
 	<xacro:property name="friction" value="0.0" />
 	<!-- synergy vector -->
-	<xacro:property name="syn_amp" value="0.00005555555" /> <!-- 1/18000 -->
+	<xacro:property name="syn_amp" value="1.0"/> <!--0.00005555555" /--> <!-- 1/18000 -->
 	<xacro:property name="thumb_abd_R" value="${1.3*syn_amp}" />
 	<xacro:property name="thumb_inner_R" value="${1.3*syn_amp}" />
@@ -54,5 +54,5 @@
 	<!-- synergy joint properties -->
 	<xacro:property name="synergy_lb" value="0.0" />
-	<xacro:property name="synergy_ub" value="18000.0" />
+	<xacro:property name="synergy_ub" value="1.0"/> <!--18000.0" /-->
 	<xacro:property name="max_synergy_velocity" value="10000" />
 	<xacro:property name="max_synergy_effort" value="100" />

Commit message: Temporal solution to HW interface

File: soft_hand/soft_hand_description/model/soft_hand.urdf.xacro (robot description, xacro)
@@ -32,5 +32,5 @@
 	<xacro:property name="friction" value="0.0" />
 	<!-- synergy vector -->
-	<xacro:property name="syn_amp" value="1.0"/> <!--0.00005555555" /--> <!-- 1/18000 -->
+	<xacro:property name="syn_amp" value="0.00005555555" /> <!-- 1/18000 -->
 	<xacro:property name="thumb_abd_R" value="${1.3*syn_amp}" />
 	<xacro:property name="thumb_inner_R" value="${1.3*syn_amp}" />
@@ -54,5 +54,5 @@
 	<!-- synergy joint properties -->
 	<xacro:property name="synergy_lb" value="0.0" />
-	<xacro:property name="synergy_ub" value="1.0"/> <!--18000.0" /-->
+	<xacro:property name="synergy_ub" value="18000.0"/> <!--18000.0" /-->
 	<xacro:property name="max_synergy_velocity" value="10000" />
 	<xacro:property name="max_synergy_effort" value="100" />

Commit message: Temporal solution to HW interface

File: soft_hand/soft_hand_description/model/soft_hand.urdf.xacro (robot description, xacro)
@@ -27,5 +27,5 @@
 	<xacro:property name="friction" value="0.0" />
 	<!-- synergy vector -->
-	<xacro:property name="syn_amp" value="1.0"/> <!--0.00005555555" /--> <!-- 1/18000 -->
+	<xacro:property name="syn_amp" value="0.00005555555" /> <!-- 1/18000 -->
 	<xacro:property name="thumb_abd_R" value="${1.3*syn_amp}" />
 	<xacro:property name="thumb_inner_R" value="${1.3*syn_amp}" />
@@ -49,5 +49,5 @@
 	<!-- synergy joint properties -->
 	<xacro:property name="synergy_lb" value="0.0" />
-	<xacro:property name="synergy_ub" value="1.0"/> <!--18000.0" /-->
+	<xacro:property name="synergy_ub" value="18000.0"/> <!--18000.0" /-->
 	<xacro:property name="max_synergy_velocity" value="10000" />
 	<xacro:property name="max_synergy_effort" value="100" />

Commit message: Updated mesh and kinematics of the right thumb, it was wrong before.

File: soft_hand/soft_hand_description/model/soft_hand.urdf.xacro (robot description, xacro)
@@ -294,5 +294,6 @@
 			<!-- PROXIMAL PHALANGE -->
 			<joint name="${name}_inner_joint" type="revolute">
-				<origin xyz="0.022726230 0.00811475 0.0" rpy="0.42662757656587236 0.0 0.18131960430075023" />
+				<!-- <origin xyz="0.022500000 -0.003300000 0.0" rpy="0.42662757656587236 0.0 0.18131960430075023" /> -->
+				<origin xyz="0.022500000 -0.003300000 0.0" rpy="0.42662757656587236 0.0 0.0"/>
 				<parent link="${name}_knuckle_link"/>
 				<child link="${name}_fake_link1"/>
@@ -444,5 +445,5 @@
 		</xacro:if>
 		<xacro:unless value="${left}">
-			<xacro:soft_thumb parent="${name}_palm_link" parent_name="${name}" name="${name}_thumb" left="${left}" position="0.005669722 0.032876873 0.018373996" orientation="0.08389097788000696 -0.4287012609015684 1.3712034099005517" useMimicTag="${useMimicTag}" abd_R="${thumb_abd_R *(thumb_abd_ub - thumb_abd_lb)*pi/180}" inner_R="${thumb_inner_R *(inner_ub - inner_lb)*pi/180}" outer_R="${thumb_outer_R *(outer_ub - outer_lb)*pi/180}"/>
+			<xacro:soft_thumb parent="${name}_palm_link" parent_name="${name}" name="${name}_thumb" left="${left}" position="0.005669722 0.032876873 0.018373996" orientation="0.0 -0.43633198577877447 1.5707963267948966" useMimicTag="${useMimicTag}" abd_R="${thumb_abd_R *(thumb_abd_ub - thumb_abd_lb)*pi/180}" inner_R="${thumb_inner_R *(inner_ub - inner_lb)*pi/180}" outer_R="${thumb_outer_R *(outer_ub - outer_lb)*pi/180}"/>
 			<xacro:soft_finger parent="${name}_palm_link" parent_name="${name}" name="${name}_index" position="-0.003300000 0.019500000 0.058891802" orientation="1.5707963267948957 -1.2217307407768807 1.570796326794897" useMimicTag="${useMimicTag}" abd_R="${index_abd_R}" inner_R="${index_inner_R *(inner_ub - inner_lb)*pi/180}" middle_R="${index_middle_R *(middle_ub - middle_lb)*pi/180}" outer_R="${index_outer_R *(outer_ub - outer_lb)*pi/180}" />
 			<xacro:soft_finger parent="${name}_palm_link" parent_name="${name}" name="${name}_middle" position="-0.003300000 0.0 0.072391802" orientation="-3.141592653589793 -1.5707963267948966 0.0" useMimicTag="${useMimicTag}" abd_R="${middle_abd_R}" inner_R="${middle_inner_R *(inner_ub - inner_lb)*pi/180}" middle_R="${middle_middle_R *(middle_ub - middle_lb)*pi/180}" outer_R="${middle_outer_R *(outer_ub - outer_lb)*pi/180}" />

Commit message: Added the pacman version of the soft hand. Still the geometries of the coupler are not well visualized in RView, so careful with gazebo simulation.

File: soft_hand/soft_hand_description/model/soft_hand.urdf.xacro (robot description, xacro)
@@ -6,8 +6,13 @@
 		CAD model available at: http://www.naturalmachinemotioninitiative.com/#!softhand/c24r2
 	-->
+	<!-- include other model components -->
 	<xacro:include filename="$(find soft_hand_description)/model/materials.urdf.xacro"/>
 	<xacro:include filename="$(find soft_hand_description)/model/soft_hand.transmission.xacro"/>
 	<xacro:include filename="$(find soft_hand_description)/model/soft_hand.gazebo.xacro"/>
 	<xacro:include filename="$(find soft_hand_description)/model/soft_hand.inertia.xacro"/>
+	<!-- accesories -->
+	<xacro:include filename="$(find soft_hand_description)/model/accesories/kuka_coupler.urdf.xacro"/>
+	<xacro:include filename="$(find soft_hand_description)/model/accesories/clamp.urdf.xacro"/>
+	<xacro:include filename="$(find soft_hand_description)/model/accesories/softhand_base.urdf.xacro"/>
 	<xacro:property name="pi" value="3.1415926535897931" />
 	<!-- joint properties -->
@@ -56,5 +61,5 @@
 	<!-- SOFT FINGER model -->
 	<!-- 4 fingers are equal (index, middle, ring, little) -->
-	<xacro:macro name="soft_finger" params="parent parent_name name position orientation useMimicTag abd_R inner_R middle_R outer_R">
+	<xacro:macro name="soft_finger" params="parent parent_name name position orientation left useMimicTag abd_R inner_R middle_R outer_R">
 		<!-- KNUCKLE -->
 		<joint name="${name}_abd_joint" type="revolute">
@@ -62,5 +67,10 @@
 			<parent link="${parent}"/>
 			<child link="${name}_knuckle_link"/>
-			<axis xyz="0 0 1" />
+			<xacro:if value="${left}">
+				<axis xyz="0 0 -1" />
+			</xacro:if>
+			<xacro:unless value="${left}">
+				<axis xyz="0 0 1" />
+			</xacro:unless>
 			<limit lower="${abd_lb *pi/180}" upper="${abd_ub *pi/180}" effort="${effort}" velocity="${velocity}"/>
 			<dynamics damping="${damping}" friction="${friction}"/>
@@ -385,8 +395,26 @@
 	<!-- SOFT HAND MODEL -->
 	<xacro:macro name="soft_hand" params="parent name withAdaptiveTransmission useMimicTag left *origin">
+		<!-- PACMAN VERION ALREADY INCLUDES THE COUPLER, CLAMP AND BASE -->
+		<!-- KUKA_COUPLER -->
+		<xacro:kuka_coupler parent="${parent}" name="${name}_kuka_coupler">
+			<insert_block name="origin"/>
+		</xacro:kuka_coupler>
+		<!-- CLAMP -->
+		<xacro:clamp parent="${name}_kuka_coupler" name="${name}_clamp">
+			<origin xyz="0 0 0.01" rpy="0 0 0"/>
+		</xacro:clamp>
+		<!-- SOFT HAND BASE -->
+		<xacro:softhand_base parent="${name}_clamp" name="${name}_softhand_base" left="${left}">
+			<origin xyz="0 0 0.004" rpy="0 0 0"/>
+		</xacro:softhand_base>
 		<!-- PALM -->
-		<joint name="${name}_palm_joint" type="fixed" >
-			<insert_block name="origin"/>
-			<parent link="${parent}" />
+		<joint name="${name}_palm_joint" type="fixed">
+			<xacro:if value="${left}">
+				<origin xyz="0.002 -0.00695 0.0535" rpy="0 0 0"/>
+			</xacro:if>
+			<xacro:unless value="${left}">
+				<origin xyz="0.002 0.00695 0.0535" rpy="0 0 0"/>
+			</xacro:unless>
+			<parent link="${name}_softhand_base" />
 			<child link="${name}_palm_link" />
 		</joint>
@@ -438,16 +466,16 @@
 		<!-- change anchor points accordingly to the leftness -->
 		<xacro:if value="${left}">
-			<xacro:soft_thumb parent="${name}_palm_link" parent_name="${name}" name="${name}_thumb" left="${left}" position="0.005669722 -0.032876873 0.018373996" orientation="0.0 -0.43633198577877463 -1.570796326794897" useMimicTag="${useMimicTag}" abd_R="${thumb_abd_R *(thumb_abd_ub - thumb_abd_lb)*pi/180}" inner_R="${thumb_inner_R *(inner_ub - inner_lb)*pi/180}" outer_R="${thumb_outer_R *(outer_ub - outer_lb)*pi/180}"/>
-			<xacro:soft_finger parent="${name}_palm_link" parent_name="${name}" name="${name}_index" position="-0.003349856 -0.019500000 0.058891802" orientation="-1.5707963267948957 -1.2217307407768807 -1.570796326794897" useMimicTag="${useMimicTag}" abd_R="${index_abd_R}" inner_R="${index_inner_R *(inner_ub - inner_lb)*pi/180}" middle_R="${index_middle_R *(middle_ub - middle_lb)*pi/180}" outer_R="${index_outer_R *(outer_ub - outer_lb)*pi/180}" />
-			<xacro:soft_finger parent="${name}_palm_link" parent_name="${name}" name="${name}_middle" position="-0.003349856 0.0 0.072391802" orientation="-3.141592653589793 -1.5707963267948966 0.0" useMimicTag="${useMimicTag}" abd_R="${middle_abd_R}" inner_R="${middle_inner_R *(inner_ub - inner_lb)*pi/180}" middle_R="${middle_middle_R *(middle_ub - middle_lb)*pi/180}" outer_R="${middle_outer_R *(outer_ub - outer_lb)*pi/180}" />
-			<xacro:soft_finger parent="${name}_palm_link" parent_name="${name}" name="${name}_ring" position="-0.003349856 0.019500000 0.058891802" orientation="1.5707963267948952 -1.3962636194521678 1.5707963267948966" useMimicTag="${useMimicTag}" abd_R="${ring_abd_R}" inner_R="${ring_inner_R *(inner_ub - inner_lb)*pi/180}" middle_R="${ring_middle_R *(middle_ub - middle_lb)*pi/180}" outer_R="${ring_outer_R *(outer_ub - outer_lb)*pi/180}" />
-			<xacro:soft_finger parent="${name}_palm_link" parent_name="${name}" name="${name}_little" position="-0.00349856 0.039000000 0.045391802" orientation="1.5707963267948957 -1.2217307407768807 1.570796326794897" useMimicTag="${useMimicTag}" abd_R="${little_abd_R}" inner_R="${little_inner_R *(inner_ub - inner_lb)*pi/180}" middle_R="${little_middle_R *(middle_ub - middle_lb)*pi/180}" outer_R="${little_outer_R *(outer_ub - outer_lb)*pi/180}" />
+			<xacro:soft_thumb parent="${name}_palm_link" parent_name="${name}" name="${name}_thumb" position="0.005669722 -0.029616 0.055314" orientation="0.0 -0.38397275793662144 -1.5707963267948966" left="${left}" useMimicTag="${useMimicTag}" abd_R="${thumb_abd_R *(thumb_abd_ub - thumb_abd_lb)*pi/180}" inner_R="${thumb_inner_R *(inner_ub - inner_lb)*pi/180}" outer_R="${thumb_outer_R *(outer_ub - outer_lb)*pi/180}"/>
+			<xacro:soft_finger parent="${name}_palm_link" parent_name="${name}" name="${name}_index" position="-0.0033 -0.0195 0.0936994" orientation="-1.5707963267948966 -1.4835299330931884 -1.5707963267948966" left="${left}" useMimicTag="${useMimicTag}" abd_R="${index_abd_R}" inner_R="${index_inner_R *(inner_ub - inner_lb)*pi/180}" middle_R="${index_middle_R *(middle_ub - middle_lb)*pi/180}" outer_R="${index_outer_R *(outer_ub - outer_lb)*pi/180}" />
+			<xacro:soft_finger parent="${name}_palm_link" parent_name="${name}" name="${name}_middle" position="-0.0033 0.0 0.100699" orientation="3.1415 -1.5707963267948966 0.0" left="${left}" useMimicTag="${useMimicTag}" abd_R="${middle_abd_R}" inner_R="${middle_inner_R *(inner_ub - inner_lb)*pi/180}" middle_R="${middle_middle_R *(middle_ub - middle_lb)*pi/180}" outer_R="${middle_outer_R *(outer_ub - outer_lb)*pi/180}" />
+			<xacro:soft_finger parent="${name}_palm_link" parent_name="${name}" name="${name}_ring" position="-0.0033 0.0195 0.0936994" orientation="1.5707963267948966 -1.5184364298870514 1.5707963267948966" left="${left}" useMimicTag="${useMimicTag}" abd_R="${ring_abd_R}" inner_R="${ring_inner_R *(inner_ub - inner_lb)*pi/180}" middle_R="${ring_middle_R *(middle_ub - middle_lb)*pi/180}" outer_R="${ring_outer_R *(outer_ub - outer_lb)*pi/180}" />
+			<xacro:soft_finger parent="${name}_palm_link" parent_name="${name}" name="${name}_little" position="-0.0033 0.039 0.0836994" orientation="1.5707963267948966 -1.4835299330931884 1.5707963267948966" left="${left}" useMimicTag="${useMimicTag}" abd_R="${little_abd_R}" inner_R="${little_inner_R *(inner_ub - inner_lb)*pi/180}" middle_R="${little_middle_R *(middle_ub - middle_lb)*pi/180}" outer_R="${little_outer_R *(outer_ub - outer_lb)*pi/180}" />
 		</xacro:if>
 		<xacro:unless value="${left}">
-			<xacro:soft_thumb parent="${name}_palm_link" parent_name="${name}" name="${name}_thumb" left="${left}" position="0.005669722 0.032876873 0.018373996" orientation="0.0 -0.43633198577877447 1.5707963267948966" useMimicTag="${useMimicTag}" abd_R="${thumb_abd_R *(thumb_abd_ub - thumb_abd_lb)*pi/180}" inner_R="${thumb_inner_R *(inner_ub - inner_lb)*pi/180}" outer_R="${thumb_outer_R *(outer_ub - outer_lb)*pi/180}"/>
-			<xacro:soft_finger parent="${name}_palm_link" parent_name="${name}" name="${name}_index" position="-0.003300000 0.019500000 0.058891802" orientation="1.5707963267948957 -1.2217307407768807 1.570796326794897" useMimicTag="${useMimicTag}" abd_R="${index_abd_R}" inner_R="${index_inner_R *(inner_ub - inner_lb)*pi/180}" middle_R="${index_middle_R *(middle_ub - middle_lb)*pi/180}" outer_R="${index_outer_R *(outer_ub - outer_lb)*pi/180}" />
-			<xacro:soft_finger parent="${name}_palm_link" parent_name="${name}" name="${name}_middle" position="-0.003300000 0.0 0.072391802" orientation="-3.141592653589793 -1.5707963267948966 0.0" useMimicTag="${useMimicTag}" abd_R="${middle_abd_R}" inner_R="${middle_inner_R *(inner_ub - inner_lb)*pi/180}" middle_R="${middle_middle_R *(middle_ub - middle_lb)*pi/180}" outer_R="${middle_outer_R *(outer_ub - outer_lb)*pi/180}" />
-			<xacro:soft_finger parent="${name}_palm_link" parent_name="${name}" name="${name}_ring" position="-0.003300000 -0.019500000 0.058891802" orientation="-1.5707963267948952 -1.3962636194521678 -1.5707963267948966" useMimicTag="${useMimicTag}" abd_R="${ring_abd_R}" inner_R="${ring_inner_R *(inner_ub - inner_lb)*pi/180}" middle_R="${ring_middle_R *(middle_ub - middle_lb)*pi/180}" outer_R="${ring_outer_R *(outer_ub - outer_lb)*pi/180}" />
-			<xacro:soft_finger parent="${name}_palm_link" parent_name="${name}" name="${name}_little" position="-0.003300000 -0.039000000 0.045391802" orientation="-1.5707963267948957 -1.2217307407768807 -1.570796326794897" useMimicTag="${useMimicTag}" abd_R="${little_abd_R}" inner_R="${little_inner_R *(inner_ub - inner_lb)*pi/180}" middle_R="${little_middle_R *(middle_ub - middle_lb)*pi/180}" outer_R="${little_outer_R *(outer_ub - outer_lb)*pi/180}" />
+			<xacro:soft_thumb parent="${name}_palm_link" parent_name="${name}" name="${name}_thumb" position="0.00566972 0.0296160 0.0553140" orientation="0.0 -0.38397275793662144 1.5707963267948966" left="${left}" useMimicTag="${useMimicTag}" abd_R="${thumb_abd_R *(thumb_abd_ub - thumb_abd_lb)*pi/180}" inner_R="${thumb_inner_R *(inner_ub - inner_lb)*pi/180}" outer_R="${thumb_outer_R *(outer_ub - outer_lb)*pi/180}"/>
+			<xacro:soft_finger parent="${name}_palm_link" parent_name="${name}" name="${name}_index" position="-0.0033 0.0195 0.0936994" orientation="1.5707963267948966 -1.4835299330931884 1.5707963267948966" left="${left}" useMimicTag="${useMimicTag}" abd_R="${index_abd_R}" inner_R="${index_inner_R *(inner_ub - inner_lb)*pi/180}" middle_R="${index_middle_R *(middle_ub - middle_lb)*pi/180}" outer_R="${index_outer_R *(outer_ub - outer_lb)*pi/180}" />
+			<xacro:soft_finger parent="${name}_palm_link" parent_name="${name}" name="${name}_middle" position="-0.003300000 0.0 0.100699" orientation="3.141592 -1.5707963267948966 0.0" left="${left}" useMimicTag="${useMimicTag}" abd_R="${middle_abd_R}" inner_R="${middle_inner_R *(inner_ub - inner_lb)*pi/180}" middle_R="${middle_middle_R *(middle_ub - middle_lb)*pi/180}" outer_R="${middle_outer_R *(outer_ub - outer_lb)*pi/180}" />
+			<xacro:soft_finger parent="${name}_palm_link" parent_name="${name}" name="${name}_ring" position="-0.0033 -0.0195 0.0936994" orientation="-1.5707963267948966 -1.5184364298870514 -1.5707963267948966 " left="${left}" useMimicTag="${useMimicTag}" abd_R="${ring_abd_R}" inner_R="${ring_inner_R *(inner_ub - inner_lb)*pi/180}" middle_R="${ring_middle_R *(middle_ub - middle_lb)*pi/180}" outer_R="${ring_outer_R *(outer_ub - outer_lb)*pi/180}" />
+			<xacro:soft_finger parent="${name}_palm_link" parent_name="${name}" name="${name}_little" position="-0.0033 -0.039 0.0836994" orientation="-1.5707963267948966 -1.4835299330931884 -1.5707963267948966" left="${left}" useMimicTag="${useMimicTag}" abd_R="${little_abd_R}" inner_R="${little_inner_R *(inner_ub - inner_lb)*pi/180}" middle_R="${little_middle_R *(middle_ub - middle_lb)*pi/180}" outer_R="${little_outer_R *(outer_ub - outer_lb)*pi/180}" />
 		</xacro:unless>
 		<xacro:soft_hand_transmission name="${name}" withAdaptiveTransmission="${withAdaptiveTransmission}"/>

File: soft_hand/soft_hand_description/robot/soft_hand_kinematic_synergy.urdf.xacro (robot description, xacro)
@@ -2,4 +2,5 @@
 <robot xmlns:xacro="http://www.ros.org/wiki/xacro" name="soft_hand">
 	<xacro:include filename="$(find soft_hand_description)/model/soft_hand.urdf.xacro"/>
+	<xacro:include filename="$(find soft_hand_description)/model/accesories/kuka_coupler.urdf.xacro"/>
 	<link name="box">
 		<inertial>
@@ -20,5 +21,5 @@
 		</collision>
 	</link>
-	<xacro:soft_hand parent="box" name="soft_hand_right" withAdaptiveTransmission="true" useMimicTag="$(arg use_mimic_tag)" left="true">
+	<xacro:soft_hand parent="box" name="soft_hand" withAdaptiveTransmission="true" useMimicTag="$(arg use_mimic_tag)" left="true">
 		<origin xyz="0.0 0.0 1.0" rpy="0 0 0"/>
 	</xacro:soft_hand>

Commit message: Solves the namespacing problem with real hardware. Soft hand commands must go from 0.0-1.0.

File: soft_hand/soft_hand_description/model/soft_hand.urdf.xacro (robot description, xacro)
@@ -32,5 +32,5 @@
 	<xacro:property name="friction" value="0.0" />
 	<!-- synergy vector -->
-	<xacro:property name="syn_amp" value="0.00005555555" /> <!-- 1/18000 -->
+	<xacro:property name="syn_amp" value="1" />
 	<xacro:property name="thumb_abd_R" value="${1.3*syn_amp}" />
 	<xacro:property name="thumb_inner_R" value="${1.3*syn_amp}" />
@@ -54,6 +54,6 @@
 	<!-- synergy joint properties -->
 	<xacro:property name="synergy_lb" value="0.0" />
-	<xacro:property name="synergy_ub" value="18000.0"/> <!--18000.0" /-->
-	<xacro:property name="max_synergy_velocity" value="10000" />
+	<xacro:property name="synergy_ub" value="18000.0"/>
+	<xacro:property name="max_synergy_velocity" value="100000" />
 	<xacro:property name="max_synergy_effort" value="100" />
 	<xacro:property name="synergy_damping" value="0.0" />

Commit message: The last commit still had 18000 as the max value of the motor. Fixing that.

File: soft_hand/soft_hand_description/model/soft_hand.urdf.xacro (robot description, xacro)
@@ -54,5 +54,5 @@
 	<!-- synergy joint properties -->
 	<xacro:property name="synergy_lb" value="0.0" />
-	<xacro:property name="synergy_ub" value="18000.0"/>
+	<xacro:property name="synergy_ub" value="1.0"/>
 	<xacro:property name="max_synergy_velocity" value="100000" />
 	<xacro:property name="max_synergy_effort" value="100" />
