Commit message: Update of configured robots: 1) two_soft_hands 2) kinematic-only synergy

File: soft_hand/soft_hand_description/robot/soft_hand_kinematic_synergy.urdf.xacro (robot description, xacro)
@@ -4,5 +4,5 @@
 	<link name="box">
 		<inertial>
-			<mass value="50.0"/>
+			<mass value="1.0"/>
 			<inertia  ixx="1" ixy="0.00"  ixz="0.00" iyy="1" iyz="0.00" izz="1" />
 		</inertial>
@@ -20,53 +20,6 @@
 		</collision>
 	</link>
-	<joint name="box_wrist_left_joint" type="fixed">
-		<origin xyz="0 -0.2 1.02" rpy="0 0 0" />
-		<parent link="box"/>
-		<child link="wrist_left"/>
-	</joint>
-	<link name="wrist_left">
-		<inertial>
-			<mass value="1.0"/>
-			<inertia  ixx="0.01" ixy="0.00"  ixz="0.00" iyy="0.01" iyz="0.00" izz="0.01" />
-		</inertial>
-		<visual>
-			<geometry>
-				<mesh filename="package://soft_hand_description/meshes/coman_coupler_left.stl" scale=" .001 .001 .001" />
-			</geometry>
-			<material name="SoftHand/LightBlue" />
-		</visual>
-		<collision>
-			<geometry>
-				<mesh filename="package://soft_hand_description/meshes/coman_coupler_left.stl" scale=" .001 .001 .001" />
-			</geometry>
-		</collision>
-	</link>
-	<xacro:soft_hand parent="wrist_left" name="soft_hand_left" withAdaptiveTransmission="true" useMimicTag="$(arg use_mimic_tag)" left="true">
-		<origin xyz="0.002 -0.009 0.038" rpy="0 0 0"/>
-	</xacro:soft_hand>
-	<joint name="box_wrist_right_joint" type="fixed">
-		<origin xyz="0 0.2 1.02" rpy="0 0 0" />
-		<parent link="box"/>
-		<child link="wrist_right"/>
-	</joint>
-	<link name="wrist_right">
-		<inertial>
-			<mass value="1.0"/>
-			<inertia  ixx="0.01" ixy="0.00"  ixz="0.00" iyy="0.01" iyz="0.00" izz="0.01" />
-		</inertial>
-		<visual>
-			<geometry>
-				<mesh filename="package://soft_hand_description/meshes/coman_coupler_right.stl" scale=" .001 .001 .001" />
-			</geometry>
-			<material name="SoftHand/LightBlue" />
-		</visual>
-		<collision>
-			<geometry>
-				<mesh filename="package://soft_hand_description/meshes/coman_coupler_right.stl" scale=" .001 .001 .001" />
-			</geometry>
-		</collision>
-	</link>
-	<xacro:soft_hand parent="wrist_right" name="soft_hand_right" withAdaptiveTransmission="true" useMimicTag="$(arg use_mimic_tag)" left="false">
-		<origin xyz="0.002 0.009 0.038" rpy="0 0 0"/>
+	<xacro:soft_hand parent="box" name="soft_hand_right" withAdaptiveTransmission="true" useMimicTag="$(arg use_mimic_tag)" left="true">
+		<origin xyz="0.0 0.0 1.0" rpy="0 0 0"/>
 	</xacro:soft_hand>
 </robot>

File: soft_hand/soft_hand_description/robot/two_soft_hands.urdf.xacro (robot description, xacro)
@@ -4,5 +4,5 @@
 	<link name="box">
 		<inertial>
-			<mass value="50.0"/>
+			<mass value="0.5"/>
 			<inertia  ixx="1" ixy="0.00"  ixz="0.00" iyy="1" iyz="0.00" izz="1" />
 		</inertial>
@@ -20,53 +20,9 @@
 		</collision>
 	</link>
-	<joint name="box_wrist_left_joint" type="fixed">
-		<origin xyz="0 -0.2 1.02" rpy="0 0 0" />
-		<parent link="box"/>
-		<child link="wrist_left"/>
-	</joint>
-	<link name="wrist_left">
-		<inertial>
-			<mass value="1.0"/>
-			<inertia  ixx="0.01" ixy="0.00"  ixz="0.00" iyy="0.01" iyz="0.00" izz="0.01" />
-		</inertial>
-		<visual>
-			<geometry>
-				<mesh filename="package://soft_hand_description/meshes/coman_coupler_left.stl" scale=" .001 .001 .001" />
-			</geometry>
-			<material name="SoftHand/LightBlue" />
-		</visual>
-		<collision>
-			<geometry>
-				<mesh filename="package://soft_hand_description/meshes/coman_coupler_left.stl" scale=" .001 .001 .001" />
-			</geometry>
-		</collision>
-	</link>
-	<xacro:soft_hand parent="wrist_left" name="soft_hand_left" withAdaptiveTransmission="true" useMimicTag="$(arg use_mimic_tag)" left="true">
-		<origin xyz="0.002 -0.009 0.038" rpy="0 0 0"/>
+	<xacro:soft_hand parent="box" name="soft_hand_left" withAdaptiveTransmission="true" useMimicTag="$(arg use_mimic_tag)" left="true">
+		<origin xyz="0.0 -0.1 1.0" rpy="0 0 0"/>
 	</xacro:soft_hand>
-	<joint name="box_wrist_right_joint" type="fixed">
-		<origin xyz="0 0.2 1.02" rpy="0 0 0" />
-		<parent link="box"/>
-		<child link="wrist_right"/>
-	</joint>
-	<link name="wrist_right">
-		<inertial>
-			<mass value="1.0"/>
-			<inertia  ixx="0.01" ixy="0.00"  ixz="0.00" iyy="0.01" iyz="0.00" izz="0.01" />
-		</inertial>
-		<visual>
-			<geometry>
-				<mesh filename="package://soft_hand_description/meshes/coman_coupler_right.stl" scale=" .001 .001 .001" />
-			</geometry>
-			<material name="SoftHand/LightBlue" />
-		</visual>
-		<collision>
-			<geometry>
-				<mesh filename="package://soft_hand_description/meshes/coman_coupler_right.stl" scale=" .001 .001 .001" />
-			</geometry>
-		</collision>
-	</link>
-	<xacro:soft_hand parent="wrist_right" name="soft_hand_right" withAdaptiveTransmission="true" useMimicTag="$(arg use_mimic_tag)" left="false">
-		<origin xyz="0.002 0.009 0.038" rpy="0 0 0"/>
+	<xacro:soft_hand parent="box" name="soft_hand_right" withAdaptiveTransmission="true" useMimicTag="$(arg use_mimic_tag)" left="false">
+		<origin xyz="0.0 0.1 1.0" rpy="0 0 0"/>
 	</xacro:soft_hand>
 </robot>
