Commit message: Update no the configured full actuation robot.

File: soft_hand/soft_hand_description/robot/soft_hand_full_actuation.urdf.xacro (robot description, xacro)
@@ -23,53 +23,6 @@
 		<static>true</static>
 	</gazebo>
-	<joint name="box_wrist_joint" type="fixed">
-		<origin xyz="0 0 1.02" rpy="0 0 0" />
-		<parent link="box"/>
-		<child link="wrist"/>
-	</joint>
-	<link name="wrist">
-		<inertial>
-			<insert_block name="negligible_inertia"/>
-		</inertial>
-		<visual>
-			<geometry>
-				<mesh filename="package://soft_hand_description/meshes/coman_coupler.stl" scale=" .001 .001 .001" />
-			</geometry>
-			<material name="SoftHand/LightBlue" />
-		</visual>
-		<collision>
-			<geometry>
-				<mesh filename="package://soft_hand_description/meshes/coman_coupler.stl" scale=" .001 .001 .001" />
-			</geometry>
-		</collision>
-	</link>
-	<xacro:soft_hand parent="wrist" name="soft_hand" left="false" withAdaptiveTransmission="false" useMimicTag="$(arg use_mimic_tag)">
+	<xacro:soft_hand parent="box" name="soft_hand" left="false" withAdaptiveTransmission="false" useMimicTag="$(arg use_mimic_tag)">
 		<origin xyz="0.002 0.009 0.038" rpy="0 0 0"/>
 	</xacro:soft_hand>
-	<!-- a wall to test the adaptivity
-	<joint name="box_object_joint" type="fixed">
-		<origin xyz="0.06 0 1.15" rpy="0 0 0" />
-		<parent link="box"/>
-		<child link="object"/>
-	</joint>
-	<link name="object">
-		<inertial>
-			<mass value="50.0"/>
-			<inertia  ixx="1" ixy="0.00"  ixz="0.00" iyy="1" iyz="0.00" izz="1" />
-		</inertial>
-		<visual>
-			<geometry>
-				<box size="0.05 0.07 0.25"/>
-			</geometry>
-		</visual>
-		<collision>
-			<geometry>
-				<box size="0.05 0.07 0.25"/>
-			</geometry>
-		</collision>
-	</link>
-	<gazebo reference="object">
-		<selfCollide>True</selfCollide>
-	</gazebo>
-	-->
 </robot>
