Commit message: adjusting kuka coupler collision geometry

File: soft_hand/soft_hand_description/model/accesories/kuka_coupler.urdf.xacro (robot description, xacro)
@@ -19,5 +19,5 @@
       <origin xyz="0 0 0.031" rpy="0 0 0"/>
       <geometry>
-        <cylinder radius="0.066" length="0.023"/>
+        <cylinder radius="0.033" length="0.023"/>
       </geometry>
     </collision>
