Commit message: Moving robots to an example folder into specific example packages.

File: examples/kinematic_synergy_example/robot/soft_hand_kinematic_synergy.urdf.xacro (robot description, xacro)
@@ -2,7 +2,8 @@
 <robot xmlns:xacro="http://www.ros.org/wiki/xacro" name="soft_hand">
 	<xacro:include filename="$(find soft_hand_description)/model/soft_hand.urdf.xacro"/>
+	<xacro:include filename="$(find soft_hand_description)/model/accesories/kuka_coupler.urdf.xacro"/>
 	<link name="box">
 		<inertial>
-			<mass value="0.5"/>
+			<mass value="1.0"/>
 			<inertia  ixx="1" ixy="0.00"  ixz="0.00" iyy="1" iyz="0.00" izz="1" />
 		</inertial>
@@ -20,9 +21,6 @@
 		</collision>
 	</link>
-	<xacro:soft_hand parent="box" name="soft_hand_left" withAdaptiveTransmission="true" useMimicTag="$(arg use_mimic_tag)" left="true">
-		<origin xyz="0.0 -0.1 1.0" rpy="0 0 0"/>
-	</xacro:soft_hand>
-	<xacro:soft_hand parent="box" name="soft_hand_right" withAdaptiveTransmission="true" useMimicTag="$(arg use_mimic_tag)" left="false">
-		<origin xyz="0.0 0.1 1.0" rpy="0 0 0"/>
+	<xacro:soft_hand parent="box" name="soft_hand" withAdaptiveTransmission="true" useMimicTag="true" left="true">
+		<origin xyz="0.0 0.0 1.0" rpy="0 0 0"/>
 	</xacro:soft_hand>
 </robot>

File: examples/two_hands_example/robot/two_soft_hands.urdf.xacro (robot description, xacro)
@@ -2,8 +2,7 @@
 <robot xmlns:xacro="http://www.ros.org/wiki/xacro" name="soft_hand">
 	<xacro:include filename="$(find soft_hand_description)/model/soft_hand.urdf.xacro"/>
-	<xacro:include filename="$(find soft_hand_description)/model/accesories/kuka_coupler.urdf.xacro"/>
 	<link name="box">
 		<inertial>
-			<mass value="1.0"/>
+			<mass value="0.5"/>
 			<inertia  ixx="1" ixy="0.00"  ixz="0.00" iyy="1" iyz="0.00" izz="1" />
 		</inertial>
@@ -21,6 +20,9 @@
 		</collision>
 	</link>
-	<xacro:soft_hand parent="box" name="soft_hand" withAdaptiveTransmission="true" useMimicTag="$(arg use_mimic_tag)" left="true">
-		<origin xyz="0.0 0.0 1.0" rpy="0 0 0"/>
+	<xacro:soft_hand parent="box" name="left_hand" withAdaptiveTransmission="true" useMimicTag="$(arg use_mimic_tag)" left="true">
+		<origin xyz="0.0 -0.1 1.0" rpy="0 0 0"/>
+	</xacro:soft_hand>
+	<xacro:soft_hand parent="box" name="right_hand" withAdaptiveTransmission="true" useMimicTag="$(arg use_mimic_tag)" left="false">
+		<origin xyz="0.0 0.1 1.0" rpy="0 0 0"/>
 	</xacro:soft_hand>
 </robot>
