Commit message: [interactive_grasping_simulator] Making the object fixed to world

File: examples/interactive_grasping_simulatior/urdf/object.urdf.xacro (robot description, xacro)
@@ -1,4 +1,9 @@
 <?xml version="1.0"?>
 <robot xmlns:xacro="http://www.ros.org/wiki/xacro" name="object">
+  <link name="world"/>
+  <joint name="ground_joint" type="fixed">
+    <parent link="world"/>
+      <child link="object"/>
+  </joint>
   <link name="object">
     <inertial>
@@ -18,4 +23,5 @@
   </link>
   <gazebo reference="$(arg name)">
+    <static>true</static>
     <gravity>true</gravity>
     <mu1>500.0</mu1>

Commit message: [interactive_grasping_simulator] RGBD camera added to the scene.

File: examples/interactive_grasping_simulatior/urdf/object.urdf.xacro (robot description, xacro)
@@ -3,6 +3,7 @@
   <link name="world"/>
   <joint name="ground_joint" type="fixed">
+    <origin xyz="0.0 0.2 0.3"/>
     <parent link="world"/>
-      <child link="object"/>
+    <child link="object"/>
   </joint>
   <link name="object">
@@ -23,5 +24,4 @@
   </link>
   <gazebo reference="$(arg name)">
-    <static>true</static>
     <gravity>true</gravity>
     <mu1>500.0</mu1>
@@ -30,3 +30,65 @@
     <kd>1.0</kd>
   </gazebo>
+  <joint name="asus_joint" type="fixed">
+    <origin xyz="-1.0 0.0 0.7" rpy="0.0 0.0 0.0"/>
+    <parent link="world"/>
+    <child link="asus_link"/>
+  </joint>
+  <link name="asus_link">
+    <inertial>
+        <mass value="0.2"/>
+        <inertia ixx="0.01" ixy="0.0" ixz="0.0" iyy="0.01" iyz="0.0" izz="0.01"/>
+    </inertial>
+    <visual>
+      <origin xyz="0 0 0" rpy="0.0 0.0 0.0"/>
+      <geometry>
+        <mesh filename="package://interactive_grasping_simulator/urdf/meshes/asus_xtion_body.stl"/>
+      </geometry>
+    </visual>
+    <collision>
+      <origin xyz="0 0 0" rpy="1.5707 0 0"/>
+      <geometry>
+        <cylinder radius="0.03" length="0.20"/>
+      </geometry>
+    </collision>
+  </link>
+  <gazebo reference="asus_link">
+    <gravity>true</gravity>
+    <mu1>500.0</mu1>
+    <mu2>500.0</mu2>
+    <kp>10000000.0</kp>
+    <kd>1.0</kd>
+    <sensor type="depth" name="asus_xtion">
+      <update_rate>10</update_rate>
+      <camera>
+        <horizontal_fov>1.09606677025</horizontal_fov>
+        <image>
+          <format>R8G8B8</format>
+          <width>640</width>
+          <height>480</height>
+        </image>
+        <clip>
+          <near>0.5</near>
+          <far>9</far>
+        </clip>
+      </camera>
+      <plugin filename="libgazebo_ros_openni_kinect.so" name="xtion_camera_controller">
+        <alwaysOn>true</alwaysOn>
+        <updateRate>10</updateRate>
+        <cameraName>asus</cameraName>
+        <imageTopicName>asus/rgb/image_raw</imageTopicName>
+        <cameraInfoTopicName>asus/rgb/camera_info</cameraInfoTopicName>
+        <depthImageTopicName>asus/depth/image_raw</depthImageTopicName>
+        <depthImageCameraInfoTopicName>asus/depth/camera_info</depthImageCameraInfoTopicName>
+        <pointCloudTopicName>asus/depth/points</pointCloudTopicName>
+        <frameName>asus/camera_rgb_optical_frame</frameName>
+        <pointCloudCutoff>0.5</pointCloudCutoff>
+        <distortion_k1>0.0</distortion_k1>
+        <distortion_k2>0.0</distortion_k2>
+        <distortion_k3>0.0</distortion_k3>
+        <distortion_t1>0.0</distortion_t1>
+        <distortion_t2>0.0</distortion_t2>
+      </plugin>
+    </sensor>
+  </gazebo>
 </robot>
