Commit message: Modified the adaptive example to use the hand of god plugin to position the hand and grasp a box

File: examples/adaptive_example/objects/object.urdf.xacro (robot description, xacro)
@@ -4,21 +4,21 @@
 	<link name="object">
 		<inertial>
-			<mass value="50.0"/>
+			<mass value="0.487"/>
 			<inertia  ixx="1" ixy="0.00"  ixz="0.00" iyy="1" iyz="0.00" izz="1" />
 		</inertial>
 		<visual>
 			<geometry>
-				<box size="0.05 0.05 0.25"/>
+				<box size=".072898 .1905 .12065 "/>
 			</geometry>
 		</visual>
 		<collision>
 			<geometry>
-				<box size="0.05 0.05 0.25"/>
+				<box size=".072898 .1905 .12065 "/>
 			</geometry>
 			<surface>
 				<friction>
 					<ode>
-			            <mu>5000.0</mu>
-			            <mu2>5000.0</mu2>
+			            <mu>7500.0</mu>
+			            <mu2>7500.0</mu2>
           			</ode>
         		</friction>

File: examples/adaptive_example/robot/soft_hand_adaptive.urdf.xacro (robot description, xacro)
@@ -4,25 +4,32 @@
 	<link name="box">
 		<inertial>
-			<mass value="50.0"/>
+			<mass value="1.0"/>
 			<inertia  ixx="1" ixy="0.00"  ixz="0.00" iyy="1" iyz="0.00" izz="1" />
 		</inertial>
 		<visual>
-			<origin xyz="0 0 0.50" rpy="0 0 0"/>
+			<origin xyz="0 0 0.01" rpy="0 0 0"/>
 			<geometry>
-				<box size="1.0 1.0 1.0"/>
+				<box size="0.01 0.01 0.01"/>
 			</geometry>
 		</visual>
 		<collision>
-			<origin xyz="0 0 0.50" rpy="0 0 0"/>
+			<origin xyz="0 0 0.01" rpy="0 0 0"/>
 			<geometry>
-				<box size="1.0 1.0 1.0"/>
+				<box size="0.01 0.01 0.01"/>
 			</geometry>
 		</collision>
 	</link>
+	<gazebo>
+		<plugin filename="libgazebo_ros_hand_of_god.so" name="HOG">
+			<linkName>box</linkName>
+			<frameId>box</frameId>
+			<kl>2000</kl>
+		</plugin>
+	</gazebo>
 	<gazebo reference="box">
-		<static>true</static>
+		<static>false</static>
 	</gazebo>
 	<xacro:soft_hand parent="box" name="soft_hand" withAdaptiveTransmission="true" useMimicTag="$(arg use_mimic_tag)" left="false">
-		<origin xyz="0.0 0.0 1.02" rpy="0 0 0"/>
+		<origin xyz="0.0 0.0 0.005" rpy="0 0 0"/>
 	</xacro:soft_hand>
 </robot>

Commit message: Modified transmission with lower stifness on joints and bigger value for thumb abd reduction, modified inertia value of pasta box and HOG box

File: examples/adaptive_example/objects/object.urdf.xacro (robot description, xacro)
@@ -1,24 +1,28 @@
 <?xml version="1.0"?>
 <robot xmlns:xacro="http://www.ros.org/wiki/xacro" name="object">
+	<xacro:property name="m" value="0.487" />
+	<xacro:property name="x" value="0.072898" />
+	<xacro:property name="y" value="0.1905" />
+	<xacro:property name="z" value="0.12065" />
 	<!-- a wall to test the adaptivity   -->
 	<link name="object">
 		<inertial>
-			<mass value="0.487"/>
-			<inertia  ixx="1" ixy="0.00"  ixz="0.00" iyy="1" iyz="0.00" izz="1" />
+			<mass value="${m}"/>
+			<inertia  ixx="${m*(y*y + z*z)/12}" ixy="0.00"  ixz="0.00" iyy="${m*(x*x + z*z)/12}" iyz="0.00" izz="${m*(x*x + y*y)/12}" />
 		</inertial>
 		<visual>
 			<geometry>
-				<box size=".072898 .1905 .12065 "/>
+				<box size="${x} ${y} ${z}"/>
 			</geometry>
 		</visual>
 		<collision>
 			<geometry>
-				<box size=".072898 .1905 .12065 "/>
+				<box size="${x} ${y} ${z}"/>
 			</geometry>
 			<surface>
 				<friction>
 					<ode>
-			            <mu>7500.0</mu>
-			            <mu2>7500.0</mu2>
+			            <mu>1.2</mu>
+			            <mu2>1.2</mu2>
           			</ode>
         		</friction>

File: examples/adaptive_example/robot/soft_hand_adaptive.urdf.xacro (robot description, xacro)
@@ -2,19 +2,21 @@
 <robot xmlns:xacro="http://www.ros.org/wiki/xacro" name="soft_hand">
 	<xacro:include filename="$(find soft_hand_description)/model/soft_hand.urdf.xacro"/>
+	<xacro:property name="box_m" value="0.1" />
+	<xacro:property name="box_s" value="0.01" />
 	<link name="box">
 		<inertial>
-			<mass value="1.0"/>
-			<inertia  ixx="1" ixy="0.00"  ixz="0.00" iyy="1" iyz="0.00" izz="1" />
+			<mass value="${box_m}"/>
+			<inertia  ixx="${box_m*box_s*box_s/6}" ixy="0.00"  ixz="0.00" iyy="${box_m*box_s*box_s/6}" iyz="0.00" izz="${box_m*box_s*box_s/6}" />
 		</inertial>
 		<visual>
-			<origin xyz="0 0 0.01" rpy="0 0 0"/>
+			<origin xyz="0 0 ${box_s}" rpy="0 0 0"/>
 			<geometry>
-				<box size="0.01 0.01 0.01"/>
+				<box size="${box_s} ${box_s} ${box_s}"/>
 			</geometry>
 		</visual>
 		<collision>
-			<origin xyz="0 0 0.01" rpy="0 0 0"/>
+			<origin xyz="0 0 ${box_s}" rpy="0 0 0"/>
 			<geometry>
-				<box size="0.01 0.01 0.01"/>
+				<box size="${box_s} ${box_s} ${box_s}"/>
 			</geometry>
 		</collision>
@@ -25,4 +27,5 @@
 			<frameId>box</frameId>
 			<kl>2000</kl>
+			<ka>500</ka>
 		</plugin>
 	</gazebo>

File: soft_hand_description/model/soft_hand.transmission.xacro (robot description, xacro)
@@ -82,5 +82,5 @@
           </joint>
           <actuator name="${name}_thumb_abd_motor">
-            <mechanicalReduction>1.0</mechanicalReduction>
+            <mechanicalReduction>10.0</mechanicalReduction>
           </actuator>
       </transmission>
@@ -149,6 +149,6 @@
             <role>joint1</role>
             <offset>-0.0</offset>
-            <mechanicalReduction>1.3</mechanicalReduction>
-            <mechanicalElasticity>10.0</mechanicalElasticity>
+            <mechanicalReduction>2.5</mechanicalReduction>
+            <mechanicalElasticity>2.0</mechanicalElasticity>
             <!-- hardwareInterface>PositionJointInterface</hardwareInterface -->
             <hardwareInterface>EffortJointInterface</hardwareInterface>
@@ -158,5 +158,5 @@
             <offset>-0.0</offset>
             <mechanicalReduction>1.0</mechanicalReduction>
-            <mechanicalElasticity>10.0</mechanicalElasticity>
+            <mechanicalElasticity>2.0</mechanicalElasticity>
             <!-- hardwareInterface>PositionJointInterface</hardwareInterface -->
             <hardwareInterface>EffortJointInterface</hardwareInterface>
@@ -166,5 +166,5 @@
             <offset>-0.0</offset>
             <mechanicalReduction>1.0</mechanicalReduction>
-            <mechanicalElasticity>10.0</mechanicalElasticity>
+            <mechanicalElasticity>2.0</mechanicalElasticity>
             <!-- hardwareInterface>PositionJointInterface</hardwareInterface -->
             <hardwareInterface>EffortJointInterface</hardwareInterface>
@@ -174,5 +174,5 @@
             <offset>-0.0</offset>
             <mechanicalReduction>-0.2</mechanicalReduction>
-            <mechanicalElasticity>10.0</mechanicalElasticity>
+            <mechanicalElasticity>2.0</mechanicalElasticity>
             <!-- hardwareInterface>PositionJointInterface</hardwareInterface -->
             <hardwareInterface>EffortJointInterface</hardwareInterface>
@@ -182,5 +182,5 @@
             <offset>-0.0</offset>
             <mechanicalReduction>1.0</mechanicalReduction>
-            <mechanicalElasticity>10.0</mechanicalElasticity>
+            <mechanicalElasticity>2.0</mechanicalElasticity>
             <!-- hardwareInterface>PositionJointInterface</hardwareInterface -->
             <hardwareInterface>EffortJointInterface</hardwareInterface>
@@ -190,5 +190,5 @@
             <offset>-0.0</offset>
             <mechanicalReduction>1.0</mechanicalReduction>
-            <mechanicalElasticity>10.0</mechanicalElasticity>
+            <mechanicalElasticity>2.0</mechanicalElasticity>
             <!-- hardwareInterface>PositionJointInterface</hardwareInterface -->
             <hardwareInterface>EffortJointInterface</hardwareInterface>
@@ -198,5 +198,5 @@
             <offset>-0.0</offset>
             <mechanicalReduction>1.0</mechanicalReduction>
-            <mechanicalElasticity>10.0</mechanicalElasticity>
+            <mechanicalElasticity>2.0</mechanicalElasticity>
             <!-- hardwareInterface>PositionJointInterface</hardwareInterface -->
             <hardwareInterface>EffortJointInterface</hardwareInterface>
@@ -206,5 +206,5 @@
             <offset>-0.0</offset>
             <mechanicalReduction>0.001</mechanicalReduction>
-            <mechanicalElasticity>10.0</mechanicalElasticity>
+            <mechanicalElasticity>2.0</mechanicalElasticity>
             <!-- hardwareInterface>PositionJointInterface</hardwareInterface -->
             <hardwareInterface>EffortJointInterface</hardwareInterface>
@@ -214,5 +214,5 @@
             <offset>-0.0</offset>
             <mechanicalReduction>1.0</mechanicalReduction>
-            <mechanicalElasticity>10.0</mechanicalElasticity>
+            <mechanicalElasticity>2.0</mechanicalElasticity>
             <!-- hardwareInterface>PositionJointInterface</hardwareInterface -->
             <hardwareInterface>EffortJointInterface</hardwareInterface>
@@ -222,5 +222,5 @@
             <offset>-0.0</offset>
             <mechanicalReduction>1.0</mechanicalReduction>
-            <mechanicalElasticity>10.0</mechanicalElasticity>
+            <mechanicalElasticity>2.0</mechanicalElasticity>
             <!-- hardwareInterface>PositionJointInterface</hardwareInterface -->
             <hardwareInterface>EffortJointInterface</hardwareInterface>
@@ -230,5 +230,5 @@
             <offset>-0.0</offset>
             <mechanicalReduction>1.0</mechanicalReduction>
-            <mechanicalElasticity>10.0</mechanicalElasticity>
+            <mechanicalElasticity>2.0</mechanicalElasticity>
             <!-- hardwareInterface>PositionJointInterface</hardwareInterface -->
             <hardwareInterface>EffortJointInterface</hardwareInterface>
@@ -238,5 +238,5 @@
             <offset>-0.0</offset>
             <mechanicalReduction>0.2</mechanicalReduction>
-            <mechanicalElasticity>10.0</mechanicalElasticity>
+            <mechanicalElasticity>2.0</mechanicalElasticity>
             <!-- hardwareInterface>PositionJointInterface</hardwareInterface -->
             <hardwareInterface>EffortJointInterface</hardwareInterface>
@@ -246,5 +246,5 @@
             <offset>-0.0</offset>
             <mechanicalReduction>1.0</mechanicalReduction>
-            <mechanicalElasticity>10.0</mechanicalElasticity>
+            <mechanicalElasticity>2.0</mechanicalElasticity>
             <!-- hardwareInterface>PositionJointInterface</hardwareInterface -->
             <hardwareInterface>EffortJointInterface</hardwareInterface>
@@ -254,5 +254,5 @@
             <offset>-0.0</offset>
             <mechanicalReduction>1.0</mechanicalReduction>
-            <mechanicalElasticity>10.0</mechanicalElasticity>
+            <mechanicalElasticity>2.0</mechanicalElasticity>
             <!-- hardwareInterface>PositionJointInterface</hardwareInterface -->
             <hardwareInterface>EffortJointInterface</hardwareInterface>
@@ -262,5 +262,5 @@
             <offset>-0.0</offset>
             <mechanicalReduction>1.0</mechanicalReduction>
-            <mechanicalElasticity>10.0</mechanicalElasticity>
+            <mechanicalElasticity>2.0</mechanicalElasticity>
             <!-- hardwareInterface>PositionJointInterface</hardwareInterface -->
             <hardwareInterface>EffortJointInterface</hardwareInterface>
@@ -270,5 +270,5 @@
             <offset>-0.0</offset>
             <mechanicalReduction>0.4</mechanicalReduction>
-            <mechanicalElasticity>10.0</mechanicalElasticity>
+            <mechanicalElasticity>2.0</mechanicalElasticity>
             <!-- hardwareInterface>PositionJointInterface</hardwareInterface -->
             <hardwareInterface>EffortJointInterface</hardwareInterface>
@@ -278,5 +278,5 @@
             <offset>-0.0</offset>
             <mechanicalReduction>1.0</mechanicalReduction>
-            <mechanicalElasticity>10.0</mechanicalElasticity>
+            <mechanicalElasticity>2.0</mechanicalElasticity>
             <!-- hardwareInterface>PositionJointInterface</hardwareInterface -->
             <hardwareInterface>EffortJointInterface</hardwareInterface>
@@ -286,5 +286,5 @@
             <offset>-0.0</offset>
             <mechanicalReduction>1.0</mechanicalReduction>
-            <mechanicalElasticity>10.0</mechanicalElasticity>
+            <mechanicalElasticity>2.0</mechanicalElasticity>
             <!-- hardwareInterface>PositionJointInterface</hardwareInterface -->
             <hardwareInterface>EffortJointInterface</hardwareInterface>
@@ -294,5 +294,5 @@
             <offset>-0.0</offset>
             <mechanicalReduction>1.0</mechanicalReduction>
-            <mechanicalElasticity>10.0</mechanicalElasticity>
+            <mechanicalElasticity>2.0</mechanicalElasticity>
             <!-- hardwareInterface>PositionJointInterface</hardwareInterface -->
             <hardwareInterface>EffortJointInterface</hardwareInterface>
