Commit message: adjusted some deprecated definitions for ros kinetic

File: soft_hand_description/model/accesories/clamp.urdf.xacro (robot description, xacro)
@@ -3,5 +3,5 @@
 <xacro:macro name="clamp" params="parent name *origin">
   <joint name="${parent}_${name}_joint" type="fixed">
-    <insert_block name="origin"/>
+    <xacro:insert_block name="origin"/>
     <parent link="${parent}"/>
     <child link="${name}"/>

File: soft_hand_description/model/accesories/kuka_coupler.urdf.xacro (robot description, xacro)
@@ -3,5 +3,5 @@
 <xacro:macro name="kuka_coupler" params="parent name *origin">
   <joint name="${parent}_${name}_joint" type="fixed">
-    <insert_block name="origin"/>
+    <xacro:insert_block name="origin"/>
     <parent link="${parent}"/>
     <child link="${name}_bottom"/>

File: soft_hand_description/model/accesories/softhand_base.urdf.xacro (robot description, xacro)
@@ -3,5 +3,5 @@
 <xacro:macro name="softhand_base" params="parent name left *origin">
   <joint name="${parent}_${name}_joint" type="fixed">
-    <insert_block name="origin"/>
+    <xacro:insert_block name="origin"/>
     <parent link="${parent}"/>
     <child link="${name}"/>

File: soft_hand_description/model/soft_hand.gazebo.xacro (robot description, xacro)
@@ -1,4 +1,4 @@
 <?xml version="1.0"?>
-<robot xmlns:xacro="http://ros.org/wiki/xacro">
+<robot xmlns:xacro="http://www.ros.org/wiki/xacro">
 	<!-- configure how all joints will behave in gazebo (particular behavior can be set at each joint as well) -->
 	<xacro:property name="gazebo_joint_elements">

File: soft_hand_description/model/soft_hand.inertia.xacro (robot description, xacro)
@@ -1,4 +1,4 @@
 <?xml version="1.0"?>
-<robot xmlns:xacro="http://ros.org/wiki/xacro">
+<robot xmlns:xacro="http://www.ros.org/wiki/xacro">
     <!-- NOTE: inertia values are approximated using meshlab and only using the significant elements -->
     <!-- from http://answers.ros.org/question/11350/is-there-any-way-to-calculate-inertial-property-of-a-robot-to-simulate-it-in-gazebo/s

File: soft_hand_description/model/soft_hand.urdf.xacro (robot description, xacro)
@@ -1,4 +1,4 @@
 <?xml version="1.0"?>
-<robot xmlns:xacro="http://ros.org/wiki/xacro">
+<robot xmlns:xacro="http://www.ros.org/wiki/xacro">
 	<!-- include other model components -->
 	<xacro:include filename="$(find soft_hand_description)/model/materials.urdf.xacro"/>
@@ -10,5 +10,4 @@
 	<xacro:include filename="$(find soft_hand_description)/model/accesories/clamp.urdf.xacro"/>
 	<xacro:include filename="$(find soft_hand_description)/model/accesories/softhand_base.urdf.xacro"/>
-	<xacro:property name="pi" value="3.1415926535897931" />
 	<!-- joint properties -->
 	<xacro:property name="abd_lb" value="-30" />
@@ -76,5 +75,5 @@
 		<link name="${name}_knuckle_link">
 			<inertial>
-				<insert_block name="knuckle_inertia"/>
+				<xacro:insert_block name="knuckle_inertia"/>
 			</inertial>
 			<visual>
@@ -104,5 +103,5 @@
 		<link name="${name}_fake_link1">
 			<inertial>
-				<insert_block name="negligible_inertia"/>
+				<xacro:insert_block name="negligible_inertia"/>
 			</inertial>
 		</link>
@@ -120,5 +119,5 @@
 		<link name="${name}_proximal_link">
 			<inertial>
-				<insert_block name="phalanx_inertia"/>
+				<xacro:insert_block name="phalanx_inertia"/>
 			</inertial>
 			<visual>
@@ -148,5 +147,5 @@
 		<link name="${name}_fake_link2">
 			<inertial>
-				<insert_block name="negligible_inertia"/>
+				<xacro:insert_block name="negligible_inertia"/>
 			</inertial>
 		</link>
@@ -164,5 +163,5 @@
 		<link name="${name}_middle_link">
 			<inertial>
-				<insert_block name="phalanx_inertia"/>
+				<xacro:insert_block name="phalanx_inertia"/>
 			</inertial>
 			<visual>
@@ -192,5 +191,5 @@
 		<link name="${name}_fake_link3">
 			<inertial>
-				<insert_block name="negligible_inertia"/>
+				<xacro:insert_block name="negligible_inertia"/>
 			</inertial>
 		</link>
@@ -208,5 +207,5 @@
 		<link name="${name}_distal_link">
 			<inertial>
-				<insert_block name="fingertip_inertia"/>
+				<xacro:insert_block name="fingertip_inertia"/>
 			</inertial>
 			<visual>
@@ -241,5 +240,5 @@
 			<link name="${name}_knuckle_link">
 				<inertial>
-					<insert_block name="thumb_knuckle_inertia"/>
+					<xacro:insert_block name="thumb_knuckle_inertia"/>
 				</inertial>
 				<visual>
@@ -283,5 +282,5 @@
 			<link name="${name}_knuckle_link">
 				<inertial>
-					<insert_block name="thumb_knuckle_inertia"/>
+					<xacro:insert_block name="thumb_knuckle_inertia"/>
 				</inertial>
 				<visual>
@@ -313,5 +312,5 @@
 		<link name="${name}_fake_link1">
 			<inertial>
-				<insert_block name="negligible_inertia"/>
+				<xacro:insert_block name="negligible_inertia"/>
 			</inertial>
 		</link>
@@ -329,5 +328,5 @@
 		<link name="${name}_proximal_link">
 			<inertial>
-				<insert_block name="phalanx_inertia"/>
+				<xacro:insert_block name="phalanx_inertia"/>
 			</inertial>
 			<visual>
@@ -357,5 +356,5 @@
 		<link name="${name}_fake_link3">
 			<inertial>
-				<insert_block name="negligible_inertia"/>
+				<xacro:insert_block name="negligible_inertia"/>
 			</inertial>
 		</link>
@@ -373,5 +372,5 @@
 		<link name="${name}_distal_link">
 			<inertial>
-				<insert_block name="fingertip_inertia"/>
+				<xacro:insert_block name="fingertip_inertia"/>
 			</inertial>
 			<visual>
@@ -393,5 +392,5 @@
 		<!-- KUKA_COUPLER -->
 		<xacro:kuka_coupler parent="${parent}" name="${name}_kuka_coupler">
-			<insert_block name="origin"/>
+			<xacro:insert_block name="origin"/>
 		</xacro:kuka_coupler>
 		<!-- CLAMP -->
@@ -416,5 +415,5 @@
 		<link name="${name}_palm_link">
 			<inertial>
-				<insert_block name="palm_inertia"/>
+				<xacro:insert_block name="palm_inertia"/>
 			</inertial>
 			<xacro:if value="${left}">
@@ -455,5 +454,5 @@
 		<link name="${name}_invisible_wire_link">
 			<inertial>
-				<insert_block name="negligible_inertia"/>
+				<xacro:insert_block name="negligible_inertia"/>
 			</inertial>
 		</link>
