Commit message: The panda flange has been scaled and now only the transforms need to be adjusted

File: soft_hand_description/model/accesories/panda_flange.urdf.xacro (robot description, xacro)
@@ -11,5 +11,5 @@
       <origin xyz="0 0 0" rpy="0 0 0"/>
       <geometry>
-        <mesh filename="package://soft_hand_description/meshes/accesories/panda_flange.stl"/>
+        <mesh filename="package://soft_hand_description/meshes/accesories/panda_flange.stl" scale="0.001 0.001 0.001"/>
       </geometry>
       <material name="SoftHand/Blue"/>

File: soft_hand_description/model/soft_hand_soma_panda.urdf.xacro (robot description, xacro)
@@ -394,5 +394,5 @@
 		</xacro:panda_flange>
 		<!-- SOFT HAND ROUND BASE -->
-		<xacro:softhand_round_base parent="${name}_panda_flange" name="${name}_softhand_round_base" left="${left}">
+		<xacro:softhand_round_base parent="${name}_panda_flange" name="${name}_softhand_round_base">
 			<origin xyz="0.0 0.0 0.0" rpy="0.0 0.0 0.0"/>
 		</xacro:softhand_round_base>

Commit message: Minor measure adjustments

File: soft_hand_description/model/accesories/panda_flange.urdf.xacro (robot description, xacro)
@@ -13,10 +13,10 @@
         <mesh filename="package://soft_hand_description/meshes/accesories/panda_flange.stl" scale="0.001 0.001 0.001"/>
       </geometry>
-      <material name="SoftHand/Blue"/>
+      <material name="SoftHand/DarkGrey"/>
     </visual>
     <collision>
-      <origin xyz="0 0 0" rpy="0 0 0"/>
+      <origin xyz="0 0.04 -0.02" rpy="0 0 0"/>
       <geometry>
-        <box size="0.066 0.0725 0.0256"/>
+        <box size="0.08 0.08 0.08"/>
       </geometry>
     </collision>

File: soft_hand_description/model/soft_hand_soma_panda.urdf.xacro (robot description, xacro)
@@ -403,5 +403,5 @@
 			</xacro:if>
 			<xacro:unless value="${left}">
-				<origin xyz="-0.008 0.008 0.018" rpy="0 0 1.5707"/>
+				<origin xyz="-0.008 0.005 0.018" rpy="0 0 1.5707"/>
 			</xacro:unless>
 			<parent link="${name}_softhand_round_base" />
