Commit message: grouping all together friction properties; noting also other properties from http://gazebosim.org/tutorials/?tut=ros_urdf

File: soft_hand_description/model/soft_hand.gazebo.xacro (robot description, xacro)
@@ -13,4 +13,24 @@
 		-->
 	</xacro:property>
+	<!-- set friction properties -->
+	<xacro:property name="gazebo_friction_properties">
+		<gravity>true</gravity>
+		<mu1>500.0</mu1>
+		<mu2>500.0</mu2>
+		<kp>10000000.0</kp>
+		<kd>1.0</kd>
+		<!-- <fdir1>string</fdir1> -->
+		<!-- <dampingFactor>double</dampingFactor> -->
+		<!-- <maxVel>double</maxVel> -->
+		<!-- <minDepth>double</minDepth> -->
+		<!-- <maxContacts>int</maxContacts> -->
+	</xacro:property>
+	<!-- <xacro:insert_block name="gazebo_friction_properties"/> -->
+	<xacro:property name="gazebo_other_properties">
+		<!-- <material>value</material> -->
+		<!-- <selfCollide>bool</selfCollide> -->
+		<!-- <laserRetro>double</laserRetro> -->
+	</xacro:property>
+	<!-- <xacro:insert_block name="gazebo_other_properties"/> -->
 	<xacro:macro name="soft_hand_gazebo" params="name withAdaptiveTransmission useMimicTag">
 		<!-- PLUGINS -->
@@ -56,10 +76,5 @@
 				</plugin>
 			</sensor>
-			<!--selfCollide>true</selfCollide-->
-			<gravity>true</gravity>
-			<mu1>500.0</mu1>
-			<mu2>500.0</mu2>
-			<kp>10000000.0</kp>
-			<kd>1.0</kd>
+			<xacro:insert_block name="gazebo_friction_properties"/>
 		</gazebo>
 		<gazebo reference="${name}_thumb_knuckle_link">
@@ -80,10 +95,5 @@
 				</plugin>
 			</sensor>
-			<!--selfCollide>true</selfCollide-->
-			<gravity>true</gravity>
-			<mu1>500.0</mu1>
-			<mu2>500.0</mu2>
-			<kp>10000000.0</kp>
-			<kd>1.0</kd>
+			<xacro:insert_block name="gazebo_friction_properties"/>
 		</gazebo>
 		<gazebo reference="${name}_thumb_proximal_link">
@@ -104,10 +114,5 @@
 				</plugin>
 			</sensor>
-			<!--selfCollide>true</selfCollide-->
-			<gravity>true</gravity>
-			<mu1>500.0</mu1>
-			<mu2>500.0</mu2>
-			<kp>10000000.0</kp>
-			<kd>1.0</kd>
+			<xacro:insert_block name="gazebo_friction_properties"/>
 		</gazebo>
 		<gazebo reference="${name}_thumb_distal_link">
@@ -128,10 +133,5 @@
 				</plugin>
 			</sensor>
-			<!-- selfCollide>true</selfCollide-->
-			<gravity>true</gravity>
-			<mu1>500.0</mu1>
-			<mu2>500.0</mu2>
-			<kp>10000000.0</kp>
-			<kd>1.0</kd>
+			<xacro:insert_block name="gazebo_friction_properties"/>
 		</gazebo>
 		<gazebo reference="${name}_index_knuckle_link">
@@ -152,10 +152,5 @@
 				</plugin>
 			</sensor>
-			<!--selfCollide>true</selfCollide-->
-			<gravity>true</gravity>
-			<mu1>500.0</mu1>
-			<mu2>500.0</mu2>
-			<kp>10000000.0</kp>
-			<kd>1.0</kd>
+			<xacro:insert_block name="gazebo_friction_properties"/>
 		</gazebo>
 		<gazebo reference="${name}_index_proximal_link">
@@ -176,10 +171,5 @@
 				</plugin>
 			</sensor>
-			<!--selfCollide>true</selfCollide-->
-			<gravity>true</gravity>
-			<mu1>500.0</mu1>
-			<mu2>500.0</mu2>
-			<kp>10000000.0</kp>
-			<kd>1.0</kd>
+			<xacro:insert_block name="gazebo_friction_properties"/>
 		</gazebo>
 		<gazebo reference="${name}_index_middle_link">
@@ -200,10 +190,5 @@
 				</plugin>
 			</sensor>
-			<!--selfCollide>true</selfCollide-->
-			<gravity>true</gravity>
-			<mu1>500.0</mu1>
-			<mu2>500.0</mu2>
-			<kp>10000000.0</kp>
-			<kd>1.0</kd>
+			<xacro:insert_block name="gazebo_friction_properties"/>
 		</gazebo>
 		<gazebo reference="${name}_index_distal_link">
@@ -224,10 +209,5 @@
 				</plugin>
 			</sensor>
-			<!-- selfCollide>true</selfCollide-->
-			<gravity>true</gravity>
-			<mu1>500.0</mu1>
-			<mu2>500.0</mu2>
-			<kp>10000000.0</kp>
-			<kd>1.0</kd>
+			<xacro:insert_block name="gazebo_friction_properties"/>
 		</gazebo>
 		<gazebo reference="${name}_middle_knuckle_link">
@@ -248,10 +228,5 @@
 				</plugin>
 			</sensor>
-			<!--selfCollide>true</selfCollide-->
-			<gravity>true</gravity>
-			<mu1>500.0</mu1>
-			<mu2>500.0</mu2>
-			<kp>10000000.0</kp>
-			<kd>1.0</kd>
+			<xacro:insert_block name="gazebo_friction_properties"/>
 		</gazebo>
 		<gazebo reference="${name}_middle_proximal_link">
@@ -272,10 +247,5 @@
 				</plugin>
 			</sensor>
-			<!--selfCollide>true</selfCollide-->
-			<gravity>true</gravity>
-			<mu1>500.0</mu1>
-			<mu2>500.0</mu2>
-			<kp>10000000.0</kp>
-			<kd>1.0</kd>
+			<xacro:insert_block name="gazebo_friction_properties"/>
 		</gazebo>
 		<gazebo reference="${name}_middle_middle_link">
@@ -296,10 +266,5 @@
 				</plugin>
 			</sensor>
-			<!--selfCollide>true</selfCollide-->
-			<gravity>true</gravity>
-			<mu1>500.0</mu1>
-			<mu2>500.0</mu2>
-			<kp>10000000.0</kp>
-			<kd>1.0</kd>
+			<xacro:insert_block name="gazebo_friction_properties"/>
 		</gazebo>
 		<gazebo reference="${name}_middle_distal_link">
@@ -320,10 +285,5 @@
 				</plugin>
 			</sensor>
-			<!-- selfCollide>true</selfCollide-->
-			<gravity>true</gravity>
-			<mu1>500.0</mu1>
-			<mu2>500.0</mu2>
-			<kp>10000000.0</kp>
-			<kd>1.0</kd>
+			<xacro:insert_block name="gazebo_friction_properties"/>
 		</gazebo>
 		<gazebo reference="${name}_ring_knuckle_link">
@@ -344,10 +304,5 @@
 				</plugin>
 			</sensor>
-			<!--selfCollide>true</selfCollide-->
-			<gravity>true</gravity>
-			<mu1>500.0</mu1>
-			<mu2>500.0</mu2>
-			<kp>10000000.0</kp>
-			<kd>1.0</kd>
+			<xacro:insert_block name="gazebo_friction_properties"/>
 		</gazebo>
 		<gazebo reference="${name}_ring_proximal_link">
@@ -368,10 +323,5 @@
 				</plugin>
 			</sensor>
-			<!--selfCollide>true</selfCollide-->
-			<gravity>true</gravity>
-			<mu1>500.0</mu1>
-			<mu2>500.0</mu2>
-			<kp>10000000.0</kp>
-			<kd>1.0</kd>
+			<xacro:insert_block name="gazebo_friction_properties"/>
 		</gazebo>
 		<gazebo reference="${name}_ring_middle_link">
@@ -392,10 +342,5 @@
 				</plugin>
 			</sensor>
-			<!--selfCollide>true</selfCollide-->
-			<gravity>true</gravity>
-			<mu1>500.0</mu1>
-			<mu2>500.0</mu2>
-			<kp>10000000.0</kp>
-			<kd>1.0</kd>
+			<xacro:insert_block name="gazebo_friction_properties"/>
 		</gazebo>
 		<gazebo reference="${name}_ring_distal_link">
@@ -416,10 +361,5 @@
 				</plugin>
 			</sensor>
-			<!-- selfCollide>true</selfCollide-->
-			<gravity>true</gravity>
-			<mu1>500.0</mu1>
-			<mu2>500.0</mu2>
-			<kp>10000000.0</kp>
-			<kd>1.0</kd>
+			<xacro:insert_block name="gazebo_friction_properties"/>
 		</gazebo>
 		<gazebo reference="${name}_little_knuckle_link">
@@ -440,10 +380,5 @@
 				</plugin>
 			</sensor>
-			<!--selfCollide>true</selfCollide-->
-			<gravity>true</gravity>
-			<mu1>500.0</mu1>
-			<mu2>500.0</mu2>
-			<kp>10000000.0</kp>
-			<kd>1.0</kd>
+			<xacro:insert_block name="gazebo_friction_properties"/>
 		</gazebo>
 		<gazebo reference="${name}_little_proximal_link">
@@ -464,10 +399,5 @@
 				</plugin>
 			</sensor>
-			<!--selfCollide>true</selfCollide-->
-			<gravity>true</gravity>
-			<mu1>500.0</mu1>
-			<mu2>500.0</mu2>
-			<kp>10000000.0</kp>
-			<kd>1.0</kd>
+			<xacro:insert_block name="gazebo_friction_properties"/>
 		</gazebo>
 		<gazebo reference="${name}_little_middle_link">
@@ -488,10 +418,5 @@
 				</plugin>
 			</sensor>
-			<!--selfCollide>true</selfCollide-->
-			<gravity>true</gravity>
-			<mu1>500.0</mu1>
-			<mu2>500.0</mu2>
-			<kp>10000000.0</kp>
-			<kd>1.0</kd>
+			<xacro:insert_block name="gazebo_friction_properties"/>
 		</gazebo>
 		<gazebo reference="${name}_little_distal_link">
@@ -512,10 +437,5 @@
 				</plugin>
 			</sensor>
-			<!-- selfCollide>true</selfCollide-->
-			<gravity>true</gravity>
-			<mu1>500.0</mu1>
-			<mu2>500.0</mu2>
-			<kp>10000000.0</kp>
-			<kd>1.0</kd>
+			<xacro:insert_block name="gazebo_friction_properties"/>
 		</gazebo>
 		<!-- JOINTS -->

Commit message: separated palm properties from other links properties

File: soft_hand_description/model/soft_hand.gazebo.xacro (robot description, xacro)
@@ -4,27 +4,36 @@
 	<xacro:property name="gazebo_joint_elements">
 		<provideFeedback>True</provideFeedback>
-		<!--
-		<kp> </kp>
-		<kd> 1.0 </kd>
-		<stopCfm> </stopCfm>
-		<stopErp> </stopErp>
-		<cfmDamping> </cfmDamping>
-		<fudgeFactor> </fudgeFactor>
-		-->
+		<!-- <stopCfm> </stopCfm> -->
+		<!-- <stopErp> </stopErp> -->
+		<implicitSpringDamper>1</implicitSpringDamper>
+		<!-- <fudgeFactor> </fudgeFactor> -->
 	</xacro:property>
 	<!-- set friction properties -->
+	<!-- rubber has kp=1000000.0, kd=100.0, as in atlas_v5.gazebo in DRCsim >> the hand has a rubber-like glove! -->
+	<!-- atlas soles have mu1=mu2=1.5 in atlas_v5.gazebo in DRCsim -->
 	<xacro:property name="gazebo_friction_properties">
-		<gravity>true</gravity>
-		<mu1>500.0</mu1>
-		<mu2>500.0</mu2>
+		<!-- <gravity>true</gravity> -->
+		<mu1>1.1</mu1>
+		<mu2>1.1</mu2>
 		<kp>1000000.0</kp>
 		<kd>100.0</kd>
 		<!-- <fdir1>string</fdir1> -->
 		<!-- <dampingFactor>double</dampingFactor> -->
-		<!-- <maxVel>double</maxVel> -->
-		<!-- <minDepth>double</minDepth> -->
-		<!-- <maxContacts>int</maxContacts> -->
+		<maxVel>0.1</maxVel>
+		<minDepth>0.001</minDepth>
+		<maxContacts>3</maxContacts>
+		<!-- <material>Gazebo/Orange</material> -->
 	</xacro:property>
 	<!-- <xacro:insert_block name="gazebo_friction_properties"/> -->
+	<xacro:property name="gazebo_friction_properties_palm">
+		<mu1>1.1</mu1>
+		<mu2>1.1</mu2>
+		<kp>1000000.0</kp>
+		<kd>10.0</kd>
+		<maxVel>0.1</maxVel>
+		<minDepth>0.001</minDepth>
+		<maxContacts>6</maxContacts>
+		<!-- <material>Gazebo/Orange</material> -->
+	</xacro:property>
 	<!-- configure how all links will behave in gazebo (particular behavior can be set at each link as well) -->
 	<xacro:property name="gazebo_link_elements">
@@ -35,4 +44,8 @@
 		<selfCollide>false</selfCollide>
 		<xacro:insert_block name="gazebo_friction_properties"/>
+	</xacro:property>
+	<xacro:property name="gazebo_palm_element">
+		<selfCollide>true</selfCollide>
+		<xacro:insert_block name="gazebo_friction_properties_palm"/>
 	</xacro:property>
 	<xacro:property name="gazebo_other_properties">
@@ -92,5 +105,5 @@
 				</plugin>
 			</sensor>
-			<xacro:insert_block name="gazebo_link_elements"/>
+			<xacro:insert_block name="gazebo_palm_element"/>
 			<collision>
 				<xacro:collideBitmask hex_collision="0x49250"/>
